File: hardware/tools/diffprobe/simpleversion_eagle/diff_probe.brd (EAGLE design)
At the start: 26.7 x 26.3 mm, 24 parts, among them U1 AD8129, X1 SMA-142-0701-801/806

Commit message: Update GIT repository
Parts:
- C7: value 10nF -> 100nF
Changed lines of the file:
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@@
 <element name="D1" library="adafruit" package="SOD-123" value="" x="13.335" y="17.78" rot="MR270"/>
 <element name="C4" library="rcl" package="C0603" value="10nF" x="19.685" y="27.305" rot="MR180"/>
-<element name="C7" library="rcl" package="C0603" value="10nF" x="18.727421875" y="27.305"/>
+<element name="C7" library="rcl" package="C0603" value="100nF" x="18.727421875" y="27.305"/>
 <element name="C6" library="rcl" package="C0805" value="10u" x="14.605" y="23.495" rot="MR180"/>
 <element name="C8" library="rcl" package="C0805" value="10u" x="18.415" y="23.495" rot="MR0"/>
