File: hardware/tools/diffprobe/simpleversion_eagle/diff_probe.sch (EAGLE design)
At the start: 24 parts, among them U1 AD8129, X1 SMA-142-0701-801/806

Commit message: Update GIT repository
Parts:
- C7: value 10nF -> 100nF
Changed lines of the file:
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@@
 <part name="SUPPLY8" library="adc_microboard" deviceset="AGND" device=""/>
 <part name="C4" library="rcl" deviceset="C-EU" device="C0603" value="10nF"/>
-<part name="C7" library="rcl" deviceset="C-EU" device="C0603" value="10nF"/>
+<part name="C7" library="rcl" deviceset="C-EU" device="C0603" value="100nF"/>
 <part name="SUPPLY9" library="adc_microboard" deviceset="AGND" device=""/>
 <part name="SUPPLY10" library="adc_microboard" deviceset="AGND" device=""/>
