File: hardware/targets/ztex/pcb/ztex_openadc_eagle/openadc_ztex.brd (EAGLE design)
At the start: 83.8 x 48.3 mm, 35 parts, among them CON1 DC_SOCKET5870, CON2 PWRCON, CON3 JTAG, CON4 JTAG, CON6 USB-FPGA1.15, IC1 AOZ1021, IC2 AOZ1021, IC3 AOZ1094

Commit message: Update PCB
Parts:
- added C9: 22µ, myrcl:C0805K
- added D1: (no value), diode:DO214AA
- added L3: 2.2uF, inductors:DR1030
- IC3: device mystuff:AOZ1021 -> mystuff:AOZ1094.PAC
- moved IC3 75.2 mm to (58.2, 27.9), turned to 90 degrees
- moved R12 67.5 mm to (52.4, 29.8), turned to 90 degrees
- moved C11 24.1 mm to (45.4, 23.5), turned to 0 degrees
- moved R9 1.62 mm to (54.9, 32.7)
- moved C14 1.42 mm to (45.4, 19.4)
- moved C7 1.27 mm to (65.0, 26.8)
- moved C8 1.27 mm to (65.0, 30.0)
- moved C10 0.63 mm to (57.1, 33.7)
Connections:
- removed net N$18: CON6.C18, CON6.C29, CON6.D18
- removed net N$19: CON6.C19, CON6.C28, CON6.D28
- removed net N$6: CON6.A22, CON6.A31, CON6.B22, CON6.B31
- new net N$5: D1.C, IC3.LX, L3.1
- net +1.2V: now also C9.2, CON6.C19, CON6.C28, CON6.D28, L3.2
- net +2.6V: now also CON6.C18, CON6.C29, CON6.D18
- net GND: now also C9.1, D1.A
- net VCCO_IO: now also CON6.A22, CON6.A31, CON6.B22, CON6.B31
- net VCCO_TOP: now also CON6.C27, CON6.C7, CON6.D27, CON6.D7
Routing:
- net GND: track 273.2 -> 287.3 mm
- net N$2: track 0.00 -> 3.35 mm
- net VIN: track 184.5 -> 182.0 mm
- net +1.2V: track 115.3 -> 113.2 mm
- net VCCO_TOP: track 79.7 -> 80.7 mm
- added copper zone on layer 1, net N$5
- removed copper zone on layer 1, net LX

Commit message: Update GIT repository
Parts:
- removed CON4: JTAG, usb-fpga-1:JTAG
- added JP2, JP3: (no value), pinhead:2X15
- JP1: value EXP1.2-VJUMP -> (none); device mystuff:EXP1.2-VJUMP -> pinhead:1X02
- moved JP1 26.2 mm to (7.94, 42.9), turned to 90 degrees
Connections:
- removed net N$12: CON6.A1, CON6.B1
- removed net N$16: CON6.C6, CON6.D6
- removed net N$9: CON6.E12, CON6.E28
- removed net VCCO_IO: CON6.A22, CON6.A31, CON6.B22, CON6.B31, JP1.V_IO
- removed net VCCO_TOP: CON6.C27, CON6.C7, CON6.D27, CON6.D7, JP1.V_TOP
- net +1.2V: no longer JP1.1V2_1, JP1.1V2_2
- net +2.6V: no longer CON4.2, JP1.2V5_1, JP1.2V5_2
- net +3V3: now also CON6.A22, CON6.A31, CON6.B22, CON6.B31, CON6.C27, CON6.C6, CON6.C7, CON6.D27, CON6.D6, CON6.D7; no longer CON4.1, JP1.3V3_1, JP1.3V3_2
- net GND: no longer CON4.8
- net N$13: now also JP1.2
- net N$23: no longer CON4.7
- net N$24: no longer CON4.6
- net N$25: no longer CON4.5
- net N$26: no longer CON4.4
- net VIN: now also CON6.A1, CON6.B1, JP1.1
Routing:
- net +3V3: track 108.4 -> 261.6 mm, vias 3 -> 4
- net GND: track 287.3 -> 138.6 mm, vias 68 -> 62
- net VCCO_TOP: track 80.7 -> 0.00 mm, vias 5 -> 0
- net +2.6V: track 141.9 -> 92.2 mm, vias 2 -> 1
- net VIN: track 182.0 -> 217.9 mm
- net N$25: track 45.0 -> 10.4 mm, vias 2 -> 1
- net VCCO_IO: track 30.1 -> 0.00 mm, vias 1 -> 0
- net N$26: track 33.4 -> 10.2 mm, vias 1 -> 0
- net N$23: track 27.7 -> 12.1 mm, vias 2 -> 1
- net N$24: track 24.2 -> 9.91 mm
- net +1.2V: track 113.2 -> 123.1 mm
- net N$13: track 0.00 -> 7.30 mm
- net N$15: track 0.00 -> 5.08 mm

Commit message: Update ZTEX
Parts:
- removed JP2, JP3: (no value), pinhead:2X15
- added U$3, U$5: OPENADC, openadc_footprint:OPENADCREV1
Connections:
- new net N$32: CON6.F23, U$5.1
- new net N$34: CON6.D20, U$5.26
- new net N$35: CON6.C24, U$5.7
- new net N$40: CON6.F20, U$5.25
- new net N$44: CON6.C21, U$5.24
- new net N$45: CON6.D21, U$5.23
- new net N$46: CON6.F21, U$5.22
- new net N$47: CON6.C22, U$5.20
- new net N$48: CON6.D22, U$5.19
- new net N$49: CON6.F22, U$5.8
- new net N$50: CON6.D24, U$5.6
- new net N$51: CON6.F24, U$5.5
- new net N$52: CON6.C25, U$5.4
- new net N$53: CON6.D25, U$5.3
- new net N$54: CON6.F25, U$5.2
- new net OA_ADC0: CON6.D10, U$3.24
- new net OA_ADC1: CON6.F11, U$3.21
- new net OA_ADC2: CON6.D11, U$3.22
- new net OA_ADC3: CON6.F12, U$3.19
- new net OA_ADC4: CON6.D12, U$3.20
- new net OA_ADC5: CON6.F13, U$3.7
- new net OA_ADC6: CON6.D13, U$3.8
- new net OA_ADC7: CON6.F14, U$3.5
- new net OA_ADC8: CON6.D14, U$3.6
- new net OA_ADC9: CON6.F15, U$3.3
- new net OA_ADCOR: CON6.D15, U$3.4
- new net OA_CLKADC: CON6.F10, U$3.23
- new net OA_CLKIN: CON6.C20, U$3.1
- new net OA_GAIN: CON6.D9, U$3.25
- new net OA_HILO: CON6.D8, U$3.26
- new net OA_TRIGIN: CON6.D16, U$3.2
- net N$13: now also CON6.C1
Changed lines of the file:
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@@
 <element name="D1" library="diode" package="DO214AA" value="" x="50.8" y="26.67" rot="R180"/>
 <element name="JP1" library="pinhead" package="1X02" value="" x="7.9375" y="42.8625" rot="R90"/>
-<element name="JP2" library="pinhead" package="2X15" value="" x="25.7175" y="62.865"/>
-<element name="JP3" library="pinhead" package="2X15" value="" x="69.5325" y="62.865"/>
+<element name="U$3" library="openadc_footprint" package="OPENADCREV1" value="OPENADC" x="26.3525" y="64.77" rot="R270"/>
+<element name="U$5" library="openadc_footprint" package="OPENADCREV1" value="OPENADC" x="66.9925" y="64.77" rot="R270"/>
 </elements>
 <signals>
@@
 <contactref element="JP1" pad="2"/>
 <wire x1="7.9375" y1="44.1325" x2="7.9375" y2="51.435" width="1.27" layer="1"/>
+<contactref element="CON6" pad="C1"/>
+<wire x1="7.9375" y1="51.435" x2="7.9375" y2="48.895" width="0" layer="19" extent="1-1"/>
 </signal>
 <signal name="N$15">
@@
 <wire x1="59.06" y1="19.685" x2="55.6295" y2="26.67" width="0" layer="19" extent="1-1"/>
 </signal>
+<signal name="OA_HILO">
+<contactref element="CON6" pad="D8"/>
+<contactref element="U$3" pad="26"/>
+<wire x1="13.6525" y1="62.23" x2="25.7175" y2="51.435" width="0" layer="19" extent="1-1"/>
+</signal>
+<signal name="OA_GAIN">
+<contactref element="CON6" pad="D9"/>
+<contactref element="U$3" pad="25"/>
+<wire x1="13.6525" y1="64.77" x2="28.2575" y2="51.435" width="0" layer="19" extent="1-1"/>
+</signal>
+<signal name="OA_ADC0">
+<contactref element="CON6" pad="D10"/>
+<contactref element="U$3" pad="24"/>
+<wire x1="16.1925" y1="62.23" x2="30.7975" y2="51.435" width="0" layer="19" extent="1-1"/>
+</signal>
+<signal name="OA_CLKADC">
+<contactref element="CON6" pad="F10"/>
+<contactref element="U$3" pad="23"/>
+<wire x1="16.1925" y1="64.77" x2="30.7975" y2="53.975" width="0" layer="19" extent="1-1"/>
+</signal>
+<signal name="OA_ADC2">
+<contactref element="U$3" pad="22"/>
+<contactref element="CON6" pad="D11"/>
+<wire x1="18.7325" y1="62.23" x2="33.3375" y2="51.435" width="0" layer="19" extent="1-1"/>
+</signal>
+<signal name="OA_ADC1">
+<contactref element="CON6" pad="F11"/>
+<contactref element="U$3" pad="21"/>
+<wire x1="18.7325" y1="64.77" x2="33.3375" y2="53.975" width="0" layer="19" extent="1-1"/>
+</signal>
+<signal name="OA_ADC4">
+<contactref element="U$3" pad="20"/>
+<contactref element="CON6" pad="D12"/>
+<wire x1="21.2725" y1="62.23" x2="35.8775" y2="51.435" width="0" layer="19" extent="1-1"/>
+</signal>
+<signal name="OA_ADC3">
+<contactref element="CON6" pad="F12"/>
+<contactref element="U$3" pad="19"/>
+<wire x1="21.2725" y1="64.77" x2="35.8775" y2="53.975" width="0" layer="19" extent="1-1"/>
+</signal>
+<signal name="OA_ADC6">
+<contactref element="CON6" pad="D13"/>
+<contactref element="U$3" pad="8"/>
+<wire x1="38.4175" y1="51.435" x2="36.5125" y2="62.23" width="0" layer="19" extent="1-1"/>
+</signal>
+<signal name="OA_ADC5">
+<contactref element="CON6" pad="F13"/>
+<contactref element="U$3" pad="7"/>
+<wire x1="38.4175" y1="53.975" x2="36.5125" y2="64.77" width="0" layer="19" extent="1-1"/>
+</signal>
+<signal name="OA_ADC8">
+<contactref element="CON6" pad="D14"/>
+<contactref element="U$3" pad="6"/>
+<wire x1="40.9575" y1="51.435" x2="39.0525" y2="62.23" width="0" layer="19" extent="1-1"/>
+</signal>
+<signal name="OA_ADC7">
+<contactref element="CON6" pad="F14"/>
+<contactref element="U$3" pad="5"/>
+<wire x1="40.9575" y1="53.975" x2="39.0525" y2="64.77" width="0" layer="19" extent="1-1"/>
+</signal>
+<signal name="OA_ADCOR">
+<contactref element="U$3" pad="4"/>
+<contactref element="CON6" pad="D15"/>
+<wire x1="43.4975" y1="51.435" x2="41.5925" y2="62.23" width="0" layer="19" extent="1-1"/>
+</signal>
+<signal name="OA_ADC9">
+<contactref element="CON6" pad="F15"/>
+<contactref element="U$3" pad="3"/>
+<wire x1="43.4975" y1="53.975" x2="41.5925" y2="64.77" width="0" layer="19" extent="1-1"/>
+</signal>
+<signal name="OA_TRIGIN">
+<contactref element="U$3" pad="2"/>
+<contactref element="CON6" pad="D16"/>
+<wire x1="46.0375" y1="51.435" x2="44.1325" y2="62.23" width="0" layer="19" extent="1-1"/>
+</signal>
+<signal name="OA_CLKIN">
+<contactref element="U$3" pad="1"/>
+<contactref element="CON6" pad="C20"/>
+<wire x1="56.1975" y1="48.895" x2="44.1325" y2="64.77" width="0" layer="19" extent="1-1"/>
+</signal>
+<signal name="N$32">
+<contactref element="CON6" pad="F23"/>
+<contactref element="U$5" pad="1"/>
+<wire x1="63.8175" y1="53.975" x2="84.7725" y2="64.77" width="0" layer="19" extent="1-1"/>
+</signal>
+<signal name="N$34">
+<contactref element="CON6" pad="D20"/>
+<contactref element="U$5" pad="26"/>
+<wire x1="56.1975" y1="51.435" x2="54.2925" y2="62.23" width="0" layer="19" extent="1-1"/>
+</signal>
+<signal name="N$40">
+<contactref element="U$5" pad="25"/>
+<contactref element="CON6" pad="F20"/>
+<wire x1="56.1975" y1="53.975" x2="54.2925" y2="64.77" width="0" layer="19" extent="1-1"/>
+</signal>
+<signal name="N$44">
+<contactref element="CON6" pad="C21"/>
+<contactref element="U$5" pad="24"/>
+<wire x1="58.7375" y1="48.895" x2="56.8325" y2="62.23" width="0" layer="19" extent="1-1"/>
+</signal>
+<signal name="N$45">
+<contactref element="U$5" pad="23"/>
+<contactref element="CON6" pad="D21"/>
+<wire x1="58.7375" y1="51.435" x2="56.8325" y2="64.77" width="0" layer="19" extent="1-1"/>
+</signal>
+<signal name="N$46">
+<contactref element="CON6" pad="F21"/>
+<contactref element="U$5" pad="22"/>
+<wire x1="58.7375" y1="53.975" x2="59.3725" y2="62.23" width="0" layer="19" extent="1-1"/>
+</signal>
+<signal name="N$47">
+<contactref element="U$5" pad="20"/>
+<contactref element="CON6" pad="C22"/>
+<wire x1="61.2775" y1="48.895" x2="61.9125" y2="62.23" width="0" layer="19" extent="1-1"/>
+</signal>
+<signal name="N$48">
+<contactref element="CON6" pad="D22"/>
+<contactref element="U$5" pad="19"/>
+<wire x1="61.2775" y1="51.435" x2="61.9125" y2="64.77" width="0" layer="19" extent="1-1"/>
+</signal>
+<signal name="N$49">
+<contactref element="U$5" pad="8"/>
+<contactref element="CON6" pad="F22"/>
+<wire x1="61.2775" y1="53.975" x2="77.1525" y2="62.23" width="0" layer="19" extent="1-1"/>
+</signal>
+<signal name="N$35">
+<contactref element="CON6" pad="C24"/>
+<contactref element="U$5" pad="7"/>
+<wire x1="66.3575" y1="48.895" x2="77.1525" y2="64.77" width="0" layer="19" extent="1-1"/>
+</signal>
+<signal name="N$50">
+<contactref element="U$5" pad="6"/>
+<contactref element="CON6" pad="D24"/>
+<wire x1="66.3575" y1="51.435" x2="79.6925" y2="62.23" width="0" layer="19" extent="1-1"/>
+</signal>
+<signal name="N$51">
+<contactref element="CON6" pad="F24"/>
+<contactref element="U$5" pad="5"/>
+<wire x1="66.3575" y1="53.975" x2="79.6925" y2="64.77" width="0" layer="19" extent="1-1"/>
+</signal>
+<signal name="N$52">
+<contactref element="CON6" pad="C25"/>
+<contactref element="U$5" pad="4"/>
+<wire x1="68.8975" y1="48.895" x2="82.2325" y2="62.23" width="0" layer="19" extent="1-1"/>
+</signal>
+<signal name="N$53">
+<contactref element="U$5" pad="3"/>
+<contactref element="CON6" pad="D25"/>
+<wire x1="68.8975" y1="51.435" x2="82.2325" y2="64.77" width="0" layer="19" extent="1-1"/>
+</signal>
+<signal name="N$54">
+<contactref element="CON6" pad="F25"/>
+<contactref element="U$5" pad="2"/>
+<wire x1="68.8975" y1="53.975" x2="84.7725" y2="62.23" width="0" layer="19" extent="1-1"/>
+</signal>
 </signals>

Commit message: More progress on ztex-pro board
Parts:
- removed CON1: DC_SOCKET5870, mystuff:PWR-5870
- removed CON2: PWRCON, usb-fpga-1:PWRCON
- added C12, C15, C46: 100nF, rcl:C0603K
- added C16, C17, C19, C21, C22, C24, C26, C28, C32, C36, C38, C39, C40, C42, C45, C50, C55, C57: 100nF, rcl:C0402
- added C18, C20, C25, C27, C54, C56: 1nF, rcl:C0402
- added C23: 18nF, rcl:C0603
- added C29, C31, C35: 10nF, rcl:C0402
- added C30: 10nF, COG, rcl:C0402
- added C33, C34: 1u, rcl:C0603
- added C37, C41: 10u, rcl:C0603
- added C43, C44: (no value), rcl:C0402
- added C47, C48, C49, C66, C67, C68, C69, C70, C71, C72, C73, C76, C77, C78, C79, C80: (no value), rcl:C0603
- added C51, C52: 1uF, rcl:C0603
- added C53: (no value), rcl:C0603K
- added C58, C60, C74, C75: (no value), resistor:C0603
- added C59: 1u, rcl:C0402
- added C61: 22pF, rcl:C0603
- added C62: (no value), adc_microboard:C0603
- added C63: 22µ, myrcl:C0805K
- added C64: 10µ, myrcl:C1206
- added C65: 2n2, myrcl:C0805K
- added D3, D4: BAV99-7-F, zetex:SOT-23
- added DC1: (no value), dc-dc-converter:NMA
- added H1: MOUNT-PAD-ROUND2.8, holes:2,8-PAD
- added IC4: AOZ1021, mystuff:AOZ1021
- added IC5: AT90USB162A, adafruit:TQFP32-08
- added IC6: (no value), v-reg:337L
- added IC7: (no value), v-reg:317L
- added JP13: TARGET, pinhead:2X10/90
- added JP14, JP2: EXP-MINI, pinhead:2X03/90
- added JP3: (no value), SparkFun:SJ_2S
- added JP4: JUMPER-3PTH, SparkFun:1X03
- added JP5: (no value), pinhead:2X20/90
- added JP6: (no value), pinhead:1X02
- added JP9: PLL_INPUT, pinhead:2X04/90
- added L10: 4.7µ, myrcl:NR60
- added L2, L5, L6, L7: 120nH, SparkFun:0603
- added L8: (no value), SparkFun:0603
- added LED1, LED2, LED3, LED4, LED5, LED6: (no value), dp_devices:LED-3MM
- added R13, R14: 33R, 0.5%, adafruit:R0603
- added R15, R16: 33R, adafruit:R0603
- added R17, R18, R19, R20, R23: 1K, adafruit:R0402
- added R21: 10K, adafruit:R0603
- added R22: 274R, adafruit:R0603
- added R24: 2K, adafruit:R0603
- added R25: (no value), adafruit:R0603
- added R26: 20k, customs:3361P
- added R27, R28: 2k2, adafruit:R0603
- added R29, R30: 36R, 0.5%, adafruit:R0603
- added R31, R34, R47: (no value), adafruit:R0805
- added R32, R33, R39, R40, R41, R42, R43, R44, R45, R46, R48, R49, R50, R51, R52, R53, R54, R55, R56, R57, R58: (no value), resistor:R0603
- added R35, R36: ?, myrcl:R0805K
- added R37, R38: 7K5, myrcl:R0805K
- added SJ1, SJ2: (no value), jumper:SJ
- added T1: TC1-1T, customs:AT224-1A
- added TP1, TP2: TPSQPAD1-13, testpad:P1-13
- added U1: AD9215BRUZ, customs:TSSOP28
- added U2: AD8331, customs:QSOP20
- added U3: LP3985IM5-3.0, SparkFun:SOT23-5
- added U5: CDCE906PW, Texas Instruments_By_element14_Batch_1:SOP65P640X120-20N
- added U6: TXB0104PWR, Texas Instruments_By_element14_Batch_1:SOP65P640X120-14N
- added U7: TXB0108PWR, Texas Instruments_By_element14_Batch_1:SOP65P640X120-20N
- added U8, U9: SN74LVC1T45DBVT, Texas Instruments_By_element14_Batch_1:SOT95P280X145-6N
- added X1, X2, X3, X4: SMA-142-0711-821/826, con-coax:J502-ND-142-0711-821/826
- added X5: PN61729-S, con-berg:PN61729-S
- added XTAL1: (no value), dp_devices:HC-49U
- C13: value 220µ -> (none); device myrcl:153CLV-0810 -> rcl:C0603
- moved CON6 104.8 mm to (53.7, 98.1), turned to 270 degrees
- moved JP1 98.7 mm to (91.4, 95.6), turned to 0 degrees
- moved C2 93.6 mm to (91.8, 91.8), turned to 270 degrees
- moved C3 93.4 mm to (87.9, 92.4), turned to 180 degrees
- moved C6 91.9 mm to (72.7, 92.4), turned to 180 degrees
- moved C5 90.9 mm to (76.5, 91.8), turned to 270 degrees
- moved L4 89.3 mm to (66.4, 89.9), turned to 90 degrees
- moved L1 88.6 mm to (81.6, 89.9), turned to 90 degrees
- moved R2 87.9 mm to (90.5, 87.9), turned to 180 degrees
- moved U$3 87.9 mm to (113.3, 77.2), turned to 180 degrees
- moved R1 87.7 mm to (86.7, 88.6), turned to 90 degrees
- moved R5 86.7 mm to (71.4, 88.6), turned to 90 degrees
- moved R6 85.5 mm to (75.2, 87.9), turned to 180 degrees
- moved R3 82.7 mm to (90.5, 84.1), turned to 90 degrees
- moved R7 80.2 mm to (75.2, 84.1), turned to 90 degrees
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Connections:
- new net +5V: C63.2, DC1.1, JP13.1, JP13.20, JP9.1, JP9.8, L10.P$2, L2.1, L6.1, R35.2
- new net +5V/2: C66.1, C78.1, C79.1, C80.1, IC5.31, IC5.32, IC5.4, JP6.1, R58.1, U7.19, X5.1
- new net +9V: C58.1, IC7.2, JP14.1, JP2.1, R48.2, TP1.TP
- new net -9V: C60.1, IC6.OUT, JP14.5, JP2.5, R50.2, TP2.TP
- new net ADC_VCC: C31.1, C32.1, C34.1, C35.1, C36.1, R17.2, R19.1, R24.2, U1.12, U1.7, U3.5
- new net AGND: C45.2, C62.2, D3.3
- new net CLK_PLL0: CON6.D23, U5.11
- new net CLK_PLL1: CON6.C23, U5.12
- new net DGND: X3.G@1, X3.G@2, X3.G@3, X3.G@4
- new net HS1: CON6.E14, U8.3
- new net HS1DIR: CON6.A15, U8.5
- new net HS2: CON6.A14, U9.3
- new net HS2DIR: CON6.B14, U9.5
- new net LED1: CON6.F16, LED1.A
- new net LED2: CON6.D17, LED2.A
- new net LED3: CON6.F17, LED3.A
- new net LED4: CON6.F18, LED4.A
- new net LED5: CON6.D19, LED5.A
- new net LED6: CON6.F19, LED6.A
- new net N$100: JP13.6, U9.4
- new net N$101: JP13.4, U8.4
- new net N$102: IC5.29, R40.2
- new net N$103: R40.1, X5.3
- new net N$104: R39.1, X5.2
- new net N$105: IC5.9, R42.1
- new net N$106: C73.1, IC5.27
- new net N$107: IC5.8, R41.1
- new net N$108: IC6.ADJ, R50.1, R51.2
- new net N$109: IC7.1, R48.1, R49.2
- new net N$11: C12.1, U2.15
- new net N$110: LED1.K, R52.1
- new net N$111: LED2.K, R53.1
- new net N$112: LED3.K, R54.1
- new net N$113: LED4.K, R55.1
- new net N$114: LED5.K, R56.1
- new net N$115: LED6.K, R57.1
- new net N$116: C76.1, IC5.1, XTAL1.2
- new net N$117: C77.1, IC5.2, XTAL1.1
- new net N$118: JP9.3, R33.1, X3.1
- new net N$12: C17.2, U2.5
- new net N$122: IC5.13, SJ1.1
- new net N$123: IC5.24, R58.2, SJ2.1
- new net N$16: C17.1, U2.7
- new net N$18: C16.2, U2.8
- new net N$19: C16.1, R22.2, U2.4
- new net N$21: C18.1, C19.1, U2.11
- new net N$22: C20.1, C21.1, R21.1, U2.12
- new net N$27: C22.2, U2.1
- new net N$28: C23.1, C46.1, C61.1, U2.2
- new net N$29: C23.2, JP3.1
- new net N$30: JP3.2, R22.1
- new net N$31: C26.1, C27.1, L6.2, U2.14
- new net N$55: C30.2, U3.4
- new net N$56: C33.1, L5.2, U3.1, U3.3
- new net N$57: C37.1, C38.1, C39.2, U1.5
- new net N$58: C37.2, C38.2, C40.2, U1.6
- new net N$59: C41.2, C42.2, R26.3, U1.4
- new net N$6: C44.1, R13.1, R15.2, R19.2, R20.2, U1.9
- new net N$60: C45.1, JP4.2, U1.3
- new net N$61: R23.1, R24.1, U1.2
- new net N$62: C43.1, R14.1, R16.2, R17.1, R18.1, U1.10
- new net N$63: JP4.1, R26.2
- new net N$64: L7.1, X2.1
- new net N$65: JP9.5, R32.1
- new net N$67: C51.1, R27.2, R28.1
- new net N$68: C52.1, D4.3, R28.2, U2.10
- new net N$69: C24.1, C25.1, C50.1, C59.2, L2.2, U2.18, U2.19, U2.3
- new net N$7: C12.2, R15.1
- new net N$70: R14.2, R30.1, T1.3
- new net N$71: C53.2, X1.1
- new net N$72: C53.1, L8.1
- new net N$73: L8.2, T1.6
- new net N$75: R13.2, R29.2, T1.1
- new net N$76: C54.1, C55.1, C56.2, C57.2, R29.1, R30.2, T1.2
- new net N$77: R33.2, R43.1, R45.2, U5.6
- new net N$78: C46.2, L7.2
- new net N$79: IC4.LX, L10.P$1
- new net N$8: C15.2, R16.1
- new net N$80: R31.1, R34.2, X4.1
- new net N$81: R32.2, R44.1, R46.2, U5.5
- new net N$82: C74.1, DC1.6, IC7.3
- new net N$83: IC4.FB, R35.1, R36.2
- new net N$84: IC4.EN, R37.1
- new net N$85: C65.2, R38.1
- new net N$86: IC4.COMP, R38.2
- new net N$87: JP13.5, U7.7
- new net N$88: IC5.30, R39.2
- new net N$89: JP13.16, U6.10
- new net N$9: C15.1, U2.16
- new net N$90: JP13.14, U6.11
- new net N$91: JP13.12, U6.12
- new net N$92: JP13.10, U6.13
- new net N$93: C68.1, C69.1, C70.1, C71.1, C72.1, JP13.8, U6.14, U7.2, U8.6, U9.6
- new net N$94: JP13.7, U7.6
- new net N$95: JP13.9, U7.5
- new net N$96: JP13.11, U7.4
- new net N$97: JP13.13, U7.3
- new net N$98: JP13.15, U7.1
- new net N$99: C75.2, DC1.4, IC6.IN
- new net PRG_MISO: IC5.17, U7.15
- new net PRG_MOSI: IC5.16, U7.16
- new net PRG_PDIC: IC5.11, U7.18
- new net PRG_PDID: R41.2, R42.2, U7.20
- new net PRG_RST: IC5.18, U7.14
- new net PRG_SCK: IC5.15, U7.17
- new net TARGET1: CON6.E13, U6.2
- new net TARGET2: CON6.A13, U6.3
- new net TARGET3: CON6.B12, U6.4
- new net TARGET4: CON6.A12, U6.5
- new net VCCIO: U6.1, U8.1, U9.1
- net +3V3: now also C13.1, C28.1, C29.1, C47.1, C48.1, C49.1, C62.1, C67.1, D3.2, JP13.18, JP13.3, JP14.4, JP2.4, JP9.2, JP9.7, L5.1, R43.2, R44.2, U$3.11, U$3.12, U$3.29, U$3.30, U$5.11, U$5.12, U$5.29, U$5.30, U1.24, U5.14, U5.18, U5.3, U5.7
- net GND: now also C13.2, C18.2, C19.2, C20.2, C21.2, C22.1, C24.2, C25.2, C26.2, C27.2, C28.2, C29.2, C30.1, C31.2, C32.2, C33.2, C34.2, C35.2, C36.2, C39.1, C40.1, C41.1, C42.1, C43.2, C44.2, C47.2, C48.2, C49.2, C50.2, C51.2, C52.2, C54.2, C55.2, C56.1, C57.1, C58.2, C59.1, C60.2, C61.2, C63.1, C64.1, C65.1, C66.2, C67.2, C68.2, C69.2, C70.2, C71.2, C72.2, C73.2, C74.2, C75.1, C76.2, C77.2, C78.2, C79.2, C80.2, D4.2, DC1.2, DC1.5, IC4.AGND, IC4.PGND, IC5.28, IC5.3, JP13.17, JP13.19, JP13.2, JP14.2, JP14.6, JP2.2, JP2.6, JP4.3, JP9.4, JP9.6, R18.2, R20.1, R21.2, R23.2, R25.1, R26.1, R34.1, R36.1, R45.1, R46.1, R47.1, R49.1, R51.1, R52.2, R53.2, R54.2, R55.2, R56.2, R57.2, SJ1.2, SJ2.2, T1.4, U$3.10, U$3.27, U$3.28, U$3.9, U$5.10, U$5.27, U$5.28, U$5.9, U1.11, U1.14, U1.23, U1.8, U2.17, U2.20, U2.6, U2.9, U3.2, U5.13, U5.17, U5.4, U5.8, U6.7, U7.11, U7.8, U7.9, U8.2, U9.2, X1.G@1, X1.G@2, X1.G@3, X1.G@4, X2.G@1, X2.G@2, X2.G@3, X2.G@4, X4.G@1, X4.G@2, X4.G@3, X4.G@4, X5.4, X5.S1, X5.S2; no longer C13.-, CON1.3, CON2.-
- net OA_ADC0: now also U1.17
- net OA_ADC1: now also U1.18
- net OA_ADC2: now also U1.19
- net OA_ADC3: now also U1.20
- net OA_ADC4: now also U1.21
- net OA_ADC5: now also U1.22
- net OA_ADC6: now also U1.25
- net OA_ADC7: now also U1.26
- net OA_ADC8: now also U1.27
- net OA_ADC9: now also U1.28
- net OA_ADCOR: now also U1.1
- net OA_CLKADC: now also R25.2, U1.13
- net OA_CLKIN: now also D3.1, R31.2, R47.2
- net OA_GAIN: now also R27.1
- net OA_HILO: now also U2.13
- net VIN: now also C64.2, IC4.VIN, JP6.2, R37.2; no longer C13.+, CON1.1, CON2.+
Routing:
- net +5V: track 0.00 -> 358.7 mm, vias 0 -> 1
- net +3V3: track 261.6 -> 541.4 mm, vias 4 -> 6
- net GND: track 138.6 -> 261.1 mm, vias 62 -> 148
- net N$93: track 0.00 -> 58.8 mm, vias 0 -> 3
- net HS2DIR: track 0.00 -> 55.6 mm, vias 0 -> 1
- net TARGET3: track 0.00 -> 54.5 mm
- net +5V/2: track 0.00 -> 54.4 mm
- net HS2: track 0.00 -> 53.0 mm, vias 0 -> 1
- net OA_CLKIN: track 0.00 -> 52.8 mm
- net TARGET4: track 0.00 -> 52.8 mm
- net TARGET2: track 0.00 -> 52.6 mm
- net OA_HILO: track 0.00 -> 50.2 mm
- net TARGET1: track 0.00 -> 49.8 mm
- net LED6: track 0.00 -> 48.9 mm
- net HS1: track 0.00 -> 48.2 mm, vias 0 -> 1
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- added copper zone on layer 16, net N$74
Other:
- board size 83.8 x 48.3 mm -> 155 x 100.3 mm
- board text added: "1"
- board text added: "AD8331"
- board text added: "AD9215"
- board text added: "ADC Fullscale"
- board text added: "ADJ"
- board text added: "FIX"
- board text added: "GND"
- board text added: "JP3"
- board text added: "POS"
- board text added: "TC1-1T"
- board text added: "TRIG"

Commit message: Finished ZTEX Board
Parts:
- added C81, C82, C83: (no value), rcl:C0603
- moved C67 126.0 mm to (130.8, 28.4), turned to 0 degrees
- moved C66 9.89 mm to (25.4, 86.1), turned to 90 degrees
- moved C69 1.02 mm to (22.8, 71.2)
- moved R39 0.51 mm to (26.7, 63.0)
- moved C71 0.25 mm to (9.65, 80.5)
Connections:
- removed net AGND: C45.2, C62.2, D3.3
- removed net DGND: X3.G@1, X3.G@2, X3.G@3, X3.G@4
- removed net VCCIO: U6.1, U8.1, U9.1
- new net N$119: CON6.B17, JP5.36
- new net N$120: CON6.E17, JP5.33
- new net N$121: CON6.A18, JP5.34
- new net N$124: CON6.B18, JP5.31
- new net N$125: CON6.E18, JP5.32
- new net N$126: CON6.A19, JP5.29
- new net N$127: CON6.B19, JP5.30
- new net N$128: CON6.E19, JP5.27
- new net N$129: CON6.A20, JP5.28
- new net N$130: CON6.B20, JP5.25
- new net N$131: CON6.E20, JP5.26
- new net N$132: CON6.E21, JP5.23
- new net N$133: CON6.E22, JP5.24
- new net N$134: CON6.E23, JP5.22
- new net N$135: CON6.A24, JP5.19
- new net N$136: CON6.B24, JP5.18
- new net N$137: CON6.E24, JP5.17
- new net N$138: CON6.A25, JP5.16
- new net N$139: CON6.B25, JP5.15
- new net N$140: CON6.E25, JP5.14
- new net N$141: CON6.A26, JP5.13
- new net N$142: CON6.B26, JP5.12
- new net N$143: CON6.E26, JP5.11
- new net N$144: CON6.A27, JP5.10
- new net N$145: CON6.B27, JP5.9
- new net N$146: CON6.E27, JP5.8
- new net N$147: CON6.A28, JP5.7
- new net N$148: CON6.B28, JP5.6
- new net N$149: CON6.A29, JP5.5
- new net N$66: CON6.A17, JP5.35
- net +3V3: now also C81.1, C82.1, C83.1, JP5.3, JP5.38, U6.1, U8.1, U9.1
- net +5V: now also JP5.1, JP5.40
- net GND: now also C45.2, C62.2, C81.2, C82.2, C83.2, D3.3, JP5.2, JP5.20, JP5.21, JP5.37, JP5.39, JP5.4, X3.G@1, X3.G@2, X3.G@3, X3.G@4
Routing:
- net +3V3: track 541.4 -> 802.8 mm, vias 6 -> 11
- net +5V: track 358.7 -> 474.5 mm, vias 1 -> 4
- net +5V/2: track 54.4 -> 166.5 mm, vias 0 -> 2
- net N$148: track 0.00 -> 62.5 mm, vias 0 -> 1
- net N$142: track 0.00 -> 61.5 mm, vias 0 -> 1
- net N$127: track 0.00 -> 60.5 mm
- net N$136: track 0.00 -> 59.7 mm
- net N$119: track 0.00 -> 58.7 mm
- net N$129: track 0.00 -> 58.3 mm
- net N$144: track 0.00 -> 58.2 mm
- net N$145: track 0.00 -> 58.2 mm, vias 0 -> 1
- net N$130: track 0.00 -> 57.7 mm, vias 0 -> 1
- net N$124: track 0.00 -> 57.2 mm, vias 0 -> 1
- net N$121: track 0.00 -> 57.2 mm
- net N$139: track 0.00 -> 57.1 mm, vias 0 -> 1
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- removed copper zone on layer 16, net N$74
- removed copper zone on layer 1, net VIN
Other:
- outline, holes or cut-outs redrawn

Commit message: Round-2 ZTEX board, fix a few more errors
Parts:
- added JP7: (no value), pinhead:1X03
- added R59, R60: (no value), resistor:R0603
- flipped CON3 to the top
Connections:
- removed net N$149: CON6.A29, JP5.5
- new net PLLSCL: CON6.A29, JP7.2, R60.2, U5.10
- new net PLLSDA: CON6.B29, JP7.1, R59.2, U5.9
- net +3V3: now also R59.1, R60.1
- net GND: now also JP7.3
Routing:
- net PLLSCL: track 0.00 -> 134.8 mm, vias 0 -> 4
- net PLLSDA: track 0.00 -> 127.0 mm, vias 0 -> 4
- net N$149: track 55.7 -> 0.00 mm
- net N$24: track 23.2 -> 28.2 mm
- net N$26: track 14.3 -> 19.1 mm
- net N$23: track 15.9 -> 13.4 mm
- net +3V3: track 802.8 -> 805.3 mm, vias 11 -> 12
- net +2.6V: track 150.8 -> 148.4 mm
- net N$25: track 15.1 -> 16.5 mm, vias 2 -> 0
- net GND: track 258.2 -> 257.7 mm, vias 269 -> 281
Other:
- board text added: "1.15 ONLY"
- board text removed: "http://www.ztex.de"

Commit message: First pass of OpenADC ZTEX Ordered
Parts:
- added JP8: (no value), pinhead:1X02
- added TP3, TP4, TP5, TP6, TP7, TP8, TP9: PTR1PAD1-13, testpad:P1-13
Connections:
- net +1.2V: now also TP4.TP
- net +2.6V: now also TP5.TP
- net +3V3: now also TP6.TP, U6.8
- net +5V: now also TP3.TP
- net CLK_PLL0: now also JP8.1
- net CLK_PLL1: now also JP8.2
- net GND: now also TP7.TP, TP8.TP, TP9.TP
Routing:
- net +2.6V: track 148.4 -> 171.3 mm
- net +3V3: track 805.3 -> 818.5 mm
- net GND: track 257.7 -> 262.8 mm, vias 281 -> 284
- net +1.2V: track 125.4 -> 128.5 mm
- net +5V: track 474.5 -> 477.6 mm
- net N$1: track 0.00 -> 1.71 mm
- net CLK_PLL1: vias 1 -> 0
- net CLK_PLL0: vias 1 -> 0
Other:
- board text added: "2.5V"
- board text added: "3.3V"
- board text added: "5.0V"
- board text added: "Colin O'Flynn"
- board text added: "REV: 3APR2013"
- board text added: "coflynn@newae.com"

Commit message: Various small other changes
Parts:
- C13, C47, C48, C49, C62, C66, C70, C72, C78, C79, C80: value (none) -> 100nF
- C67, C68, C69, C81, C82, C83: value (none) -> 22nF
- C71, C73: value (none) -> 1uF
- C76, C77: value (none) -> 22pF
- LED1: value (none) -> RED
- LED2: value (none) -> YELLOW
- LED3, LED6: value (none) -> GREEN
- LED4, LED5: value (none) -> BLUE
- R31: value (none) -> 50R
- R32, R33: value (none) -> 100R
- R35: value ? -> 52k3
- R36: value ? -> 10k
- R39, R40: value (none) -> 27R
- R41: value (none) -> 470R
- R52, R53, R54, R55, R56, R57: value (none) -> 220R
- R58: value (none) -> 1K
- R59, R60: value (none) -> 4k7
- R7: value 5K4 -> 5K36
- XTAL1: value (none) -> 16MHz
