File: hardware/targets/ztex/pcb/ztex_openadc_eagle/openadc_ztex.brd (EAGLE design)
At the start: 155 x 100.3 mm, 211 parts, among them CON3 JTAG, CON6 USB-FPGA1.15, IC1 AOZ1021, IC2 AOZ1021, IC3 AOZ1094, IC4 AOZ1021, IC5 AT90USB162A, T1 TC1-1T, U1 AD9215BRUZ, U2 AD8331, U3 LP3985IM5-3.0, U5 CDCE906PW, U6 TXB0104PWR, U7 TXB0108PWR, U8 SN74LVC1T45DBVT, U9 SN74LVC1T45DBVT, X1 SMA-142-0711-821/826, X2 SMA-142-0711-821/826, X3 SMA-142-0711-821/826, X4 SMA-142-0711-821/826, X5 PN61729-S

Commit message: Fixes to ZTEX PCB. Still need to fix physical issues with placement of ZTEX board
Parts:
- added R61: 470R, resistor:M0805
Connections:
- net +5V/2: now also R61.2
- net N$93: now also U7.10
- net PRG_RST: now also R61.1
Changed lines of the file:
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@@
 <attribute name="TP_SIGNAL_NAME" value="" x="41.402" y="86.36" size="1.016" layer="27" font="vector" ratio="16" display="off"/>
 </element>
+<element name="R61" library="resistor" package="M0805" value="470R" x="-5.334" y="-51.562"/>
 </elements>
 <signals>
@@
 <wire x1="22.606" y1="70.14" x2="21.5794" y2="70.14" width="0.508" layer="1"/>
 <wire x1="21.5794" y1="70.14" x2="21.2598" y2="70.4596" width="0.508" layer="1"/>
+<contactref element="U7" pad="10"/>
+<wire x1="18.034" y1="74.676" x2="17.399" y2="79.629" width="0" layer="19" extent="1-1"/>
 </signal>
 <signal name="N$89">
@@
 <wire x1="2.794" y1="97.282" x2="43.18" y2="97.282" width="1.524" layer="1"/>
 <wire x1="43.18" y1="97.282" x2="44.958" y2="95.504" width="1.524" layer="1"/>
+<contactref element="R61" pad="2"/>
+<wire x1="-4.384" y1="-51.562" x2="12.192" y2="57.404" width="0" layer="19" extent="1-1"/>
 </signal>
 <signal name="N$88">
@@
 <wire x1="26.67" y1="76.835" x2="27.3624" y2="76.835" width="0.3" layer="1"/>
 <wire x1="27.3624" y1="76.835" x2="27.4574" y2="76.93" width="0.3" layer="1"/>
+<contactref element="R61" pad="1"/>
+<wire x1="-6.284" y1="-51.562" x2="26.67" y2="76.835" width="0" layer="19" extent="1-1"/>
 </signal>
 <signal name="PRG_PDIC">

Commit message: Fixes in PCB.. still more to go
Parts:
- removed C65: 2n2, myrcl:C0805K
- removed IC4: AOZ1021, mystuff:AOZ1021
- removed L10: 4.7µ, myrcl:NR60
- removed R35: 52k3, myrcl:R0805K
- removed R36: 10k, myrcl:R0805K
- removed R37, R38: 7K5, myrcl:R0805K
- JP5: device pinhead:2X20/90 -> pinhead:2X15/90
- moved R61 115.2 mm to (26.4, 59.2)
- moved C64 52.6 mm to (18.8, 50.3), turned to 270 degrees
- moved C63 52.2 mm to (122.2, 13.2), turned to 270 degrees
- moved JP6 47.4 mm to (24.6, 53.3), turned to 270 degrees
- moved X5 5.05 mm to (9.91, 55.9)
- moved JP13 3.79 mm to (2.79, 80.5)
- moved C71 3.64 mm to (13.0, 79.0), flipped to the bottom, turned to 90 degrees
- moved JP5 3.45 mm to (2.79, 25.9)
- moved CON6 2.79 mm to (53.7, 95.3)
Connections:
- removed net N$119: CON6.B17, JP5.36
- removed net N$120: CON6.E17, JP5.33
- removed net N$121: CON6.A18, JP5.34
- removed net N$124: CON6.B18, JP5.31
- removed net N$125: CON6.E18, JP5.32
- removed net N$126: CON6.A19, JP5.29
- removed net N$127: CON6.B19, JP5.30
- removed net N$128: CON6.E19, JP5.27
- removed net N$129: CON6.A20, JP5.28
- removed net N$130: CON6.B20, JP5.25
- removed net N$131: CON6.E20, JP5.26
- removed net N$132: CON6.E21, JP5.23
- removed net N$133: CON6.E22, JP5.24
- removed net N$134: CON6.E23, JP5.22
- removed net N$135: CON6.A24, JP5.19
- removed net N$136: CON6.B24, JP5.18
- removed net N$137: CON6.E24, JP5.17
- removed net N$138: CON6.A25, JP5.16
- removed net N$139: CON6.B25, JP5.15
- removed net N$140: CON6.E25, JP5.14
- removed net N$141: CON6.A26, JP5.13
- removed net N$142: CON6.B26, JP5.12
- removed net N$143: CON6.E26, JP5.11
- removed net N$144: CON6.A27, JP5.10
- removed net N$145: CON6.B27, JP5.9
- removed net N$146: CON6.E27, JP5.8
- removed net N$147: CON6.A28, JP5.7
- removed net N$148: CON6.B28, JP5.6
- removed net N$66: CON6.A17, JP5.35
- removed net N$79: IC4.LX, L10.P$1
- removed net N$83: IC4.FB, R35.1, R36.2
- removed net N$84: IC4.EN, R37.1
- removed net N$85: C65.2, R38.1
- removed net N$86: IC4.COMP, R38.2
- new net EXPIO10: CON6.E25, JP5.10
- new net EXPIO11: CON6.A24, JP5.11
- new net EXPIO12: CON6.B24, JP5.12
- new net EXPIO13: CON6.E24, JP5.13
- new net EXPIO14: CON6.E23, JP5.14
- new net EXPIO15: CON6.E22, JP5.15
- new net EXPIO16: CON6.E21, JP5.16
- new net EXPIO17: CON6.E20, JP5.17
- new net EXPIO18: CON6.B20, JP5.18
- new net EXPIO19: CON6.A20, JP5.19
- new net EXPIO20: CON6.E19, JP5.20
- new net EXPIO21: CON6.B19, JP5.21
- new net EXPIO22: CON6.A19, JP5.22
- new net EXPIO23: CON6.A18, JP5.23
- new net EXPIO24: CON6.B18, JP5.24
- new net EXPIO25: CON6.E18, JP5.25
- new net EXPIO26: CON6.B17, JP5.26
- new net EXPIO27: CON6.A17, JP5.27
- new net EXPIO28: CON6.E17, JP5.28
- new net EXPIO5: CON6.A27, JP5.5
- new net EXPIO6: CON6.B26, JP5.6
- new net EXPIO7: CON6.A26, JP5.7
- new net EXPIO8: CON6.A25, JP5.8
- new net EXPIO9: CON6.B25, JP5.9
- net +3V3: no longer JP5.38
- net +5V: now also C1.2, C4.2, C64.2, C7.2, C8.2, IC1.VIN, IC2.VIN, IC3.VIN, JP6.2, R1.2, R12.2, R5.2; no longer JP5.40, L10.P$2, R35.2
- net GND: now also JP5.29, JP5.30; no longer C65.1, IC4.AGND, IC4.PGND, JP5.20, JP5.21, JP5.37, JP5.39, R36.1
- net VIN: no longer C1.2, C4.2, C64.2, C7.2, C8.2, IC1.VIN, IC2.VIN, IC3.VIN, IC4.VIN, JP6.2, R1.2, R12.2, R37.2, R5.2
Routing:
- net VIN: track 236.4 -> 0.00 mm
- net +5V/2: track 166.5 -> 76.4 mm
- net +5V: track 477.6 -> 540.4 mm, vias 4 -> 1
- net N$148: track 62.5 -> 0.00 mm, vias 1 -> 0
- net N$142: track 61.5 -> 0.00 mm, vias 1 -> 0
- net N$127: track 60.5 -> 0.00 mm
- net N$136: track 59.7 -> 0.00 mm
- net EXPIO6: track 0.00 -> 59.4 mm, vias 0 -> 1
- net N$119: track 58.7 -> 0.00 mm
- net EXPIO18: track 0.00 -> 58.7 mm
- net EXPIO26: track 0.00 -> 58.4 mm, vias 0 -> 1
- net N$129: track 58.3 -> 0.00 mm
- net N$144: track 58.2 -> 0.00 mm
- net N$145: track 58.2 -> 0.00 mm, vias 1 -> 0
- net N$130: track 57.7 -> 0.00 mm, vias 1 -> 0
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
Commit message: Bring back 3.3-5v converter
Parts:
- added C65: 100nF, rcl:C0603
- added C84, C85, C86, C87: 1u, rcl:C0603
- added L9: 120nH, SparkFun:0603
- added U4: LTC3200ES6, customs:SOT23-6L
- R61: device resistor:M0805 -> resistor:R0603
- moved R61 23.1 mm to (25.4, 82.3), flipped to the bottom, turned to 90 degrees
Connections:
- new net N$74: C85.1, U4.4
- new net N$79: C85.2, U4.6
- new net N$85: C86.2, L9.1, U4.3, U4.5
- new net N$86: C84.1, C87.2, L2.1, L6.1, U4.1
- net +3V3: now also C65.1, L9.2
- net +5V: no longer L2.1, L6.1
- net GND: now also C65.2, C84.2, C86.1, C87.1, U4.2
Routing:
- net VIN: track 0.00 -> 37.9 mm
- net GND: track 258.5 -> 288.2 mm, vias 273 -> 293
- net N$85: track 0.00 -> 7.05 mm
- net N$86: track 0.00 -> 5.85 mm
- net +3V3: track 780.3 -> 784.8 mm
- net +5V: track 540.4 -> 537.7 mm, vias 1 -> 0
- net PRG_RST: track 8.08 -> 10.8 mm, vias 0 -> 1
- net +5V/2: track 76.4 -> 78.6 mm
- net N$79: track 0.00 -> 1.79 mm
- net N$74: track 0.00 -> 1.79 mm
- net N$89: track 14.3 -> 14.9 mm
Other:
- board text added: "REV: 6JUNE2013"
- board text removed: "REV: 3APR2013"

Commit message: Fix other spacing issues - done?
Parts:
- removed JP14: EXP-MINI, pinhead:2X03/90
- moved JP2 5.59 mm to (154.9, 12.4)
- moved JP9 2.79 mm to (154.9, 27.4)
Connections:
- net +3V3: no longer JP14.4
- net +9V: no longer JP14.1
- net -9V: no longer JP14.5
- net GND: no longer JP14.2, JP14.6
Routing:
- net -9V: track 37.1 -> 27.3 mm
- net +9V: track 20.4 -> 11.6 mm
- net +3V3: track 784.8 -> 779.7 mm
- net N$118: track 21.5 -> 23.8 mm
- net N$65: track 6.21 -> 8.31 mm
- net +5V: track 537.7 -> 539.6 mm
- net +2.6V: track 168.6 -> 167.0 mm
- net GND: vias 293 -> 292

Commit message: Updating HW Design Files
Parts:
- C14: value 560µ -> 470u
- C58, C60, C74, C75: value (none) -> 100nF
- R42: value (none) -> 470
- R43, R44, R45, R46, R49, R51: value (none) -> 1k,1%
- R48, R50: value (none) -> 200R,1%
- R9: value 25K -> 24k9,1%
Changed lines of the file:
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@@
 <layer number="23" name="tOrigins" color="15" fill="1" visible="no" active="yes"/>
 <layer number="24" name="bOrigins" color="15" fill="1" visible="no" active="yes"/>
-<layer number="25" name="tNames" color="7" fill="1" visible="no" active="yes"/>
+<layer number="25" name="tNames" color="7" fill="1" visible="yes" active="yes"/>
 <layer number="26" name="bNames" color="7" fill="1" visible="no" active="yes"/>
 <layer number="27" name="tValues" color="7" fill="1" visible="no" active="yes"/>
@@
 </element>
 <element name="C2" library="myrcl" package="C0805K" value="2n2" x="91.7575" y="91.7575" smashed="yes" rot="R270">
-<attribute name="NAME" x="93.232" y="93.8055" size="1.0668" layer="25" ratio="12" rot="R90"/>
+<attribute name="NAME" x="93.994" y="90.7575" size="1.0668" layer="25" ratio="12" rot="R90"/>
 <attribute name="VALUE" x="90.7465" y="96.631" size="1.0668" layer="27" ratio="12" rot="R270"/>
 </element>
@@
 <attribute name="VALUE" x="85.7835" y="41.418" size="1.0668" layer="27" ratio="12" rot="R90"/>
 </element>
-<element name="R9" library="myrcl" package="R0805K" value="25K" x="81.28" y="48.5775" smashed="yes" rot="R180">
+<element name="R9" library="myrcl" package="R0805K" value="24k9,1%" x="81.28" y="48.5775" smashed="yes" rot="R180">
 <attribute name="NAME" x="79.9625" y="49.8335" size="1.0668" layer="25" ratio="12"/>
 <attribute name="VALUE" x="79.899" y="51.186" size="1.0668" layer="27" ratio="12"/>
@@
 <attribute name="VALUE" x="74.9935" y="34.4805" size="1.0668" layer="27" ratio="12" rot="R270"/>
 </element>
-<element name="C14" library="myrcl" package="E2,5-6" value="560µ" x="67.945" y="58.1025" smashed="yes" rot="R90">
+<element name="C14" library="myrcl" package="E2,5-6" value="470u" x="67.945" y="58.1025" smashed="yes" rot="R90">
 <attribute name="NAME" x="66.5735" y="61.722" size="1.0668" layer="25" ratio="12" rot="R90"/>
 <attribute name="VALUE" x="64.5795" y="56.642" size="1.0668" layer="27" ratio="12" rot="R90"/>
@@
 <attribute name="VALUE" x="41.402" y="79.756" size="1.27" layer="27" rot="R90"/>
 </element>
-<element name="R42" library="resistor" package="R0603" value="" x="37.465" y="80.645" smashed="yes" rot="R90">
+<element name="R42" library="resistor" package="R0603" value="470" x="37.465" y="80.645" smashed="yes" rot="R90">
 <attribute name="NAME" x="37.846" y="82.55" size="1.016" layer="25" font="vector" ratio="16" rot="R90"/>
 <attribute name="VALUE" x="39.497" y="79.756" size="1.27" layer="27" rot="R90"/>
@@
 <attribute name="VALUE" x="143.891" y="36.322" size="1.27" layer="27" rot="R180"/>
 </element>
-<element name="R43" library="resistor" package="R0603" value="" x="137.16" y="35.306" smashed="yes" rot="R90">
+<element name="R43" library="resistor" package="R0603" value="1k,1%" x="137.16" y="35.306" smashed="yes" rot="R90">
 <attribute name="NAME" x="137.541" y="36.957" size="1.016" layer="25" font="vector" ratio="16" rot="R90"/>
 <attribute name="VALUE" x="139.192" y="34.417" size="1.27" layer="27" rot="R90"/>
 </element>
-<element name="R44" library="resistor" package="R0603" value="" x="137.16" y="31.496" smashed="yes" rot="R270">
+<element name="R44" library="resistor" package="R0603" value="1k,1%" x="137.16" y="31.496" smashed="yes" rot="R270">
 <attribute name="NAME" x="136.779" y="30.099" size="1.016" layer="25" font="vector" ratio="16" rot="R270"/>
 <attribute name="VALUE" x="135.128" y="32.385" size="1.27" layer="27" rot="R270"/>
 </element>
-<element name="R45" library="resistor" package="R0603" value="" x="139.446" y="35.306" smashed="yes" rot="R270">
+<element name="R45" library="resistor" package="R0603" value="1k,1%" x="139.446" y="35.306" smashed="yes" rot="R270">
 <attribute name="NAME" x="138.811" y="40.005" size="1.016" layer="25" font="vector" ratio="16" rot="R270"/>
 <attribute name="VALUE" x="137.414" y="36.195" size="1.27" layer="27" rot="R270"/>
 </element>
-<element name="R46" library="resistor" package="R0603" value="" x="139.446" y="31.496" smashed="yes" rot="R90">
+<element name="R46" library="resistor" package="R0603" value="1k,1%" x="139.446" y="31.496" smashed="yes" rot="R90">
 <attribute name="NAME" x="140.081" y="27.305" size="1.016" layer="25" font="vector" ratio="16" rot="R90"/>
 <attribute name="VALUE" x="141.478" y="30.607" size="1.27" layer="27" rot="R90"/>
@@
 <attribute name="VALUE" x="140.462" y="14.351" size="1.27" layer="27" ratio="10" rot="R270"/>
 </element>
-<element name="R48" library="resistor" package="R0603" value="" x="142.494" y="21.082" smashed="yes">
+<element name="R48" library="resistor" package="R0603" value="200R,1%" x="142.494" y="21.082" smashed="yes">
 <attribute name="NAME" x="141.605" y="21.971" size="1.27" layer="25" font="vector"/>
 <attribute name="VALUE" x="141.605" y="19.05" size="1.27" layer="27"/>
 </element>
-<element name="R49" library="resistor" package="R0603" value="" x="138.684" y="21.082" smashed="yes">
+<element name="R49" library="resistor" package="R0603" value="1k,1%" x="138.684" y="21.082" smashed="yes">
 <attribute name="NAME" x="137.795" y="21.971" size="1.27" layer="25" font="vector"/>
 <attribute name="VALUE" x="137.795" y="19.05" size="1.27" layer="27"/>
 </element>
-<element name="R50" library="resistor" package="R0603" value="" x="134.874" y="21.082" smashed="yes">
+<element name="R50" library="resistor" package="R0603" value="200R,1%" x="134.874" y="21.082" smashed="yes">
 <attribute name="NAME" x="133.985" y="21.971" size="1.27" layer="25" font="vector"/>
 <attribute name="VALUE" x="133.985" y="19.05" size="1.27" layer="27"/>
 </element>
-<element name="R51" library="resistor" package="R0603" value="" x="131.064" y="21.082" smashed="yes">
+<element name="R51" library="resistor" package="R0603" value="1k,1%" x="131.064" y="21.082" smashed="yes">
 <attribute name="NAME" x="130.175" y="21.971" size="1.27" layer="25" font="vector"/>
 <attribute name="VALUE" x="130.175" y="19.05" size="1.27" layer="27"/>
 </element>
-<element name="C58" library="resistor" package="C0603" value="" x="145.796" y="21.082" smashed="yes" rot="R90">
+<element name="C58" library="resistor" package="C0603" value="100nF" x="145.796" y="21.082" smashed="yes" rot="R90">
 <attribute name="NAME" x="147.828" y="19.685" size="1.27" layer="25" font="vector" rot="R90"/>
 <attribute name="VALUE" x="147.828" y="20.193" size="1.27" layer="27" rot="R90"/>
 </element>
-<element name="C60" library="resistor" package="C0603" value="" x="129.286" y="18.034" smashed="yes" rot="R90">
+<element name="C60" library="resistor" package="C0603" value="100nF" x="129.286" y="18.034" smashed="yes" rot="R90">
 <attribute name="NAME" x="128.27" y="16.383" size="1.27" layer="25" font="vector" rot="R90"/>
 <attribute name="VALUE" x="131.318" y="17.145" size="1.27" layer="27" rot="R90"/>
 </element>
-<element name="C74" library="resistor" package="C0603" value="" x="139.192" y="17.272" smashed="yes" rot="R90">
+<element name="C74" library="resistor" package="C0603" value="100nF" x="139.192" y="17.272" smashed="yes" rot="R90">
 <attribute name="NAME" x="140.97" y="15.621" size="1.27" layer="25" font="vector" rot="R90"/>
 <attribute name="VALUE" x="141.224" y="16.383" size="1.27" layer="27" rot="R90"/>
 </element>
-<element name="C75" library="resistor" package="C0603" value="" x="131.572" y="14.732" smashed="yes">
+<element name="C75" library="resistor" package="C0603" value="100nF" x="131.572" y="14.732" smashed="yes">
 <attribute name="NAME" x="129.921" y="12.7" size="1.27" layer="25" font="vector"/>
 <attribute name="VALUE" x="130.683" y="12.7" size="1.27" layer="27"/>
