File: hardware/targets/ztex/pcb/ztex_openadc_eagle/openadc_ztex.sch (EAGLE design)
At the start: 35 parts, among them CON1 DC_SOCKET5870, CON2 PWRCON, CON3 JTAG, CON4 JTAG, CON6 USB-FPGA1.15, IC1 AOZ1021, IC2 AOZ1021, IC3 AOZ1094

Commit message: Update PCB
Parts:
- added C9: 22µ, myrcl:C-EUC0805K
- added D1: (no value), diode:DIODE-DO214AA
- added L3: 2.2uF, inductors:DR1030
Connections:
- removed net N$18: CON6_CDF-PWR.C18~2.5V, CON6_CDF-PWR.C29~2.5V, CON6_CDF-PWR.D18~2.5V
- removed net N$19: CON6_CDF-PWR.C19~1.2V, CON6_CDF-PWR.C28~1.2V, CON6_CDF-PWR.D28~1.2V
- removed net N$6: CON6_ABE-PWR.A22~VCCO_IO, CON6_ABE-PWR.A31~VCCO_IO, CON6_ABE-PWR.B22~VCCO_IO, CON6_ABE-PWR.B31~VCCO_IO
- new net N$5: D1.C, IC3.LX, L3.1
- net +1.2V: now also C9.2, CON6_CDF-PWR.C19~1.2V, CON6_CDF-PWR.C28~1.2V, CON6_CDF-PWR.D28~1.2V, L3.2
- net +2.6V: now also CON6_CDF-PWR.C18~2.5V, CON6_CDF-PWR.C29~2.5V, CON6_CDF-PWR.D18~2.5V
- net GND: now also C9.1, D1.A
- net VCCO_IO: now also CON6_ABE-PWR.A22~VCCO_IO, CON6_ABE-PWR.A31~VCCO_IO, CON6_ABE-PWR.B22~VCCO_IO, CON6_ABE-PWR.B31~VCCO_IO
- net VCCO_TOP: now also CON6_COMPAT.C27~VCCO_TOP, CON6_COMPAT.C7~VCCO_TOP, CON6_COMPAT.D27~VCCO_TOP, CON6_COMPAT.D7~VCCO_TOP
Other:
- moved on the sheet: CON6_COMPAT

Commit message: Update GIT repository
Parts:
- removed CON4: JTAG, usb-fpga-1:JTAG
- added JP2, JP3: (no value), pinhead:PINHD-2X15
- JP1: value EXP1.2-VJUMP -> (none); device mystuff:EXP1.2-VJUMP -> pinhead:PINHD-1X2
Connections:
- removed net N$12: CON6_ABE-PWR.A1~4..35V, CON6_ABE-PWR.B1~4..35V
- removed net N$16: CON6_CDF-PWR.C6~3.3V, CON6_CDF-PWR.D6~3.3V
- removed net N$9: CON6_ABE-PWR.E12~VREF_IO, CON6_ABE-PWR.E28~VREF_IO
- removed net VCCO_IO: CON6_ABE-PWR.A22~VCCO_IO, CON6_ABE-PWR.A31~VCCO_IO, CON6_ABE-PWR.B22~VCCO_IO, CON6_ABE-PWR.B31~VCCO_IO, JP1.V_IO
- removed net VCCO_TOP: CON6_COMPAT.C27~VCCO_TOP, CON6_COMPAT.C7~VCCO_TOP, CON6_COMPAT.D27~VCCO_TOP, CON6_COMPAT.D7~VCCO_TOP, JP1.V_TOP
- net +1.2V: no longer JP1.1V2_1, JP1.1V2_2
- net +2.6V: no longer CON4.VIO, JP1.2V5_1, JP1.2V5_2
- net +3V3: now also CON6_ABE-PWR.A22~VCCO_IO, CON6_ABE-PWR.A31~VCCO_IO, CON6_ABE-PWR.B22~VCCO_IO, CON6_ABE-PWR.B31~VCCO_IO, CON6_CDF-PWR.C6~3.3V, CON6_CDF-PWR.D6~3.3V, CON6_COMPAT.C27~VCCO_TOP, CON6_COMPAT.C7~VCCO_TOP, CON6_COMPAT.D27~VCCO_TOP, CON6_COMPAT.D7~VCCO_TOP; no longer CON4.3.3V, JP1.3V3_1, JP1.3V3_2
- net GND: no longer CON4.GND
- net N$13: now also JP1.2
- net N$23: no longer CON4.TDO
- net N$24: no longer CON4.TDI
- net N$25: no longer CON4.TCK
- net N$26: no longer CON4.TMS
- net VIN: now also CON6_ABE-PWR.A1~4..35V, CON6_ABE-PWR.B1~4..35V, JP1.1
Other:
- moved on the sheet: CON6_CDF-FPGA

Commit message: Update ZTEX
Parts:
- removed JP2, JP3: (no value), pinhead:PINHD-2X15
- added U$3, U$5: OPENADC, openadc_footprint:OPENADC
Connections:
- new net N$32: CON6_CDF-FPGA.F23~W11~IO_L29P_GCLK3_2, U$5.CLKIN
- new net N$34: CON6_CDF-FPGA.D20~W15~IO_L14P_D11_2, U$5.HILO
- new net N$35: CON6_CDF-FPGA.C24~Y13~IO_L41P_2, U$5.ADC5
- new net N$40: CON6_CDF-FPGA.F20~Y16~IO_L14N_D12_2, U$5.GAIN
- new net N$44: CON6_CDF-FPGA.C21~AA12~IO_L30P_GCLK1_D13_2, U$5.ADC0
- new net N$45: CON6_CDF-FPGA.D21~AA14~IO_L15P_2, U$5.CLKADC
- new net N$46: CON6_CDF-FPGA.F21~AB14~IO_L15N_2, U$5.ADC2
- new net N$47: CON6_CDF-FPGA.C22~Y10~IO_L29N_GCLK2_2, U$5.ADC4
- new net N$48: CON6_CDF-FPGA.D22~AB12~IO_L30N_GCLK0_USERCCLK_2, U$5.ADC3
- new net N$49: CON6_CDF-FPGA.F22~AB11~IO_L31N_GCLK30_D15_2, U$5.ADC6
- new net N$50: CON6_CDF-FPGA.D24~T14~IO_L20P_2, U$5.ADC8
- new net N$51: CON6_CDF-FPGA.F24~U14~IO_L20N_2, U$5.ADC7
- new net N$52: CON6_CDF-FPGA.C25~W9~IO_L47P_2, U$5.ADCOR
- new net N$53: CON6_CDF-FPGA.D25~W12~IO_L42P_2, U$5.ADC9
- new net N$54: CON6_CDF-FPGA.F25~Y12~IO_L42N_2, U$5.TRIGIN
- new net OA_ADC0: CON6_CDF-FPGA.D10~AA22~IO_L63N_1, U$3.ADC0
- new net OA_ADC1: CON6_CDF-FPGA.F11~AB21~IO_L61N_1, U$3.ADC1
- new net OA_ADC2: CON6_CDF-FPGA.D11~Y21~IO_L59P_1, U$3.ADC2
- new net OA_ADC3: CON6_CDF-FPGA.F12~Y20~IO_L67N_1, U$3.ADC3
- new net OA_ADC4: CON6_CDF-FPGA.D12~W20~IO_L53P_1, U$3.ADC4
- new net OA_ADC5: CON6_CDF-FPGA.F13~AB20~IO_L65N_1, U$3.ADC5
- new net OA_ADC6: CON6_CDF-FPGA.D13~AA20~IO_L61P_1, U$3.ADC6
- new net OA_ADC7: CON6_CDF-FPGA.F14~AB19~IO_L65P_1, U$3.ADC7
- new net OA_ADC8: CON6_CDF-FPGA.D14~V19~IO_L71P_1, U$3.ADC8
- new net OA_ADC9: CON6_CDF-FPGA.F15~AB18~IO_L2N_CMPMOSI_2, U$3.ADC9
- new net OA_ADCOR: CON6_CDF-FPGA.D15~Y19~IO_L67P_1, U$3.ADCOR
- new net OA_CLKADC: CON6_CDF-FPGA.F10~AA21~IO_L63P_1, U$3.CLKADC
- new net OA_CLKIN: CON6_CDF-FPGA.C20~Y11~IO_L31P_GCLK31_D14_2, U$3.CLKIN
- new net OA_GAIN: CON6_CDF-FPGA.D9~Y22~IO_L59N_1, U$3.GAIN
- new net OA_HILO: CON6_CDF-FPGA.D8~V20~IO_L71N_1, U$3.HILO
- new net OA_TRIGIN: CON6_CDF-FPGA.D16~V18~IO_L73N_1, U$3.TRIGIN
- net N$13: now also CON6_CDF-PWR.C1~USB_5V

Commit message: More progress on ztex-pro board
Parts:
- removed CON1: DC_SOCKET5870, mystuff:DC_SOCKET5870
- removed CON2: PWRCON, usb-fpga-1:PWRCON
- added C12, C15, C46: 100nF, rcl:C-EUC0603K
- added C16, C17, C19, C21, C22, C24, C26, C28, C32, C36, C38, C39, C40, C42, C45, C50, C55, C57: 100nF, rcl:C-EUC0402
- added C18, C20, C25, C27, C54, C56: 1nF, rcl:C-EUC0402
- added C23: 18nF, rcl:C-EUC0603
- added C29, C31, C35: 10nF, rcl:C-EUC0402
- added C30: 10nF, COG, rcl:C-EUC0402
- added C33, C34: 1u, rcl:C-EUC0603
- added C37, C41: 10u, rcl:C-EUC0603
- added C43, C44: (no value), rcl:C-EUC0402
- added C47, C48, C49, C66, C67, C68, C69, C70, C71, C72, C73, C76, C77, C78, C79, C80: (no value), rcl:C-EUC0603
- added C51, C52: 1uF, rcl:C-EUC0603
- added C53: (no value), rcl:C-EUC0603K
- added C58, C60, C74, C75: (no value), resistor:C-EUC0603
- added C59: 1u, rcl:C-EUC0402
- added C61: 22pF, rcl:C-EUC0603
- added C62: (no value), adc_microboard:C-EUC0603
- added C63: 22µ, myrcl:C-EUC0805K
- added C64: 10µ, myrcl:C-EUC1206
- added C65: 2n2, myrcl:C-EUC0805K
- added D3, D4: BAV99-7-F, zetex:D_ACACSOT23
- added DC1: (no value), dc-dc-converter:NMA
- added H1: MOUNT-PAD-ROUND2.8, holes:MOUNT-PAD-ROUND2.8
- added IC4: AOZ1021, mystuff:AOZ1021
- added IC5: AT90USB162A, adafruit:AT90USB162A
- added IC6: (no value), v-reg:LM337L
- added IC7: (no value), v-reg:LM317L
- added JP13: TARGET, pinhead:PINHD-2X10/90
- added JP14, JP2: EXP-MINI, pinhead:PINHD-2X3/90
- added JP3: (no value), SparkFun:JUMPER-2SMD-NC
- added JP4: JUMPER-3PTH, SparkFun:JUMPER-3PTH
- added JP5: (no value), pinhead:PINHD-2X20/90
- added JP6: (no value), pinhead:PINHD-1X2
- added JP9: PLL_INPUT, pinhead:PINHD-2X4/90
- added L10: 4.7µ, myrcl:L-EUNR60
- added L2, L5, L6, L7: 120nH, SparkFun:INDUCTOR0603
- added L8: (no value), SparkFun:INDUCTOR0603
- added LED1, LED2, LED3, LED4, LED5, LED6: (no value), dp_devices:LED-3MM
- added R13, R14: 33R, 0.5%, adafruit:R-US_R0603
- added R15, R16: 33R, adafruit:R-US_R0603
- added R17, R18, R19, R20, R23: 1K, adafruit:R-US_R0402
- added R21: 10K, adafruit:R-US_R0603
- added R22: 274R, adafruit:R-US_R0603
- added R24: 2K, adafruit:R-US_R0603
- added R25: (no value), adafruit:R-US_R0603
- added R26: 20k, customs:TRIM_US-3361P
- added R27, R28: 2k2, adafruit:R-US_R0603
- added R29, R30: 36R, 0.5%, adafruit:R-US_R0603
- added R31, R34, R47: (no value), adafruit:R-US_R0805
- added R32, R33, R39, R40, R41, R42, R43, R44, R45, R46, R48, R49, R50, R51, R52, R53, R54, R55, R56, R57, R58: (no value), resistor:R-US_R0603
- added R35, R36: ?, myrcl:R-EU_R0805K
- added R37, R38: 7K5, myrcl:R-EU_R0805K
- added SJ1, SJ2: (no value), jumper:SJ
- added T1: TC1-1T, customs:TC1-1T
- added TP1, TP2: TPSQPAD1-13, testpad:TPSQPAD1-13
- added U1: AD9215BRUZ, customs:AD9215BRUZ
- added U2: AD8331, customs:AD8331
- added U3: LP3985IM5-3.0, SparkFun:V_REG_LDOSMD
- added U5: CDCE906PW, Texas Instruments_By_element14_Batch_1:CDCE906PW
- added U6: TXB0104PWR, Texas Instruments_By_element14_Batch_1:TXB0104PWR
- added U7: TXB0108PWR, Texas Instruments_By_element14_Batch_1:TXB0108PWR
- added U8, U9: SN74LVC1T45DBVT, Texas Instruments_By_element14_Batch_1:SN74LVC1T45DBVT
- added X1, X2, X3, X4: SMA-142-0711-821/826, con-coax:SMA-142-0711-821/826
- added X5: PN61729-S, con-berg:PN61729-S
- added XTAL1: (no value), dp_devices:OSC-XTAL-HC-49U-SMD
- C13: value 220µ -> (none); device myrcl:CPOL-EU153CLV-0810 -> rcl:C-EUC0603
Connections:
- new net +5V: C63.2, DC1.+VIN, JP13.1, JP13.20, JP9.1, JP9.8, L10.2, L2.1, L6.1, R35.2
- new net +5V/2: C66.1, C78.1, C79.1, C80.1, IC5.AVCC, IC5.UVCC, IC5.VCC, JP6.1, R58.1, U7.VCCB, X5.1
- new net +9V: C58.1, IC7.OUT, JP14.1, JP2.1, R48.2, TP1.TP
- new net -9V: C60.1, IC6.OUT, JP14.5, JP2.5, R50.2, TP2.TP
- new net ADC_VCC: C31.1, C32.1, C34.1, C35.1, C36.1, R17.2, R19.1, R24.2, U1.AVDD@0, U1.AVDD@1, U3.OUT
- new net AGND: C45.2, C62.2, D3.A
- new net CLK_PLL0: CON6_CDF-FPGA.D23~AA10~IO_L32P_GCLK29_2, U5.Y0
- new net CLK_PLL1: CON6_CDF-FPGA.C23~AB10~IO_L32N_GCLK28_2, U5.Y1
- new net DGND: X3.2
- new net HS1: CON6_ABE-FPGA.E14~B16~IO_L63P_SCP7_0, U8.A
- new net HS1DIR: CON6_ABE-FPGA.A15~C14~IO_L46N_0, U8.DIR
- new net HS2: CON6_ABE-FPGA.A14~A17~IO_L64N_SCP4_0, U9.A
- new net HS2DIR: CON6_ABE-FPGA.B14~C17~IO_L64P_SCP5_0, U9.DIR
- new net LED1: CON6_CDF-FPGA.F16~AA18~IO_L2P_CMPCLK_2, LED1.A
- new net LED2: CON6_CDF-FPGA.D17~Y15~IO_L5P_2, LED2.A
- new net LED3: CON6_CDF-FPGA.F17~AA16~IO_L4P_2, LED3.A
- new net LED4: CON6_CDF-FPGA.F18~AB15~IO_L5N_2, LED4.A
- new net LED5: CON6_CDF-FPGA.D19~V15~IO_L13N_D10_2, LED5.A
- new net LED6: CON6_CDF-FPGA.F19~W14~IO_L16P_2, LED6.A
- new net N$100: JP13.6, U9.B
- new net N$101: JP13.4, U8.B
- new net N$102: IC5.D+, R40.2
- new net N$103: R40.1, X5.3
- new net N$104: R39.1, X5.2
- new net N$105: IC5.PD3(INT3/TXD1), R42.1
- new net N$106: C73.1, IC5.UCAP
- new net N$107: IC5.PD2(INT2/AIN1/RXD1), R41.1
- new net N$108: IC6.ADJ, R50.1, R51.2
- new net N$109: IC7.ADJ, R48.1, R49.2
- new net N$11: C12.1, U2.VOH
- new net N$110: LED1.C, R52.1
- new net N$111: LED2.C, R53.1
- new net N$112: LED3.C, R54.1
- new net N$113: LED4.C, R55.1
- new net N$114: LED5.C, R56.1
- new net N$115: LED6.C, R57.1
- new net N$116: C76.1, IC5.XTAL1, XTAL1.2
- new net N$117: C77.1, IC5.XTAL2, XTAL1.1
- new net N$118: JP9.3, R33.1, X3.1
- new net N$12: C17.2, U2.LOP
- new net N$122: IC5.PD7(INT7/HWB/CTS/T0), SJ1.1
- new net N$123: IC5.PC1(/RESET), R58.2, SJ2.1
- new net N$16: C17.1, U2.VIP
- new net N$18: C16.2, U2.VIN
- new net N$19: C16.1, R22.2, U2.LON
- new net N$21: C18.1, C19.1, U2.VCM
- new net N$22: C20.1, C21.1, R21.1, U2.RCLMP
- new net N$27: C22.2, U2.LMD
- new net N$28: C23.1, C46.1, C61.1, U2.INH
- new net N$29: C23.2, JP3.1
- new net N$30: JP3.2, R22.1
- new net N$31: C26.1, C27.1, L6.2, U2.VPOS
- new net N$55: C30.2, U3.BP
- new net N$56: C33.1, L5.2, U3.EN, U3.IN
- new net N$57: C37.1, C38.1, C39.2, U1.REFB
- new net N$58: C37.2, C38.2, C40.2, U1.REFT
- new net N$59: C41.2, C42.2, R26.A, U1.VREF
- new net N$6: C44.1, R13.1, R15.2, R19.2, R20.2, U1.VIN+
- new net N$60: C45.1, JP4.2, U1.SENSE
- new net N$61: R23.1, R24.1, U1.MODE
- new net N$62: C43.1, R14.1, R16.2, R17.1, R18.1, U1.VIN-
- new net N$63: JP4.1, R26.S
- new net N$64: L7.1, X2.1
- new net N$65: JP9.5, R32.1
- new net N$67: C51.1, R27.2, R28.1
- new net N$68: C52.1, D4.A, R28.2, U2.GAIN
- new net N$69: C24.1, C25.1, C50.1, C59.2, L2.2, U2.ENBL, U2.ENBV, U2.VPSL
- new net N$7: C12.2, R15.1
- new net N$70: R14.2, R30.1, T1.S2
- new net N$71: C53.2, X1.1
- new net N$72: C53.1, L8.1
- new net N$73: L8.2, T1.P1
- new net N$75: R13.2, R29.2, T1.S1
- new net N$76: C54.1, C55.1, C56.2, C57.2, R29.1, R30.2, T1.ST
- new net N$77: R33.2, R43.1, R45.2, U5.CLK_IN1
- new net N$78: C46.2, L7.2
- new net N$79: IC4.LX, L10.1
- new net N$8: C15.2, R16.1
- new net N$80: R31.1, R34.2, X4.1
- new net N$81: R32.2, R44.1, R46.2, U5.CLK_IN0
- new net N$82: C74.1, DC1.+VOUT, IC7.IN
- new net N$83: IC4.FB, R35.1, R36.2
- new net N$84: IC4.EN, R37.1
- new net N$85: C65.2, R38.1
- new net N$86: IC4.COMP, R38.2
- new net N$87: JP13.5, U7.A6
- new net N$88: IC5.D-, R39.2
- new net N$89: JP13.16, U6.B4
- new net N$9: C15.1, U2.VOL
- new net N$90: JP13.14, U6.B3
- new net N$91: JP13.12, U6.B2
- new net N$92: JP13.10, U6.B1
- new net N$93: C68.1, C69.1, C70.1, C71.1, C72.1, JP13.8, U6.VCCB, U7.VCCA, U8.VCCB, U9.VCCB
- new net N$94: JP13.7, U7.A5
- new net N$95: JP13.9, U7.A4
- new net N$96: JP13.11, U7.A3
- new net N$97: JP13.13, U7.A2
- new net N$98: JP13.15, U7.A1
- new net N$99: C75.2, DC1.-VOUT, IC6.IN
- new net PRG_MISO: IC5.PB3(PDO/MISO), U7.B5
- new net PRG_MOSI: IC5.PB2(PDI/MISO), U7.B4
- new net PRG_PDIC: IC5.PD5(XCK), U7.B2
- new net PRG_PDID: R41.2, R42.2, U7.B1
- new net PRG_RST: IC5.PB4(T1), U7.B6
- new net PRG_SCK: IC5.PB1(SCK), U7.B3
- new net TARGET1: CON6_ABE-FPGA.E13~C16~IO_L65N_SCP2_0, U6.A1
- new net TARGET2: CON6_ABE-FPGA.A13~D17~IO_L65P_SCP3_0, U6.A2
- new net TARGET3: CON6_ABE-FPGA.B12~B18~IO_L66P_SCP1_0, U6.A3
- new net TARGET4: CON6_ABE-FPGA.A12~A18~IO_L66N_SCP0_0, U6.A4
- new net VCCIO: U6.VCCA, U8.VCCA, U9.VCCA
- net +3V3: now also C13.1, C28.1, C29.1, C47.1, C48.1, C49.1, C62.1, C67.1, D3.C, JP13.18, JP13.3, JP14.4, JP2.4, JP9.2, JP9.7, L5.1, R43.2, R44.2, U$3.AVCC@0, U$3.AVCC@1, U$3.DVCC@0, U$3.DVCC@1, U$5.AVCC@0, U$5.AVCC@1, U$5.DVCC@0, U$5.DVCC@1, U1.DRVDD, U5.VCC, U5.VCCOUT1, U5.VCCOUT2, U5.VCC_2
- net GND: now also C13.2, C18.2, C19.2, C20.2, C21.2, C22.1, C24.2, C25.2, C26.2, C27.2, C28.2, C29.2, C30.1, C31.2, C32.2, C33.2, C34.2, C35.2, C36.2, C39.1, C40.1, C41.1, C42.1, C43.2, C44.2, C47.2, C48.2, C49.2, C50.2, C51.2, C52.2, C54.2, C55.2, C56.1, C57.1, C58.2, C59.1, C60.2, C61.2, C63.1, C64.1, C65.1, C66.2, C67.2, C68.2, C69.2, C70.2, C71.2, C72.2, C73.2, C74.2, C75.1, C76.2, C77.2, C78.2, C79.2, C80.2, D4.C, DC1.-VIN, DC1.COM, IC4.AGND, IC4.PGND, IC5.GND, IC5.UGND, JP13.17, JP13.19, JP13.2, JP14.2, JP14.6, JP2.2, JP2.6, JP4.3, JP9.4, JP9.6, R18.2, R20.1, R21.2, R23.2, R25.1, R26.E, R34.1, R36.1, R45.1, R46.1, R47.1, R49.1, R51.1, R52.2, R53.2, R54.2, R55.2, R56.2, R57.2, SJ1.2, SJ2.2, T1.P2, U$3.GND@0, U$3.GND@1, U$3.GND@2, U$3.GND@3, U$5.GND@0, U$5.GND@1, U$5.GND@2, U$5.GND@3, U1.AGND@0, U1.AGND@1, U1.DRGND, U1.PDWN, U2.COML, U2.COMM@0, U2.COMM@1, U2.MODE, U3.GND, U5.GND, U5.GND_2, U5.GND_3, U5.GND_4, U6.GND, U7.A7, U7.A8, U7.GND, U8.GND, U9.GND, X1.2, X2.2, X4.2, X5.4, X5.S1, X5.S2; no longer C13.-, CON1.3, CON2.-
- net OA_ADC0: now also U1.D0
- net OA_ADC1: now also U1.D1
- net OA_ADC2: now also U1.D2
- net OA_ADC3: now also U1.D3
- net OA_ADC4: now also U1.D4
- net OA_ADC5: now also U1.D5
- net OA_ADC6: now also U1.D6
- net OA_ADC7: now also U1.D7
- net OA_ADC8: now also U1.D8
- net OA_ADC9: now also U1.D9
- net OA_ADCOR: now also U1.OR
- net OA_CLKADC: now also R25.2, U1.CLK
- net OA_CLKIN: now also D3.CA, R31.2, R47.2
- net OA_GAIN: now also R27.1
- net OA_HILO: now also U2.HILO
- net VIN: now also C64.2, IC4.VIN, JP6.2, R37.2; no longer C13.+, CON1.1, CON2.+
Other:
- note added: "1. External Enclosure = 1455N1602"
- note added: "5V"
- note added: "Analog Portion"
- note added: "DNM"
- note added: "NOTES PAGE"
- note added: "PMOD Connectors"
- note removed: "Input voltage: 4.5..16V"

Commit message: Finished ZTEX Board
Parts:
- added C81, C82, C83: (no value), rcl:C-EUC0603
Connections:
- removed net AGND: C45.2, C62.2, D3.A
- removed net DGND: X3.2
- removed net VCCIO: U6.VCCA, U8.VCCA, U9.VCCA
- new net N$119: CON6_ABE-FPGA.B17~C11~IO_L35P_GCLK17_0, JP5.36
- new net N$120: CON6_ABE-FPGA.E17~A12~IO_L36N_GCLK14_0, JP5.33
- new net N$121: CON6_ABE-FPGA.A18~C13~IO_L48P_0, JP5.34
- new net N$124: CON6_ABE-FPGA.B18~A13~IO_L48N_0, JP5.31
- new net N$125: CON6_ABE-FPGA.E18~B14~IO_L50P_0, JP5.32
- new net N$126: CON6_ABE-FPGA.A19~C12~IO_L37N_GCLK12_0, JP5.29
- new net N$127: CON6_ABE-FPGA.B19~D11~IO_L37P_GCLK13_0, JP5.30
- new net N$128: CON6_ABE-FPGA.E19~A14~IO_L50N_0, JP5.27
- new net N$129: CON6_ABE-FPGA.A20~C15~IO_L62P_0, JP5.28
- new net N$130: CON6_ABE-FPGA.B20~F10~IO_L38P_0, JP5.25
- new net N$131: CON6_ABE-FPGA.E20~D12~IO_L47N_0_NC45, JP5.26
- new net N$132: CON6_ABE-FPGA.E21~D13~IO_L47P_0_NC45, JP5.23
- new net N$133: CON6_ABE-FPGA.E22~A10~IO_L34N_GCLK18_0, JP5.24
- new net N$134: CON6_ABE-FPGA.E23~B10~IO_L34P_GCLK19_0, JP5.22
- new net N$135: CON6_ABE-FPGA.A24~C10~IO_L33N_0, JP5.19
- new net N$136: CON6_ABE-FPGA.B24~D10~IO_L33P_0, JP5.18
- new net N$137: CON6_ABE-FPGA.E24~C9~IO_L8P_0, JP5.17
- new net N$138: CON6_ABE-FPGA.A25~D8~IO_L32N_0, JP5.16
- new net N$139: CON6_ABE-FPGA.B25~D9~IO_L32P_0, JP5.15
- new net N$140: CON6_ABE-FPGA.E25~C7~IO_L5P_0, JP5.14
- new net N$141: CON6_ABE-FPGA.A26~A8~IO_L6N_0, JP5.13
- new net N$142: CON6_ABE-FPGA.B26~B8~IO_L6P_0, JP5.12
- new net N$143: CON6_ABE-FPGA.E26~A7~IO_L5N_0, JP5.11
- new net N$144: CON6_ABE-FPGA.A27~C8~IO_L7N_0, JP5.10
- new net N$145: CON6_ABE-FPGA.B27~D7~IO_L7P_0, JP5.9
- new net N$146: CON6_ABE-FPGA.E27~B6~IO_L4P_0, JP5.8
- new net N$147: CON6_ABE-FPGA.A28~C6~IO_L3N_0, JP5.7
- new net N$148: CON6_ABE-FPGA.B28~D6~IO_L3P_0, JP5.6
- new net N$149: CON6_ABE-FPGA.A29~A5~IO_L2N_0, JP5.5
- new net N$66: CON6_ABE-FPGA.A17~A11~IO_L35N_GCLK16_0, JP5.35
- net +3V3: now also C81.1, C82.1, C83.1, JP5.3, JP5.38, U6.VCCA, U8.VCCA, U9.VCCA
- net +5V: now also JP5.1, JP5.40
- net GND: now also C45.2, C62.2, C81.2, C82.2, C83.2, D3.A, JP5.2, JP5.20, JP5.21, JP5.37, JP5.39, JP5.4, X3.2

Commit message: Round-2 ZTEX board, fix a few more errors
Parts:
- added JP7: (no value), pinhead:PINHD-1X3
- added R59, R60: (no value), resistor:R-US_R0603
Connections:
- removed net N$149: CON6_ABE-FPGA.A29~A5~IO_L2N_0, JP5.5
- new net PLLSCL: CON6_ABE-FPGA.A29~A5~IO_L2N_0, JP7.2, R60.2, U5.SCLOCK
- new net PLLSDA: CON6_ABE-FPGA.B29~C5~IO_L2P_0, JP7.1, R59.2, U5.SDATA
- net +3V3: now also R59.1, R60.1
- net GND: now also JP7.3
Changed lines of the file:
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@@
 <part name="+3V33" library="supply1" deviceset="+3V3" device=""/>
 <part name="SUPPLY38" library="supply2" deviceset="GND" device=""/>
+<part name="R59" library="resistor" deviceset="R-US_" device="R0603"/>
+<part name="R60" library="resistor" deviceset="R-US_" device="R0603"/>
+<part name="+3V34" library="supply1" deviceset="+3V3" device=""/>
+<part name="+3V35" library="supply1" deviceset="+3V3" device=""/>
+<part name="JP7" library="pinhead" deviceset="PINHD-1X3" device=""/>
+<part name="SUPPLY113" library="supply2" deviceset="GND" device=""/>
 </parts>
 <sheets>
@@
 <instance part="+3V31" gate="G$1" x="193.04" y="180.34"/>
 <instance part="SUPPLY38" gate="GND" x="15.24" y="162.56"/>
+<instance part="R59" gate="G$1" x="81.28" y="124.46"/>
+<instance part="R60" gate="G$1" x="81.28" y="111.76"/>
+<instance part="+3V34" gate="G$1" x="76.2" y="127"/>
+<instance part="+3V35" gate="G$1" x="76.2" y="114.3"/>
+<instance part="JP7" gate="A" x="99.06" y="116.84"/>
+<instance part="SUPPLY113" gate="GND" x="88.9" y="111.76"/>
 </instances>
 <busses>
@@
 <pinref part="SUPPLY38" gate="GND" pin="GND"/>
 </segment>
+<segment>
+<pinref part="JP7" gate="A" pin="3"/>
+<pinref part="SUPPLY113" gate="GND" pin="GND"/>
+<wire x1="88.9" y1="114.3" x2="96.52" y2="114.3" width="0.1524" layer="91"/>
+</segment>
 </net>
 <net name="N$93" class="0">
@@
 <pinref part="+3V31" gate="G$1" pin="+3V3"/>
 </segment>
+<segment>
+<pinref part="R59" gate="G$1" pin="1"/>
+<pinref part="+3V34" gate="G$1" pin="+3V3"/>
+</segment>
+<segment>
+<pinref part="R60" gate="G$1" pin="1"/>
+<pinref part="+3V35" gate="G$1" pin="+3V3"/>
+</segment>
 </net>
 <net name="N$89" class="0">
@@
 </segment>
 </net>
+<net name="PLLSDA" class="0">
+<segment>
+<pinref part="U5" gate="A" pin="SDATA"/>
+<wire x1="73.66" y1="147.32" x2="71.12" y2="147.32" width="0.1524" layer="91"/>
+<wire x1="71.12" y1="147.32" x2="71.12" y2="119.38" width="0.1524" layer="91"/>
+<wire x1="71.12" y1="119.38" x2="86.36" y2="119.38" width="0.1524" layer="91"/>
+<pinref part="R59" gate="G$1" pin="2"/>
+<wire x1="86.36" y1="119.38" x2="86.36" y2="124.46" width="0.1524" layer="91"/>
+<pinref part="JP7" gate="A" pin="1"/>
+<wire x1="96.52" y1="119.38" x2="86.36" y2="119.38" width="0.1524" layer="91"/>
+<junction x="86.36" y="119.38"/>
+<label x="99.06" y="119.38" size="1.778" layer="95" xref="yes"/>
+</segment>
+</net>
+<net name="PLLSCL" class="0">
+<segment>
+<pinref part="U5" gate="A" pin="SCLOCK"/>
+<wire x1="73.66" y1="157.48" x2="68.58" y2="157.48" width="0.1524" layer="91"/>
+<wire x1="68.58" y1="157.48" x2="68.58" y2="116.84" width="0.1524" layer="91"/>
+<wire x1="68.58" y1="116.84" x2="86.36" y2="116.84" width="0.1524" layer="91"/>
+<pinref part="R60" gate="G$1" pin="2"/>
+<wire x1="86.36" y1="111.76" x2="86.36" y2="116.84" width="0.1524" layer="91"/>
+<pinref part="JP7" gate="A" pin="2"/>
+<wire x1="86.36" y1="116.84" x2="96.52" y2="116.84" width="0.1524" layer="91"/>
+<junction x="86.36" y="116.84"/>
+<label x="99.06" y="116.84" size="1.778" layer="95" xref="yes"/>
+</segment>
+</net>
 </nets>
 </sheet>
@@
 </segment>
 </net>
-<net name="N$149" class="0">
-<segment>
-<pinref part="CON6" gate="_ABE-FPGA" pin="A29~A5~IO_L2N_0"/>
-<pinref part="JP5" gate="A" pin="5"/>
-<wire x1="165.1" y1="63.5" x2="157.48" y2="63.5" width="0.1524" layer="91"/>
-<wire x1="157.48" y1="63.5" x2="104.14" y2="116.84" width="0.1524" layer="91"/>
-</segment>
-</net>
 <net name="+5V" class="0">
 <segment>
@@
 </segment>
 </net>
+<net name="PLLSDA" class="0">
+<segment>
+<pinref part="CON6" gate="_ABE-FPGA" pin="B29~C5~IO_L2P_0"/>
+<wire x1="165.1" y1="60.96" x2="152.4" y2="60.96" width="0.1524" layer="91"/>
+<label x="152.4" y="60.96" size="1.778" layer="95" rot="R180" xref="yes"/>
+</segment>
+</net>
+<net name="PLLSCL" class="0">
+<segment>
+<pinref part="CON6" gate="_ABE-FPGA" pin="A29~A5~IO_L2N_0"/>
+<wire x1="165.1" y1="63.5" x2="152.4" y2="63.5" width="0.1524" layer="91"/>
+<label x="152.4" y="63.5" size="1.778" layer="95" rot="R180" xref="yes"/>
+</segment>
+</net>

Commit message: First pass of OpenADC ZTEX Ordered
Parts:
- added JP8: (no value), pinhead:PINHD-1X2
- added TP3, TP4, TP5, TP6, TP7, TP8, TP9: PTR1PAD1-13, testpad:PTR1PAD1-13
Connections:
- net +1.2V: now also TP4.TP
- net +2.6V: now also TP5.TP
- net +3V3: now also TP6.TP, U6.OE
- net +5V: now also TP3.TP
- net CLK_PLL0: now also JP8.1
- net CLK_PLL1: now also JP8.2
- net GND: now also TP7.TP, TP8.TP, TP9.TP
Changed lines of the file:
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@@
 <part name="JP7" library="pinhead" deviceset="PINHD-1X3" device=""/>
 <part name="SUPPLY113" library="supply2" deviceset="GND" device=""/>
+<part name="JP8" library="pinhead" deviceset="PINHD-1X2" device=""/>
+<part name="TP3" library="testpad" deviceset="PTR1" device="PAD1-13"/>
+<part name="TP4" library="testpad" deviceset="PTR1" device="PAD1-13"/>
+<part name="TP5" library="testpad" deviceset="PTR1" device="PAD1-13"/>
+<part name="TP6" library="testpad" deviceset="PTR1" device="PAD1-13"/>
+<part name="TP7" library="testpad" deviceset="PTR1" device="PAD1-13"/>
+<part name="TP8" library="testpad" deviceset="PTR1" device="PAD1-13"/>
+<part name="TP9" library="testpad" deviceset="PTR1" device="PAD1-13"/>
 </parts>
 <sheets>
@@
 <instance part="SUPPLY98" gate="G$1" x="25.4" y="109.22"/>
 <instance part="JP6" gate="G$1" x="35.56" y="101.6"/>
+<instance part="TP3" gate="G$1" x="132.08" y="53.34"/>
+<instance part="TP4" gate="G$1" x="193.04" y="104.14" rot="R90"/>
+<instance part="TP5" gate="G$1" x="193.04" y="154.94" rot="R90"/>
+<instance part="TP6" gate="G$1" x="119.38" y="154.94" rot="R90"/>
+<instance part="TP7" gate="G$1" x="63.5" y="127"/>
+<instance part="TP8" gate="G$1" x="68.58" y="127"/>
+<instance part="TP9" gate="G$1" x="73.66" y="127"/>
 </instances>
 <busses>
@@
 <wire x1="53.34" y1="144.78" x2="53.34" y2="129.54" width="0.1524" layer="91"/>
 <wire x1="53.34" y1="129.54" x2="60.96" y2="129.54" width="0.1524" layer="91"/>
-<wire x1="60.96" y1="129.54" x2="76.2" y2="129.54" width="0.1524" layer="91"/>
+<wire x1="60.96" y1="129.54" x2="63.5" y2="129.54" width="0.1524" layer="91"/>
+<wire x1="63.5" y1="129.54" x2="68.58" y2="129.54" width="0.1524" layer="91"/>
+<wire x1="68.58" y1="129.54" x2="73.66" y2="129.54" width="0.1524" layer="91"/>
+<wire x1="73.66" y1="129.54" x2="76.2" y2="129.54" width="0.1524" layer="91"/>
 <wire x1="76.2" y1="129.54" x2="76.2" y2="137.16" width="0.1524" layer="91"/>
 <wire x1="86.36" y1="129.54" x2="76.2" y2="129.54" width="0.1524" layer="91"/>
@@
 <pinref part="R4" gate="G$1" pin="1"/>
 <pinref part="C3" gate="G$1" pin="1"/>
+<pinref part="TP7" gate="G$1" pin="TP"/>
+<junction x="63.5" y="129.54"/>
+<pinref part="TP8" gate="G$1" pin="TP"/>
+<junction x="68.58" y="129.54"/>
+<pinref part="TP9" gate="G$1" pin="TP"/>
+<junction x="73.66" y="129.54"/>
 </segment>
 <segment>
@@
 <wire x1="185.42" y1="96.52" x2="185.42" y2="104.14" width="0.1524" layer="91"/>
 <junction x="185.42" y="104.14"/>
+<pinref part="TP4" gate="G$1" pin="TP"/>
 </segment>
 </net>
@@
 <pinref part="R3" gate="G$1" pin="2"/>
 <pinref part="+3V1" gate="G$1" pin="+3V3"/>
+<pinref part="TP6" gate="G$1" pin="TP"/>
 </segment>
 </net>
@@
 <pinref part="R7" gate="G$1" pin="2"/>
 <pinref part="U$12" gate="G$1" pin="+2.6V"/>
+<pinref part="TP5" gate="G$1" pin="TP"/>
 </segment>
 </net>
@@
 <junction x="119.38" y="55.88"/>
 <pinref part="DC1" gate="G$1" pin="+VIN"/>
-<wire x1="119.38" y1="55.88" x2="144.78" y2="55.88" width="0.1524" layer="91"/>
+<wire x1="119.38" y1="55.88" x2="132.08" y2="55.88" width="0.1524" layer="91"/>
+<pinref part="TP3" gate="G$1" pin="TP"/>
+<wire x1="132.08" y1="55.88" x2="144.78" y2="55.88" width="0.1524" layer="91"/>
+<junction x="132.08" y="55.88"/>
 </segment>
 </net>
@@
 <instance part="JP7" gate="A" x="99.06" y="116.84"/>
 <instance part="SUPPLY113" gate="GND" x="88.9" y="111.76"/>
+<instance part="JP8" gate="G$1" x="147.32" y="170.18"/>
 </instances>
 <busses>
@@
 <pinref part="+3V28" gate="G$1" pin="+3V3"/>
 <junction x="241.3" y="160.02"/>
+<pinref part="U6" gate="A" pin="OE"/>
+<wire x1="236.22" y1="76.2" x2="241.3" y2="76.2" width="0.1524" layer="91"/>
+<wire x1="241.3" y1="76.2" x2="241.3" y2="83.82" width="0.1524" layer="91"/>
+<junction x="241.3" y="83.82"/>
 </segment>
 <segment>
@@
 <pinref part="U5" gate="A" pin="Y0"/>
 <wire x1="134.62" y1="172.72" x2="144.78" y2="172.72" width="0.1524" layer="91"/>
-<label x="144.78" y="172.72" size="1.778" layer="95" xref="yes"/>
+<label x="154.94" y="172.72" size="1.778" layer="95" xref="yes"/>
+<pinref part="JP8" gate="G$1" pin="1"/>
+<wire x1="144.78" y1="172.72" x2="154.94" y2="172.72" width="0.1524" layer="91"/>
+<junction x="144.78" y="172.72"/>
 </segment>
 </net>
@@
 <pinref part="U5" gate="A" pin="Y1"/>
 <wire x1="134.62" y1="170.18" x2="144.78" y2="170.18" width="0.1524" layer="91"/>
-<label x="144.78" y="170.18" size="1.778" layer="95" xref="yes"/>
+<label x="154.94" y="170.18" size="1.778" layer="95" xref="yes"/>
+<pinref part="JP8" gate="G$1" pin="2"/>
+<wire x1="144.78" y1="170.18" x2="154.94" y2="170.18" width="0.1524" layer="91"/>
+<junction x="144.78" y="170.18"/>
 </segment>
 </net>

Commit message: Various small other changes
Parts:
- C13, C47, C48, C49, C62, C66, C70, C72, C78, C79, C80: value (none) -> 100nF
- C67, C68, C69, C81, C82, C83: value (none) -> 22nF
- C71, C73: value (none) -> 1uF
- C76, C77: value (none) -> 22pF
- LED1: value (none) -> RED
- LED2: value (none) -> YELLOW
- LED3, LED6: value (none) -> GREEN
- LED4, LED5: value (none) -> BLUE
- R31: value (none) -> 50R
- R32, R33: value (none) -> 100R
- R35: value ? -> 52k3
- R36: value ? -> 10k
- R39, R40: value (none) -> 27R
- R41: value (none) -> 470R
- R52, R53, R54, R55, R56, R57: value (none) -> 220R
- R58: value (none) -> 1K
- R59, R60: value (none) -> 4k7
- R7: value 5K4 -> 5K36
- XTAL1: value (none) -> 16MHz
