File: hardware/targets/ztex/pcb/ztex_openadc_eagle/openadc_ztex.sch (EAGLE design)
At the start: 211 parts, among them CON3 JTAG, CON6 USB-FPGA1.15, IC1 AOZ1021, IC2 AOZ1021, IC3 AOZ1094, IC4 AOZ1021, IC5 AT90USB162A, T1 TC1-1T, U1 AD9215BRUZ, U2 AD8331, U3 LP3985IM5-3.0, U5 CDCE906PW, U6 TXB0104PWR, U7 TXB0108PWR, U8 SN74LVC1T45DBVT, U9 SN74LVC1T45DBVT, X1 SMA-142-0711-821/826, X2 SMA-142-0711-821/826, X3 SMA-142-0711-821/826, X4 SMA-142-0711-821/826, X5 PN61729-S

Commit message: Fixes to ZTEX PCB. Still need to fix physical issues with placement of ZTEX board
Parts:
- added R61: 470R, resistor:R-US_M0805
Connections:
- net +5V/2: now also R61.2
- net N$93: now also U7.OE
- net PRG_RST: now also R61.1
Other:
- note added: "A13"
- note added: "A14"
- note added: "A5"
- note added: "B14"
- note added: "C11"
- note added: "C13"
- note added: "CW"
- note added: "Clock from Victim"
- note added: "Clock to Victim"
- note added: "D11"
- note added: "D12"
- note added: "DIR"
- note added: "Direction"
- note added: "E11"
- note added: "FPGA3/Spare"
- note added: "H"
- note added: "HS1"
- note added: "HS2"
- note added: "I was in a huge rush getting this PCB made in time"
- note added: "INPUT"
- note added: "K15"
- note added: "K16"
- note added: "L"
- note added: "L12"
- note added: "L13"
- note added: "L14"
- note added: "L16"
- note added: "M10"
- note added: "M11"
- note added: "M12"
- note added: "M13"
- note added: "M15"
- note added: "M16"
- note added: "N14"
- note added: "N16"
- note added: "OUTPUT"
- note added: "Oh sweet lord these are a mess, sorry"
- note added: "P15"
- note added: "P16"
- note added: "P8"
- note added: "PRG_MISO"
- note added: "PRG_MOSI"
- note added: "PRG_PDIC"
- note added: "PRG_PDID"
- note added: "PRG_RST"
- note added: "PRG_SCK"
- note added: "R12"
- note added: "R14"
- note added: "R15"
- note added: "RXD"
- note added: "T12"
- note added: "T15"
- note added: "TARG1"
- note added: "TARG2"
- note added: "TARG3"
- note added: "TARG4"
- note added: "TXD"
- note added: "Trigger"
- note added: "Typical Uses"
- note added: "VICTIM"
- note added: "VREF_TARG"
- note added: "ZTEX 1.11 FPGA"
- note added: "and still need to clean this section up, the actual"
- note added: "connections are OK though..."

Commit message: Fixes in PCB.. still more to go
Parts:
- removed C65: 2n2, myrcl:C-EUC0805K
- removed IC4: AOZ1021, mystuff:AOZ1021
- removed L10: 4.7µ, myrcl:L-EUNR60
- removed R35: 52k3, myrcl:R-EU_R0805K
- removed R36: 10k, myrcl:R-EU_R0805K
- removed R37, R38: 7K5, myrcl:R-EU_R0805K
- JP5: device pinhead:PINHD-2X20/90 -> pinhead:PINHD-2X15/90
Connections:
- removed net N$119: CON6_ABE-FPGA.B17~C11~IO_L35P_GCLK17_0, JP5.36
- removed net N$120: CON6_ABE-FPGA.E17~A12~IO_L36N_GCLK14_0, JP5.33
- removed net N$121: CON6_ABE-FPGA.A18~C13~IO_L48P_0, JP5.34
- removed net N$124: CON6_ABE-FPGA.B18~A13~IO_L48N_0, JP5.31
- removed net N$125: CON6_ABE-FPGA.E18~B14~IO_L50P_0, JP5.32
- removed net N$126: CON6_ABE-FPGA.A19~C12~IO_L37N_GCLK12_0, JP5.29
- removed net N$127: CON6_ABE-FPGA.B19~D11~IO_L37P_GCLK13_0, JP5.30
- removed net N$128: CON6_ABE-FPGA.E19~A14~IO_L50N_0, JP5.27
- removed net N$129: CON6_ABE-FPGA.A20~C15~IO_L62P_0, JP5.28
- removed net N$130: CON6_ABE-FPGA.B20~F10~IO_L38P_0, JP5.25
- removed net N$131: CON6_ABE-FPGA.E20~D12~IO_L47N_0_NC45, JP5.26
- removed net N$132: CON6_ABE-FPGA.E21~D13~IO_L47P_0_NC45, JP5.23
- removed net N$133: CON6_ABE-FPGA.E22~A10~IO_L34N_GCLK18_0, JP5.24
- removed net N$134: CON6_ABE-FPGA.E23~B10~IO_L34P_GCLK19_0, JP5.22
- removed net N$135: CON6_ABE-FPGA.A24~C10~IO_L33N_0, JP5.19
- removed net N$136: CON6_ABE-FPGA.B24~D10~IO_L33P_0, JP5.18
- removed net N$137: CON6_ABE-FPGA.E24~C9~IO_L8P_0, JP5.17
- removed net N$138: CON6_ABE-FPGA.A25~D8~IO_L32N_0, JP5.16
- removed net N$139: CON6_ABE-FPGA.B25~D9~IO_L32P_0, JP5.15
- removed net N$140: CON6_ABE-FPGA.E25~C7~IO_L5P_0, JP5.14
- removed net N$141: CON6_ABE-FPGA.A26~A8~IO_L6N_0, JP5.13
- removed net N$142: CON6_ABE-FPGA.B26~B8~IO_L6P_0, JP5.12
- removed net N$143: CON6_ABE-FPGA.E26~A7~IO_L5N_0, JP5.11
- removed net N$144: CON6_ABE-FPGA.A27~C8~IO_L7N_0, JP5.10
- removed net N$145: CON6_ABE-FPGA.B27~D7~IO_L7P_0, JP5.9
- removed net N$146: CON6_ABE-FPGA.E27~B6~IO_L4P_0, JP5.8
- removed net N$147: CON6_ABE-FPGA.A28~C6~IO_L3N_0, JP5.7
- removed net N$148: CON6_ABE-FPGA.B28~D6~IO_L3P_0, JP5.6
- removed net N$66: CON6_ABE-FPGA.A17~A11~IO_L35N_GCLK16_0, JP5.35
- removed net N$79: IC4.LX, L10.1
- removed net N$83: IC4.FB, R35.1, R36.2
- removed net N$84: IC4.EN, R37.1
- removed net N$85: C65.2, R38.1
- removed net N$86: IC4.COMP, R38.2
- new net EXPIO10: CON6_ABE-FPGA.E25~C7~IO_L5P_0, JP5.10
- new net EXPIO11: CON6_ABE-FPGA.A24~C10~IO_L33N_0, JP5.11
- new net EXPIO12: CON6_ABE-FPGA.B24~D10~IO_L33P_0, JP5.12
- new net EXPIO13: CON6_ABE-FPGA.E24~C9~IO_L8P_0, JP5.13
- new net EXPIO14: CON6_ABE-FPGA.E23~B10~IO_L34P_GCLK19_0, JP5.14
- new net EXPIO15: CON6_ABE-FPGA.E22~A10~IO_L34N_GCLK18_0, JP5.15
- new net EXPIO16: CON6_ABE-FPGA.E21~D13~IO_L47P_0_NC45, JP5.16
- new net EXPIO17: CON6_ABE-FPGA.E20~D12~IO_L47N_0_NC45, JP5.17
- new net EXPIO18: CON6_ABE-FPGA.B20~F10~IO_L38P_0, JP5.18
- new net EXPIO19: CON6_ABE-FPGA.A20~C15~IO_L62P_0, JP5.19
- new net EXPIO20: CON6_ABE-FPGA.E19~A14~IO_L50N_0, JP5.20
- new net EXPIO21: CON6_ABE-FPGA.B19~D11~IO_L37P_GCLK13_0, JP5.21
- new net EXPIO22: CON6_ABE-FPGA.A19~C12~IO_L37N_GCLK12_0, JP5.22
- new net EXPIO23: CON6_ABE-FPGA.A18~C13~IO_L48P_0, JP5.23
- new net EXPIO24: CON6_ABE-FPGA.B18~A13~IO_L48N_0, JP5.24
- new net EXPIO25: CON6_ABE-FPGA.E18~B14~IO_L50P_0, JP5.25
- new net EXPIO26: CON6_ABE-FPGA.B17~C11~IO_L35P_GCLK17_0, JP5.26
- new net EXPIO27: CON6_ABE-FPGA.A17~A11~IO_L35N_GCLK16_0, JP5.27
- new net EXPIO28: CON6_ABE-FPGA.E17~A12~IO_L36N_GCLK14_0, JP5.28
- new net EXPIO5: CON6_ABE-FPGA.A27~C8~IO_L7N_0, JP5.5
- new net EXPIO6: CON6_ABE-FPGA.B26~B8~IO_L6P_0, JP5.6
- new net EXPIO7: CON6_ABE-FPGA.A26~A8~IO_L6N_0, JP5.7
- new net EXPIO8: CON6_ABE-FPGA.A25~D8~IO_L32N_0, JP5.8
- new net EXPIO9: CON6_ABE-FPGA.B25~D9~IO_L32P_0, JP5.9
- net +3V3: no longer JP5.38
- net +5V: now also C1.2, C4.2, C64.2, C7.2, C8.2, IC1.VIN, IC2.VIN, IC3.VIN, JP6.2, R1.2, R12.2, R5.2; no longer JP5.40, L10.2, R35.2
- net GND: now also JP5.29, JP5.30; no longer C65.1, IC4.AGND, IC4.PGND, JP5.20, JP5.21, JP5.37, JP5.39, R36.1
- net VIN: no longer C1.2, C4.2, C64.2, C7.2, C8.2, IC1.VIN, IC2.VIN, IC3.VIN, IC4.VIN, JP6.2, R1.2, R12.2, R37.2, R5.2
Other:
- note removed: "5V"
- note removed: "I was in a huge rush getting this PCB made in time"
- note removed: "Oh sweet lord these are a mess, sorry"
- note removed: "and still need to clean this section up, the actual"
- note removed: "connections are OK though..."

Commit message: Bring back 3.3-5v converter
Parts:
- added C65: 100nF, rcl:C-EUC0603
- added C84, C85, C86, C87: 1u, rcl:C-EUC0603
- added L9: 120nH, SparkFun:INDUCTOR0603
- added U4: LTC3200ES6, customs:LTC3200ES6
- R61: device resistor:R-US_M0805 -> resistor:R-US_R0603
Connections:
- new net N$74: C85.1, U4.C-
- new net N$79: C85.2, U4.C+
- new net N$85: C86.2, L9.1, U4.!SHDN, U4.VIN
- new net N$86: C84.1, C87.2, L2.1, L6.1, U4.VOUT
- net +3V3: now also C65.1, L9.2
- net +5V: no longer L2.1, L6.1
- net GND: now also C65.2, C84.2, C86.1, C87.1, U4.GND

Commit message: Fix other spacing issues - done?
Parts:
- removed JP14: EXP-MINI, pinhead:PINHD-2X3/90
Connections:
- net +3V3: no longer JP14.4
- net +9V: no longer JP14.1
- net -9V: no longer JP14.5
- net GND: no longer JP14.2, JP14.6
Changed lines of the file:
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@@
 </part>
 <part name="X3" library="con-coax" deviceset="SMA-" device="142-0711-821/826"/>
-<part name="JP14" library="pinhead" deviceset="PINHD-2X3" device="/90" value="EXP-MINI"/>
 <part name="JP13" library="pinhead" deviceset="PINHD-2X10" device="/90" value="TARGET"/>
 <part name="C63" library="myrcl" deviceset="C-EU" device="C0805K" value="22µ"/>
@@
 <part name="SUPPLY84" library="supply2" deviceset="+9V" device=""/>
 <part name="SUPPLY85" library="supply2" deviceset="-9V" device=""/>
-<part name="SUPPLY86" library="supply2" deviceset="GND" device=""/>
 <part name="SUPPLY87" library="supply2" deviceset="GND" device=""/>
 <part name="LED1" library="dp_devices" deviceset="LED" device="-3MM" value="RED"/>
@@
 <instance part="JP9" gate="A" x="22.86" y="134.62"/>
 <instance part="X3" gate="G1" x="12.7" y="175.26"/>
-<instance part="JP14" gate="A" x="22.86" y="109.22"/>
 <instance part="JP13" gate="A" x="152.4" y="71.12"/>
 <instance part="SUPPLY15" gate="GND" x="142.24" y="48.26"/>
@@
 <instance part="+3V25" gate="G$1" x="152.4" y="157.48"/>
 <instance part="+3V26" gate="G$1" x="152.4" y="154.94"/>
-<instance part="SUPPLY84" gate="G$1" x="10.16" y="114.3"/>
+<instance part="SUPPLY84" gate="G$1" x="12.7" y="96.52"/>
 <instance part="SUPPLY85" gate="G$1" x="12.7" y="81.28"/>
-<instance part="SUPPLY86" gate="GND" x="35.56" y="104.14"/>
 <instance part="SUPPLY87" gate="GND" x="35.56" y="83.82"/>
-<instance part="+3V27" gate="G$1" x="33.02" y="121.92"/>
+<instance part="+3V27" gate="G$1" x="33.02" y="99.06"/>
 <instance part="+3V28" gate="G$1" x="241.3" y="162.56"/>
 <instance part="C81" gate="G$1" x="193.04" y="175.26"/>
@@
 </segment>
 <segment>
-<pinref part="JP14" gate="A" pin="6"/>
-<wire x1="27.94" y1="106.68" x2="35.56" y2="106.68" width="0.1524" layer="91"/>
-<wire x1="35.56" y1="106.68" x2="35.56" y2="111.76" width="0.1524" layer="91"/>
-<wire x1="35.56" y1="111.76" x2="27.94" y2="111.76" width="0.1524" layer="91"/>
-<pinref part="JP14" gate="A" pin="2"/>
-<pinref part="SUPPLY86" gate="GND" pin="GND"/>
-<junction x="35.56" y="106.68"/>
-</segment>
-<segment>
 <pinref part="JP2" gate="A" pin="6"/>
 <wire x1="27.94" y1="86.36" x2="35.56" y2="86.36" width="0.1524" layer="91"/>
@@
 </segment>
 <segment>
-<pinref part="JP14" gate="A" pin="4"/>
-<wire x1="27.94" y1="109.22" x2="33.02" y2="109.22" width="0.1524" layer="91"/>
-<wire x1="33.02" y1="109.22" x2="33.02" y2="119.38" width="0.1524" layer="91"/>
 <pinref part="+3V27" gate="G$1" pin="+3V3"/>
 <pinref part="JP2" gate="A" pin="4"/>
 <wire x1="27.94" y1="88.9" x2="33.02" y2="88.9" width="0.1524" layer="91"/>
-<wire x1="33.02" y1="88.9" x2="33.02" y2="109.22" width="0.1524" layer="91"/>
-<junction x="33.02" y="109.22"/>
+<wire x1="33.02" y1="88.9" x2="33.02" y2="96.52" width="0.1524" layer="91"/>
 </segment>
 <segment>
@@
 <net name="+9V" class="0">
 <segment>
-<pinref part="JP14" gate="A" pin="1"/>
-<wire x1="20.32" y1="111.76" x2="10.16" y2="111.76" width="0.1524" layer="91"/>
-<wire x1="10.16" y1="111.76" x2="10.16" y2="91.44" width="0.1524" layer="91"/>
+<wire x1="12.7" y1="93.98" x2="12.7" y2="91.44" width="0.1524" layer="91"/>
 <pinref part="JP2" gate="A" pin="1"/>
-<wire x1="10.16" y1="91.44" x2="20.32" y2="91.44" width="0.1524" layer="91"/>
+<wire x1="12.7" y1="91.44" x2="20.32" y2="91.44" width="0.1524" layer="91"/>
 <pinref part="SUPPLY84" gate="G$1" pin="+9V"/>
-<junction x="10.16" y="111.76"/>
 </segment>
 </net>
@@
 <pinref part="SUPPLY85" gate="G$1" pin="-9V"/>
 <wire x1="12.7" y1="86.36" x2="12.7" y2="83.82" width="0.1524" layer="91"/>
-<pinref part="JP14" gate="A" pin="5"/>
-<wire x1="20.32" y1="106.68" x2="12.7" y2="106.68" width="0.1524" layer="91"/>
-<wire x1="12.7" y1="106.68" x2="12.7" y2="86.36" width="0.1524" layer="91"/>
-<junction x="12.7" y="86.36"/>
 </segment>
 </net>

Commit message: Updating HW Design Files
Parts:
- C14: value 560µ -> 470u
- C58, C60, C74, C75: value (none) -> 100nF
- R42: value (none) -> 470
- R43, R44, R45, R46, R49, R51: value (none) -> 1k,1%
- R48, R50: value (none) -> 200R,1%
- R9: value 25K -> 24k9,1%
