File: hardware/capture/sakura-g/adapter-pcb/adapter-pcb.sch (EAGLE design)
At the start: 6 parts

Commit message: Update PCBs
Changed lines of the file:
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@@
 <pinref part="JP1" gate="A" pin="28"/>
 <wire x1="88.9" y1="60.96" x2="88.9" y2="71.12" width="0.1524" layer="91"/>
+<label x="88.9" y="68.58" size="1.778" layer="95" rot="R90"/>
 </segment>
 </net>
@@
 <pinref part="JP1" gate="A" pin="27"/>
 <wire x1="88.9" y1="53.34" x2="88.9" y2="45.72" width="0.1524" layer="91"/>
+<label x="88.9" y="40.64" size="1.778" layer="95" rot="R90"/>
 </segment>
 </net>
@@
 <pinref part="JP1" gate="A" pin="26"/>
 <wire x1="86.36" y1="60.96" x2="86.36" y2="71.12" width="0.1524" layer="91"/>
+<label x="86.36" y="68.58" size="1.778" layer="95" rot="R90"/>
 </segment>
 </net>
@@
 <pinref part="JP1" gate="A" pin="25"/>
 <wire x1="86.36" y1="53.34" x2="86.36" y2="45.72" width="0.1524" layer="91"/>
+<label x="86.36" y="40.64" size="1.778" layer="95" rot="R90"/>
 </segment>
 </net>
@@
 <pinref part="JP1" gate="A" pin="24"/>
 <wire x1="83.82" y1="60.96" x2="83.82" y2="71.12" width="0.1524" layer="91"/>
+<label x="83.82" y="68.58" size="1.778" layer="95" rot="R90"/>
 </segment>
 </net>
@@
 <pinref part="JP1" gate="A" pin="23"/>
 <wire x1="83.82" y1="53.34" x2="83.82" y2="45.72" width="0.1524" layer="91"/>
+<label x="83.82" y="40.64" size="1.778" layer="95" rot="R90"/>
 </segment>
 </net>
@@
 <pinref part="JP1" gate="A" pin="18"/>
 <wire x1="76.2" y1="60.96" x2="76.2" y2="68.58" width="0.1524" layer="91"/>
-<label x="73.66" y="68.58" size="1.778" layer="95" rot="R270"/>
+<label x="74.422" y="75.184" size="1.778" layer="95" rot="R270"/>
 </segment>
 </net>
@@
 <pinref part="JP1" gate="A" pin="17"/>
 <wire x1="76.2" y1="53.34" x2="76.2" y2="45.72" width="0.1524" layer="91"/>
-<label x="76.2" y="45.72" size="1.778" layer="95" rot="R90"/>
+<label x="76.2" y="40.64" size="1.778" layer="95" rot="R90"/>
 </segment>
 </net>
@@
 <pinref part="JP1" gate="A" pin="16"/>
 <wire x1="73.66" y1="60.96" x2="73.66" y2="68.58" width="0.1524" layer="91"/>
+<label x="73.66" y="68.58" size="1.778" layer="95" rot="R90"/>
 </segment>
 </net>
@@
 <pinref part="JP1" gate="A" pin="15"/>
 <wire x1="73.66" y1="53.34" x2="73.66" y2="45.72" width="0.1524" layer="91"/>
-<label x="73.66" y="45.72" size="1.778" layer="95" rot="R90"/>
+<label x="73.66" y="40.64" size="1.778" layer="95" rot="R90"/>
 </segment>
 </net>
@@
 <pinref part="JP1" gate="A" pin="14"/>
 <wire x1="71.12" y1="60.96" x2="71.12" y2="68.58" width="0.1524" layer="91"/>
+<label x="71.12" y="68.58" size="1.778" layer="95" rot="R90"/>
 </segment>
 </net>
@@
 <pinref part="JP1" gate="A" pin="13"/>
 <wire x1="71.12" y1="53.34" x2="71.12" y2="45.72" width="0.1524" layer="91"/>
-<label x="71.12" y="45.72" size="1.778" layer="95" rot="R90"/>
+<label x="71.12" y="40.64" size="1.778" layer="95" rot="R90"/>
 </segment>
 </net>
@@
 <pinref part="JP1" gate="A" pin="12"/>
 <wire x1="68.58" y1="60.96" x2="68.58" y2="68.58" width="0.1524" layer="91"/>
+<label x="68.58" y="68.58" size="1.778" layer="95" rot="R90"/>
 </segment>
 </net>
@@
 <pinref part="JP1" gate="A" pin="11"/>
 <wire x1="68.58" y1="53.34" x2="68.58" y2="45.72" width="0.1524" layer="91"/>
-<label x="68.58" y="45.72" size="1.778" layer="95" rot="R90"/>
+<label x="68.58" y="40.64" size="1.778" layer="95" rot="R90"/>
 </segment>
 </net>
@@
 <pinref part="U$1" gate="G$1" pin="NC@4"/>
 <wire x1="30.48" y1="43.18" x2="48.26" y2="43.18" width="0.1524" layer="91"/>
-<wire x1="48.26" y1="43.18" x2="48.26" y2="73.66" width="0.1524" layer="91"/>
+<wire x1="48.26" y1="43.18" x2="48.26" y2="78.74" width="0.1524" layer="91"/>
 <pinref part="JP1" gate="A" pin="22"/>
-<wire x1="48.26" y1="73.66" x2="81.28" y2="73.66" width="0.1524" layer="91"/>
-<wire x1="81.28" y1="73.66" x2="81.28" y2="60.96" width="0.1524" layer="91"/>
+<wire x1="48.26" y1="78.74" x2="81.28" y2="78.74" width="0.1524" layer="91"/>
+<wire x1="81.28" y1="78.74" x2="81.28" y2="60.96" width="0.1524" layer="91"/>
 </segment>
 </net>
