File: hardware/capture/chipwhisperer-rev2/cwrev2_eagleproj/openadc_ztex.brd (EAGLE design)
At the start: 155 x 100.3 mm, 211 parts, among them CON3 JTAG, CON6 USB-FPGA1.15, IC1 AOZ1021, IC2 AOZ1021, IC3 AOZ1094, IC5 AT90USB162A, T1 TC1-1T, U1 AD9215BRUZ, U2 AD8331, U3 LP3985IM5-3.0, U4 LTC3200ES6, U5 CDCE906PW, U6 TXB0104PWR, U7 TXB0108PWR, U8 SN74LVC1T45DBVT, U9 SN74LVC1T45DBVT, X1 SMA-142-0711-821/826, X2 SMA-142-0711-821/826, X3 SMA-142-0711-821/826, X4 SMA-142-0711-821/826, X5 PN61729-S

Commit message: Fix CWRev2 mistakes
Parts:
- added C88, C89, C90: 100nF, rcl:C0603
- added C91: (no value), resistor:C0603
- added JP10: (no value), pinhead:1X02
- added R35, R36: 2k2, resistor:R0603
- added U10: ATSHA204-SH, customs:SO08
- D1: device diode:DO214AA -> diode:MELF-MLL41
- L3: device inductors:DR1030 -> inductors:DR1030MOD.PAC
- moved R32 5.09 mm to (137.9, 32.8)
- moved R33 5.08 mm to (137.9, 34.3), turned to 0 degrees
- moved R44 5.04 mm to (140.5, 35.3), turned to 90 degrees
- moved R43 4.85 mm to (140.5, 31.8), turned to 270 degrees
- moved R46 4.58 mm to (142.0, 35.3), turned to 270 degrees
- moved R45 4.37 mm to (142.0, 31.8), turned to 90 degrees
- moved U$5 2.54 mm to (113.3, 34.0)
- moved L3 1.30 mm to (67.0, 48.6)
- moved R12 1.02 mm to (79.4, 51.1)
- moved JP2 0.76 mm to (154.9, 11.7)
- moved D1 0.46 mm to (74.8, 52.6)
Connections:
- removed net VIN: CON6.A1, CON6.B1, JP1.1
- new net N$119: JP10.2, U5.2
- new net N$120: JP10.1, U5.1
- new net N$121: CON6.B28, R36.2, U10.6
- new net N$124: CON6.A28, R35.2, U10.5
- new net N$125: R32.2, U5.5
- new net N$66: C90.1, JP9.3
- new net N$84: R33.1, U5.6
- net +3V3: now also C91.1, R35.1, R36.1, U10.8
- net +5V: now also CON6.A1, CON6.B1, JP1.1
- net GND: now also C91.2, U10.4
- net N$118: now also C88.1; no longer JP9.3, R33.1
- net N$65: now also C89.1; no longer R32.1
- net N$77: now also C89.2, R32.1; no longer R33.2, U5.6
- net N$81: now also C88.2, C90.2, R33.2; no longer R32.2, U5.5
Routing:
- net +5V: track 539.6 -> 603.0 mm
- net VIN: track 37.9 -> 0.00 mm
- net +3V3: track 779.7 -> 810.9 mm
- net N$121: track 0.00 -> 17.0 mm
- net N$124: track 0.00 -> 15.5 mm, vias 0 -> 1
- net N$118: track 23.8 -> 10.0 mm
- net N$119: track 0.00 -> 7.93 mm
- net GND: track 288.2 -> 282.2 mm, vias 292 -> 291
- net N$120: track 0.00 -> 5.83 mm
- net N$66: track 0.00 -> 4.40 mm
- net N$84: track 0.00 -> 3.99 mm
- net N$125: track 0.00 -> 3.88 mm
- net N$81: track 10.4 -> 13.2 mm
- net N$77: track 10.4 -> 7.76 mm
- net N$49: track 20.1 -> 22.6 mm
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Other:
- board text added: "1.2V"
- board text added: "REV: 1SEPT2013"
- board text removed: "REV: 6JUNE2013"

Commit message: Update CW PCB & Clock Recovery PCB
Other:
- board text added: "+3.3V"
- board text added: "+VUSB (5V)"
- board text added: "1 2,4,29,30 3"
- board text added: "1,20"
- board text added: "11"
- board text added: "13"
- board text added: "15"
- board text added: "17"
- board text added: "17,19,2"
- board text added: "19"
- board text added: "2"
- board text added: "20"
- board text added: "29"
- board text added: "3"
- board text added: "3,18"
- board text added: "30"
- board text added: "4 5 6 7 8 9 10 11 12 13 14 15 16"
- board text added: "5"
- board text added: "5 6 7 8 9 10 11 12 13 14 15 16 17 18 19 20 21 22 23 24 25 26 27 28"
- board text added: "7"
- board text added: "9"
- board text added: "A27 B26 A26 A25 B25 E25 A24 B24 E24 E23 E22 E21 E20 B20 A20 E19 B19 A19 A18 B18 E18 B17 A17 E17"
- board text added: "A6 D6 C6 E6 F7 NC A7 C7 NC E7 E8 B8 A8 D8 C8 D9 C9 A9 B12 A12 F9 E10 C10 A10"
- board text added: "ChipWhisperer"
- board text added: "FPGA-HS1 PROG-RESET FPGA-HS2 PROG-MISO VTarget (IN) PROG-MOSI FPGA-TARG1(TX) PROG-SCK FPGA-TARG2(RX) PROG-PDIC FPGA-TARG3(SCARD) PROG-PDIC FPGA-TARG4(TRIG)"
- board text added: "JP13 (TARGET) Pinout:"
- board text added: "JP5 Pinout"
- board text added: "LX25FPGA"
- board text added: "PIN"
- board text added: "ZTEX"
- board text added: "www.ChipWhisperer.com"
- board text removed: "Colin O'Flynn"
- board text removed: "Power Supply Module 1.1"
- board text removed: "coflynn@newae.com"
- board text removed: "for ZTEX FPGA Modules"
Changed lines of the file:
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@@
 <layer number="24" name="bOrigins" color="15" fill="1" visible="yes" active="yes"/>
 <layer number="25" name="tNames" color="7" fill="1" visible="yes" active="yes"/>
-<layer number="26" name="bNames" color="7" fill="1" visible="no" active="yes"/>
+<layer number="26" name="bNames" color="7" fill="1" visible="yes" active="yes"/>
 <layer number="27" name="tValues" color="7" fill="1" visible="no" active="yes"/>
 <layer number="28" name="bValues" color="7" fill="1" visible="no" active="yes"/>
@@
 <wire x1="85.725" y1="14.2875" x2="85.725" y2="26.3525" width="0.1524" layer="22"/>
 <wire x1="77.47" y1="28.2575" x2="77.47" y2="26.9875" width="0.2032" layer="22"/>
-<text x="20.8415" y="37.354" size="1.6764" layer="26" ratio="12" rot="MR90">Power Supply Module 1.1</text>
-<text x="18.327" y="37.354" size="1.6764" layer="26" ratio="12" rot="MR90">for ZTEX FPGA Modules</text>
 <wire x1="111.3511" y1="63.279" x2="108.1253" y2="63.279" width="0.4064" layer="41"/>
 <wire x1="111.3511" y1="63.279" x2="108.1253" y2="63.279" width="0.4064" layer="42"/>
@@
 <text x="111.252" y="10.16" size="1.016" layer="21" font="vector" ratio="16">GND</text>
 <text x="40.132" y="83.82" size="1.016" layer="21" font="vector" ratio="16">GND</text>
-<text x="10.414" y="4.826" size="2.54" layer="21" font="vector" ratio="16">Colin O'Flynn</text>
-<text x="42.164" y="7.874" size="1.778" layer="21" font="vector" ratio="16">REV: 1SEPT2013</text>
-<text x="41.91" y="5.842" size="1.778" layer="21" font="vector" ratio="16">coflynn@newae.com</text>
+<text x="48.768" y="6.858" size="1.778" layer="21" font="vector" ratio="16">REV: 1SEPT2013</text>
 <text x="88.138" y="39.624" size="1.016" layer="21" font="vector" ratio="16">1.2V</text>
+<text x="17.526" y="0.508" size="3.81" layer="21" ratio="16" rot="R19">ChipWhisperer</text>
+<text x="49.022" y="4.318" size="1.6764" layer="21" font="vector" ratio="16">www.ChipWhisperer.com</text>
+<text x="10.414" y="68.58" size="1.016" layer="21" font="vector" ratio="16">1</text>
+<text x="10.414" y="71.12" size="1.016" layer="21" font="vector" ratio="16">3</text>
+<text x="10.414" y="73.66" size="1.016" layer="21" font="vector" ratio="16">5</text>
+<text x="10.668" y="76.2" size="1.016" layer="21" font="vector" ratio="16">7</text>
+<text x="10.668" y="78.74" size="1.016" layer="21" font="vector" ratio="16">9</text>
+<text x="10.414" y="81.28" size="1.016" layer="21" font="vector" ratio="16">11</text>
+<text x="10.414" y="83.82" size="1.016" layer="21" font="vector" ratio="16">13</text>
+<text x="10.414" y="86.36" size="1.016" layer="21" font="vector" ratio="16">15</text>
+<text x="10.16" y="88.9" size="1.016" layer="21" font="vector" ratio="16">17</text>
+<text x="10.16" y="91.44" size="1.016" layer="21" font="vector" ratio="16">19</text>
+<text x="5.842" y="93.218" size="1.016" layer="21" font="vector" ratio="16">20</text>
+<text x="6.604" y="66.802" size="1.016" layer="21" font="vector" ratio="16">2</text>
+<text x="28.448" y="57.658" size="1.016" layer="21" font="vector" ratio="16">JP13 (TARGET) Pinout:</text>
+<text x="29.464" y="55.626" size="1.016" layer="21" font="vector" ratio="16">1,20</text>
+<text x="34.798" y="55.626" size="1.016" layer="21" font="vector" ratio="16">+VUSB (5V)</text>
+<text x="29.464" y="54.102" size="1.016" layer="21" font="vector" ratio="16">3,18</text>
+<text x="34.798" y="54.102" size="1.016" layer="21" font="vector" ratio="16">3.3V</text>
+<text x="29.464" y="52.324" size="1.016" layer="21" font="vector" ratio="16">17,19,2</text>
+<text x="36.83" y="52.324" size="1.016" layer="21" font="vector" ratio="16">GND</text>
+<text x="29.21" y="32.512" size="1.016" layer="21" font="vector" ratio="16">4
+5
+6
+7
+8
+9
+10
+11
+12
+13
+14
+15
+16</text>
+<text x="34.798" y="32.258" size="1.016" layer="21" font="vector" ratio="16">FPGA-HS1
+PROG-RESET
+FPGA-HS2
+PROG-MISO
+VTarget (IN)
+PROG-MOSI
+FPGA-TARG1(TX)
+PROG-SCK
+FPGA-TARG2(RX)
+PROG-PDIC
+FPGA-TARG3(SCARD)
+PROG-PDIC
+FPGA-TARG4(TRIG)</text>
+<wire x1="27.94" y1="59.182" x2="27.94" y2="56.896" width="0.254" layer="21"/>
+<wire x1="27.94" y1="56.896" x2="27.94" y2="31.496" width="0.254" layer="21"/>
+<wire x1="27.94" y1="31.496" x2="50.8" y2="31.496" width="0.254" layer="21"/>
+<wire x1="50.8" y1="31.496" x2="50.8" y2="56.896" width="0.254" layer="21"/>
+<wire x1="50.8" y1="56.896" x2="50.8" y2="59.182" width="0.254" layer="21"/>
+<wire x1="50.8" y1="59.182" x2="27.94" y2="59.182" width="0.254" layer="21"/>
+<wire x1="27.94" y1="56.896" x2="50.8" y2="56.896" width="0.254" layer="21"/>
+<text x="11.7475" y="23.114" size="1.016" layer="21" font="vector" ratio="16" rot="R90">JP5 Pinout</text>
+<text x="12.192" y="6.35" size="1.016" layer="21" font="vector" ratio="16">5
+6
+7
+8
+9
+10
+11
+12
+13
+14
+15
+16
+17
+18
+19
+20
+21
+22
+23
+24
+25
+26
+27
+28</text>
+<text x="8.89" y="5.588" size="1.016" layer="21" font="vector" ratio="16">1</text>
+<text x="6.096" y="5.588" size="1.016" layer="21" font="vector" ratio="16">2</text>
+<text x="8.382" y="44.958" size="1.016" layer="21" font="vector" ratio="16">29</text>
+<text x="5.588" y="44.958" size="1.016" layer="21" font="vector" ratio="16">30</text>
+<text x="26.416" y="28.448" size="1.016" layer="21" font="vector" ratio="16">+VUSB (5V)</text>
+<text x="32.766" y="26.924" size="1.016" layer="21" font="vector" ratio="16">GND</text>
+<text x="26.416" y="25.4" size="1.016" layer="21" font="vector" ratio="16">+3.3V</text>
+<text x="15.494" y="6.35" size="1.016" layer="21" font="vector" ratio="16">A27
+B26
+A26
+A25
+B25
+E25
+A24
+B24
+E24
+E23
+E22
+E21
+E20
+B20
+A20
+E19
+B19
+A19
+A18
+B18
+E18
+B17
+A17
+E17</text>
+<text x="11.684" y="43.18" size="1.016" layer="21" font="vector" ratio="16">PIN</text>
+<text x="15.24" y="43.18" size="1.016" layer="21" font="vector" ratio="16">ZTEX</text>
+<text x="20.066" y="43.18" size="1.016" layer="21" font="vector" ratio="16">LX25FPGA</text>
+<text x="20.066" y="6.35" size="1.016" layer="21" font="vector" ratio="16">A6
+D6
+C6
+E6
+F7
+NC
+A7
+C7
+NC
+E7
+E8
+B8
+A8
+D8
+C8
+D9
+C9
+A9
+B12
+A12
+F9
+E10
+C10
+A10</text>
+<text x="24.384" y="25.4" size="1.016" layer="21" font="vector" ratio="16">1
+2,4,29,30
+3</text>
+<wire x1="10.414" y1="44.45" x2="10.414" y2="5.334" width="0.254" layer="21"/>
+<wire x1="10.414" y1="5.334" x2="23.114" y2="5.334" width="0.254" layer="21"/>
+<wire x1="23.114" y1="5.334" x2="23.114" y2="24.384" width="0.254" layer="21"/>
+<wire x1="23.114" y1="24.384" x2="23.368" y2="24.638" width="0.254" layer="21"/>
+<wire x1="23.368" y1="24.638" x2="36.068" y2="24.638" width="0.254" layer="21"/>
+<wire x1="36.068" y1="24.638" x2="36.068" y2="30.226" width="0.254" layer="21"/>
+<wire x1="36.068" y1="30.226" x2="27.178" y2="30.226" width="0.254" layer="21"/>
+<wire x1="27.178" y1="30.226" x2="27.178" y2="44.704" width="0.254" layer="21"/>
+<wire x1="27.178" y1="44.704" x2="10.668" y2="44.704" width="0.254" layer="21"/>
+<wire x1="10.668" y1="44.704" x2="10.414" y2="44.45" width="0.254" layer="21"/>
+<circle x="37.592" y="24.892" radius="0.359209375" width="0.254" layer="21"/>
+<wire x1="36.576" y1="24.384" x2="38.862" y2="24.384" width="0.254" layer="21"/>
+<wire x1="38.862" y1="24.384" x2="40.64" y2="24.384" width="0.254" layer="21"/>
+<wire x1="40.64" y1="24.384" x2="42.672" y2="24.384" width="0.254" layer="21"/>
+<wire x1="36.576" y1="18.796" x2="42.926" y2="18.796" width="0.254" layer="21"/>
+<wire x1="38.862" y1="24.384" x2="40.64" y2="24.384" width="0.254" layer="21" curve="180"/>
 </plain>
 <attributes>
@@
 </element>
 <element name="R61" library="resistor" package="R0603" value="470R" x="25.4" y="82.296" rot="MR90"/>
-<element name="JP5" library="pinhead" package="2X15/90" value="" x="2.794" y="25.908" rot="R90"/>
+<element name="JP5" library="pinhead" package="2X15/90" value="" x="2.794" y="25.908" smashed="yes" rot="R90">
+<attribute name="NAME" x="9.144" y="4.699" size="1.27" layer="25" ratio="10" rot="R180"/>
+<attribute name="VALUE" x="6.604" y="46.863" size="1.27" layer="27" rot="R180"/>
+</element>
 <element name="C65" library="rcl" package="C0603" value="100nF" x="14.478" y="94.742" smashed="yes" rot="R180">
 <attribute name="NAME" x="15.621" y="93.853" size="1.016" layer="25" font="vector" ratio="16" rot="R180"/>
@@
 </board>
 </drawing>
+<compatibility>
+<note version="6.3" minversion="6.2.2" severity="warning">
+Since Version 6.2.2 text objects can contain more than one line,
+which will not be processed correctly with this version.
+</note>
+</compatibility>
 </eagle>

Commit message: Add missing projects back to GIT
Parts:
- U6: value TXB0104PWR -> TXS0104EPWR
Changed lines of the file:
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@@
 <attribute name="VALUE" x="34.7726" y="76.2" size="0.8128" layer="27" rot="R180"/>
 </element>
-<element name="U6" library="Texas Instruments_By_element14_Batch_1" package="SOP65P640X120-14N" value="TXB0104PWR" x="20.32" y="91.44" smashed="yes" rot="R180">
+<element name="U6" library="Texas Instruments_By_element14_Batch_1" package="SOP65P640X120-14N" value="TXS0104EPWR" x="20.32" y="91.44" smashed="yes" rot="R180">
 <attribute name="PACKAGE" value="TSSOP-14" x="20.32" y="91.44" size="1.778" layer="27" rot="R180" display="off"/>
 <attribute name="OC_NEWARK" value="99K4466" x="20.32" y="91.44" size="1.778" layer="27" rot="R180" display="off"/>

Commit message: fix issue w/ CW Short on 1.2V rail
Parts:
- moved C9 0.36 mm to (74.0, 58.4)
- moved D1 0.36 mm to (74.5, 52.3)
- moved C11 0.25 mm to (72.1, 58.4)
Changed lines of the file:
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@@
 <attribute name="VALUE" x="90.7465" y="96.631" size="1.0668" layer="27" ratio="12" rot="R270"/>
 </element>
-<element name="C11" library="myrcl" package="C0805K" value="22µ" x="72.0725" y="58.1025" smashed="yes" rot="R270">
-<attribute name="NAME" x="72.658" y="60.214" size="1.0668" layer="25" ratio="12" rot="R90"/>
-<attribute name="VALUE" x="70.988" y="56.404" size="1.0668" layer="27" ratio="12" rot="R90"/>
+<element name="C11" library="myrcl" package="C0805K" value="22µ" x="72.0725" y="58.3565" smashed="yes" rot="R270">
+<attribute name="NAME" x="72.658" y="60.468" size="1.0668" layer="25" ratio="12" rot="R90"/>
+<attribute name="VALUE" x="70.988" y="56.658" size="1.0668" layer="27" ratio="12" rot="R90"/>
 </element>
 <element name="R10" library="myrcl" package="R0805K" value="1K2" x="82.8675" y="39.6875" smashed="yes">
@@
 <attribute name="MPN" value="CDRH104RNP-2R5NC" x="66.9925" y="48.641" size="1.778" layer="27" rot="R180" display="off"/>
 </element>
-<element name="C9" library="myrcl" package="C0805K" value="22µ" x="74.295" y="58.1025" smashed="yes" rot="R270">
-<attribute name="NAME" x="73.9" y="62.1505" size="1.016" layer="25" rot="R270"/>
-<attribute name="VALUE" x="72.395" y="59.1025" size="1.016" layer="27" rot="R270"/>
-</element>
-<element name="D1" library="diode" package="MELF-MLL41" value="" x="74.803" y="52.578" rot="R90"/>
+<element name="C9" library="myrcl" package="C0805K" value="22µ" x="74.041" y="58.3565" smashed="yes" rot="R270">
+<attribute name="NAME" x="73.646" y="62.4045" size="1.016" layer="25" rot="R270"/>
+<attribute name="VALUE" x="72.141" y="59.3565" size="1.016" layer="27" rot="R270"/>
+</element>
+<element name="D1" library="diode" package="MELF-MLL41" value="" x="74.549" y="52.324" rot="R90"/>
 <element name="JP1" library="pinhead" package="1X02" value="" x="91.44" y="95.5675"/>
 <element name="U$3" library="openadc_footprint" package="OPENADCREV1" value="OPENADC" x="113.3475" y="77.1525" rot="R180"/>
@@
 <contactref element="CON6" pad="D28"/>
 <contactref element="CON6" pad="C28"/>
-<wire x1="74.295" y1="57.1025" x2="72.0725" y2="57.1025" width="1.524" layer="1"/>
+<wire x1="74.041" y1="57.3565" x2="72.0725" y2="57.3565" width="1.524" layer="1"/>
 <contactref element="TP4" pad="TP"/>
 <wire x1="89.408" y1="42.164" x2="86.614" y2="42.164" width="1.27" layer="1"/>
