File: hardware/capture/chipwhisperer-rev2/cwrev2_eagleproj/openadc_ztex.brd (EAGLE design)
At the start: 155 x 100.3 mm, 219 parts, among them CON3 JTAG, CON6 USB-FPGA1.15, IC1 AOZ1021, IC2 AOZ1021, IC3 AOZ1094, IC5 AT90USB162A, T1 TC1-1T, U1 AD9215BRUZ, U10 ATSHA204-SH, U2 AD8331, U3 LP3985IM5-3.0, U4 LTC3200ES6, U5 CDCE906PW, U6 TXS0104EPWR, U7 TXB0108PWR, U8 SN74LVC1T45DBVT, U9 SN74LVC1T45DBVT, X1 SMA-142-0711-821/826, X2 SMA-142-0711-821/826, X3 SMA-142-0711-821/826, X4 SMA-142-0711-821/826, X5 PN61729-S

Commit message: Update #1
Parts:
- added LED10, LED11: BLUE, dp_devices:LED-805
- added LED12, LED9: GREEN, dp_devices:LED-805
- added LED7: RED, dp_devices:LED-805
- added LED8: YELLOW, dp_devices:LED-805
- LED1, LED2, LED3, LED4, LED5, LED6: device dp_devices:LED-3MM -> dp_devices:LED-805
- flipped LED1 to the bottom, turned to 180 degrees
- flipped LED2 to the bottom, turned to 180 degrees
- flipped LED3 to the bottom, turned to 180 degrees
- flipped LED4 to the bottom, turned to 180 degrees
- flipped LED5 to the bottom, turned to 180 degrees
- flipped LED6 to the bottom, turned to 180 degrees
Connections:
- net LED1: now also LED7.A
- net LED2: now also LED8.A
- net LED3: now also LED9.A
- net LED4: now also LED10.A
- net LED5: now also LED11.A
- net LED6: now also LED12.A
- net N$110: now also LED1.C, LED7.C; no longer LED1.K
- net N$111: now also LED2.C, LED8.C; no longer LED2.K
- net N$112: now also LED3.C, LED9.C; no longer LED3.K
- net N$113: now also LED10.C, LED4.C; no longer LED4.K
- net N$114: now also LED11.C, LED5.C; no longer LED5.K
- net N$115: now also LED12.C, LED6.C; no longer LED6.K
Routing:
- net LED1: track 21.9 -> 26.3 mm, vias 2 -> 3
- net LED2: track 28.4 -> 32.3 mm, vias 0 -> 1
- net LED4: track 35.9 -> 39.5 mm, vias 0 -> 1
- net N$113: track 2.22 -> 5.00 mm, vias 0 -> 1
- net N$115: track 2.22 -> 5.00 mm, vias 0 -> 1
- net N$110: track 2.22 -> 5.00 mm, vias 0 -> 1
- net N$114: track 2.22 -> 5.00 mm, vias 0 -> 1
- net N$112: track 2.22 -> 4.92 mm, vias 0 -> 1
- net LED6: track 50.4 -> 53.0 mm, vias 0 -> 1
- net LED5: track 45.7 -> 48.3 mm, vias 0 -> 1
- net N$111: track 2.22 -> 4.50 mm, vias 0 -> 1
- net LED3: track 33.3 -> 34.8 mm, vias 1 -> 2

Commit message: Update designs + gerbers
Parts:
- removed U7: TXB0108PWR, Texas Instruments_By_element14_Batch_1:SOP65P640X120-20N
- added C92: 100nF, rcl:C0603
- added IC4: GTL2003, manekinen_diy:TSSOP20
- added JP11: (no value), pinhead:1X02
- added R37: 220R, resistor:R0603
- added R38: 100k, resistor:R0603
- added U$11, U$13, U$14, U$15, U$17, U$18: FIDUCIAL, adafruit:FIDUCIAL_1MM
- C67: value 22nF -> 1uF
- moved JP1 42.7 mm to (48.7, 94.5), turned to 90 degrees
- moved C72 5.75 mm to (14.7, 86.4), turned to 180 degrees
- moved C66 3.56 mm to (29.0, 86.1)
- moved JP2 0.87 mm to (154.9, 10.8)
- moved R60 0.33 mm to (132.4, 38.1)
Connections:
- removed net N$49 (its old number): CON6.F22, U$5.8
- new net AVCC: C13.1, C47.1, C48.1, C49.1, C67.1, JP11.1, R43.2, R44.2, R59.1, R60.1, U5.14, U5.18, U5.3, U5.7
- new net N$35: CON6.D22, U$5.20
- new net N$83: C92.1, IC4.19, IC4.20, R38.2
- net +3V3: now also JP11.2, R37.2; no longer C13.1, C47.1, C48.1, C49.1, C67.1, R43.2, R44.2, R59.1, R60.1, U5.14, U5.18, U5.3, U5.7
- net +5V/2: now also R38.1; no longer U7.19
- net GND: now also C92.2, IC4.1, IC4.10, IC4.9; no longer U7.11, U7.8, U7.9
- net LED1: now also R37.1
- net N$32: now also CON6.C22, U$5.21; no longer CON6.F23, U$5.1
- net N$47: now also CON6.F22, U$5.19; no longer CON6.C22, U$5.20
- net N$48: now also CON6.F23, U$5.8; no longer CON6.D22, U$5.19
- net N$87: now also IC4.8; no longer U7.7
- net N$93: now also IC4.2; no longer U7.10, U7.2
- net N$94: now also IC4.7; no longer U7.6
- net N$95: now also IC4.6; no longer U7.5
- net N$96: now also IC4.5; no longer U7.4
- net N$97: now also IC4.4; no longer U7.3
- net N$98: now also IC4.3; no longer U7.1
- net PRG_MISO: now also IC4.14; no longer U7.15
- net PRG_MOSI: now also IC4.15; no longer U7.16
- net PRG_PDIC: now also IC4.17; no longer U7.18
- net PRG_PDID: now also IC4.18; no longer U7.20
- net PRG_RST: now also IC4.13; no longer U7.14
- net PRG_SCK: now also IC4.16; no longer U7.17
Routing:
- net AVCC: track 0.00 -> 53.2 mm
- net +3V3: track 810.9 -> 759.3 mm, vias 14 -> 12
- net N$13: track 8.06 -> 53.8 mm
- net +5V: track 603.0 -> 575.0 mm
- net N$49 (its old number): track 22.6 -> 0.00 mm
- net N$32: track 33.3 -> 17.1 mm, vias 2 -> 0
- net GND: track 282.2 -> 266.6 mm, vias 291 -> 288
- net N$35: track 0.00 -> 11.7 mm
- net N$53: track 22.6 -> 28.3 mm
- net N$83: track 0.00 -> 5.03 mm
- net N$49: track 22.9 -> 27.8 mm
- net N$48: track 14.9 -> 19.0 mm
- net +5V/2: track 78.6 -> 75.4 mm
- net N$54: track 23.1 -> 20.1 mm
- net N$47: track 14.5 -> 11.6 mm
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Other:
- board size 155 x 100.3 mm -> 155 x 100 mm
- board text added: "+"
- board text added: "Armed"
- board text added: "C:/E/eagle/flag.bmp"
- board text added: "Capture"
- board text added: "MiniUSB PWR"
- board text added: "NewAE Technology Inc"
- board text added: "OpenADC Channel 1"
- board text added: "OpenADC Channel 2"
- board text added: "PLL PWR"
- board text added: "REV: 11MAR2014"
- board text added: "STATUS"
- board text added: "TM"
- board text added: "Targ. Act."
- board text added: "Targ. Clock"
- board text added: "USB"
- board text added: "USB-A PWR"
- board text added: "newae.com/sidechannel"
- board text removed: "REV: 17DEC2013"

Commit message: HW:pcbs: updates to latest version (mainly BOM fixes)
Parts:
- removed U$11, U$13, U$14, U$15, U$17, U$18: FIDUCIAL, adafruit:FIDUCIAL_1MM
- added FID1, FID2, FID3, FID4, FID5, FID6: FIDUCIAL, adafruit:FIDUCIAL_1MM
- LED1, LED7: value RED -> GREEN
- LED10, LED11, LED4, LED5: value BLUE -> YELLOW
- LED12, LED6: value GREEN -> YELLOW
- LED2, LED8: value YELLOW -> GREEN
- LED3, LED9: value GREEN -> BLUE
- R31: value 50R -> 100R
- renumbered U$3 to CHANNEL2, U$5 to CHANNEL1
