File: hardware/capture/chipwhisperer-rev2/cwrev2_eagleproj/openadc_ztex.sch (EAGLE design)
At the start: 211 parts, among them CON3 JTAG, CON6 USB-FPGA1.15, IC1 AOZ1021, IC2 AOZ1021, IC3 AOZ1094, IC5 AT90USB162A, T1 TC1-1T, U1 AD9215BRUZ, U2 AD8331, U3 LP3985IM5-3.0, U4 LTC3200ES6, U5 CDCE906PW, U6 TXB0104PWR, U7 TXB0108PWR, U8 SN74LVC1T45DBVT, U9 SN74LVC1T45DBVT, X1 SMA-142-0711-821/826, X2 SMA-142-0711-821/826, X3 SMA-142-0711-821/826, X4 SMA-142-0711-821/826, X5 PN61729-S

Commit message: Fix CWRev2 mistakes
Parts:
- added C88, C89, C90: 100nF, rcl:C-EUC0603
- added C91: (no value), resistor:C-EUC0603
- added JP10: (no value), pinhead:PINHD-1X2
- added R35, R36: 2k2, resistor:R-US_R0603
- added U10: ATSHA204-SH, customs:ATSHA204-SH
- D1: device diode:DIODE-DO214AA -> diode:DIODE-MELF-MLL41
- L3: device inductors:DR1030 -> inductors:DR1030FAKE
Connections:
- removed net VIN: CON6_ABE-PWR.A1~4..35V, CON6_ABE-PWR.B1~4..35V, JP1.1
- new net N$119: JP10.2, U5.S1/A1
- new net N$120: JP10.1, U5.S0/A0/CLK_SEL
- new net N$121: CON6_ABE-FPGA.B28~D6~IO_L3P_0, R36.2, U10.SCL
- new net N$124: CON6_ABE-FPGA.A28~C6~IO_L3N_0, R35.2, U10.SDA
- new net N$125: R32.2, U5.CLK_IN0
- new net N$66: C90.1, JP9.3
- new net N$84: R33.1, U5.CLK_IN1
- net +3V3: now also C91.1, R35.1, R36.1, U10.VCC
- net +5V: now also CON6_ABE-PWR.A1~4..35V, CON6_ABE-PWR.B1~4..35V, JP1.1
- net GND: now also C91.2, U10.GND
- net N$118: now also C88.1; no longer JP9.3, R33.1
- net N$65: now also C89.1; no longer R32.1
- net N$77: now also C89.2, R32.1; no longer R33.2, U5.CLK_IN1
- net N$81: now also C88.2, C90.2, R33.2; no longer R32.2, U5.CLK_IN0
Other:
- note added: "B5"
- moved on the sheet: C47, C49, C67, R32, R33, R43, R44, R45, R46

Commit message: Add missing projects back to GIT
Parts:
- U6: value TXB0104PWR -> TXS0104EPWR
Changed lines of the file:
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@@
 <part name="+3V9" library="supply1" deviceset="+3V3" device=""/>
 <part name="P+4" library="supply1" deviceset="+5V" device=""/>
-<part name="U6" library="Texas Instruments_By_element14_Batch_1" deviceset="TXB0104PWR" device=""/>
+<part name="U6" library="Texas Instruments_By_element14_Batch_1" deviceset="TXB0104PWR" device="" value="TXS0104EPWR"/>
 <part name="SUPPLY16" library="supply2" deviceset="GND" device=""/>
 <part name="U7" library="Texas Instruments_By_element14_Batch_1" deviceset="TXB0108PWR" device=""/>

Commit message: Update #1
Parts:
- added LED10, LED11: BLUE, dp_devices:LED-0805
- added LED12, LED9: GREEN, dp_devices:LED-0805
- added LED7: RED, dp_devices:LED-0805
- added LED8: YELLOW, dp_devices:LED-0805
- LED1, LED2, LED3, LED4, LED5, LED6: device dp_devices:LED-3MM -> dp_devices:LED-0805
Connections:
- net LED1: now also LED7.A
- net LED2: now also LED8.A
- net LED3: now also LED9.A
- net LED4: now also LED10.A
- net LED5: now also LED11.A
- net LED6: now also LED12.A
- net N$110: now also LED7.C
- net N$111: now also LED8.C
- net N$112: now also LED9.C
- net N$113: now also LED10.C
- net N$114: now also LED11.C
- net N$115: now also LED12.C
Other:
- note added: "1.2V/6A"
- moved on the sheet: LED1, LED2, LED3, LED4, LED5, R52, R53, R54, R55, R56

Commit message: Update designs + gerbers
Parts:
- removed U7: TXB0108PWR, Texas Instruments_By_element14_Batch_1:TXB0108PWR
- added C92: 100nF, rcl:C-EUC0603
- added IC4: GTL2003, manekinen_diy:GTL2003
- added JP11: (no value), pinhead:PINHD-1X2
- added R37: 220R, resistor:R-US_R0603
- added R38: 100k, resistor:R-US_R0603
- added U$11, U$13, U$14, U$15, U$17, U$18: FIDUCIAL, adafruit:FIDUCIAL
- C67: value 22nF -> 1uF
Connections:
- removed net N$49 (its old number): CON6_CDF-FPGA.F22~AB11~IO_L31N_GCLK30_D15_2, U$5.ADC6
- new net AVCC: C13.1, C47.1, C48.1, C49.1, C67.1, JP11.1, R43.2, R44.2, R59.1, R60.1, U5.VCC, U5.VCCOUT1, U5.VCCOUT2, U5.VCC_2
- new net N$35: CON6_CDF-FPGA.D22~AB12~IO_L30N_GCLK0_USERCCLK_2, U$5.ADC4
- new net N$83: C92.1, IC4.DREF, IC4.GREF, R38.2
- net +3V3: now also JP11.2, R37.2; no longer C13.1, C47.1, C48.1, C49.1, C67.1, R43.2, R44.2, R59.1, R60.1, U5.VCC, U5.VCCOUT1, U5.VCCOUT2, U5.VCC_2
- net +5V/2: now also R38.1; no longer U7.VCCB
- net GND: now also C92.2, IC4.GND, IC4.S7, IC4.S8; no longer U7.A7, U7.A8, U7.GND
- net LED1: now also R37.1
- net N$32: now also CON6_CDF-FPGA.C22~Y10~IO_L29N_GCLK2_2, U$5.ADC1; no longer CON6_CDF-FPGA.F23~W11~IO_L29P_GCLK3_2, U$5.CLKIN
- net N$47: now also CON6_CDF-FPGA.F22~AB11~IO_L31N_GCLK30_D15_2, U$5.ADC3; no longer CON6_CDF-FPGA.C22~Y10~IO_L29N_GCLK2_2, U$5.ADC4
- net N$48: now also CON6_CDF-FPGA.F23~W11~IO_L29P_GCLK3_2, U$5.ADC6; no longer CON6_CDF-FPGA.D22~AB12~IO_L30N_GCLK0_USERCCLK_2, U$5.ADC3
- net N$87: now also IC4.S6; no longer U7.A6
- net N$93: now also IC4.SREF; no longer U7.OE, U7.VCCA
- net N$94: now also IC4.S5; no longer U7.A5
- net N$95: now also IC4.S4; no longer U7.A4
- net N$96: now also IC4.S3; no longer U7.A3
- net N$97: now also IC4.S2; no longer U7.A2
- net N$98: now also IC4.S1; no longer U7.A1
- net PRG_MISO: now also IC4.D5; no longer U7.B5
- net PRG_MOSI: now also IC4.D4; no longer U7.B4
- net PRG_PDIC: now also IC4.D2; no longer U7.B2
- net PRG_PDID: now also IC4.D1; no longer U7.B1
- net PRG_RST: now also IC4.D6; no longer U7.B6
- net PRG_SCK: now also IC4.D3; no longer U7.B3
Other:
- note added: "M6"
- note added: "M7"
- note added: "M9"
- note added: "N6"
- note added: "N8"
- note added: "N9"
- note added: "P4"
- note added: "P6"
- note added: "P7"
- note added: "P9"
- note added: "R7"
- note added: "R9"
- note added: "T4"
- note added: "T6"
- note added: "T7"
- note added: "T8"
- note added: "T9"

Commit message: HW:pcbs: updates to latest version (mainly BOM fixes)
Parts:
- LED1, LED7: value RED -> GREEN
- LED10, LED11, LED4, LED5: value BLUE -> YELLOW
- LED12, LED6: value GREEN -> YELLOW
- LED2, LED8: value YELLOW -> GREEN
- LED3, LED9: value GREEN -> BLUE
- R31: value 50R -> 100R
- renumbered U$11 to FID1, U$13 to FID6, U$14 to FID2, U$15 to FID5, U$17 to FID3, U$18 to FID4, U$3 to CHANNEL2, U$5 to CHANNEL1
