File: hardware/victims/ztex_multivictim/generic_victim.brd (EAGLE design)
At the start: 123.2 x 84.8 mm, 77 parts, among them CON1 CHIPCARD-SOCKET, IC1 ATMEGA48/88/168-PU, IC3 XMEGA16A4A, Q2 OSC-OSCILLATOR, Q3 OSC-OSCILLATOR, U1 BGA2801, U2 BGA2801, X1 BU-SMA-V, X2 BU-SMA-V, X3 BU-SMA-V, X4 BU-SMA-V

Commit message: Fix a few layout issues in victim
Parts:
- moved R8 0.25 mm to (31.8, 75.4)
Routing:
- net GND: track 436.3 -> 287.2 mm, vias 18 -> 161

Commit message: Various small other changes
Parts:
- added JP25: (no value), pinhead:1X06
- added JP26: (no value), pinhead:1X01
- added LED1: (no value), adafruit:LED3MM
- added R10: 220R, resistor:R0805
- C10, C13, C17, C18, C19, C20, C21, C22, C28, C3, C8: value (none) -> 100nF
- C11: value (none) -> 470nF
- C12, C15, C16: value (none) -> 10nF
- C14, C25, C26, C4, C9: value (none) -> 1uF
- C23, C24: value (none) -> 22nF
- C27: value (none) -> 10uF
- C29, C30: value (none) -> 220uF
- C6, C7: value (none) -> 22pF
- IC3: value XMEGA16A4A -> XMEGA16A4-AU
- L1: value (none) -> 1uH
- R1, R2, R3, R4, R5, R6: value (none) -> 50R
- R7, R8: value (none) -> 100R
- R9: value (none) -> 5R
Connections:
- new net N$41: IC1.24, JP25.1
- new net N$42: IC1.25, JP25.2
- new net N$43: IC1.26, JP25.3
- new net N$44: IC1.27, JP25.4
- new net N$45: IC1.28, JP25.5
- new net N$46: LED1.K, R10.1
- net +3V3: now also LED1.A
- net GND: now also JP25.6, R10.2
- net VMON: now also JP26.1
Routing:
- net N$45: track 0.00 -> 6.10 mm
- net N$44: track 0.00 -> 6.10 mm
- net N$43: track 0.00 -> 6.10 mm
- net N$42: track 0.00 -> 6.10 mm
- net N$41: track 0.00 -> 6.10 mm
- net +3V3: track 320.3 -> 325.7 mm
- net VMON: track 129.5 -> 134.7 mm
- net N$46: track 0.00 -> 1.94 mm
- net GND: vias 161 -> 215
Other:
- board text added: "1"
- board text added: "14/8"
- board text added: "7334L2622F05LF"
- board text added: "ATMega8/48/168/328"
- board text added: "Colin O'Flynn"
- board text added: "DUP."
- board text added: "EXT."
- board text added: "INT."
- board text added: "MOD."
- board text added: "NewAE.com"
- board text added: "XMEGA16A4A"

Commit message: Fixes in PCB.. still more to go
Connections:
- removed net N$9: C8.1, C9.1, JP20.2, JP7.6, R3.1
- new net VREF: C8.1, C9.1, JP20.2, JP7.6, JP9.8, R3.1
- net +3V3: no longer JP9.8
Routing:
- net VREF: track 0.00 -> 69.3 mm, vias 0 -> 1
- net N$9: track 21.1 -> 0.00 mm
- net GND: track 287.2 -> 267.3 mm, vias 215 -> 214
- net +3V3: track 325.7 -> 322.9 mm
Changed lines of the file:
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@@
 <wire x1="74.842" y1="64.682" x2="75.184" y2="65.024" width="1.27" layer="16"/>
 <wire x1="75.184" y1="65.024" x2="79.248" y2="65.024" width="1.27" layer="16"/>
-<wire x1="79.248" y1="65.024" x2="80.772" y2="66.548" width="1.27" layer="16"/>
-<wire x1="80.772" y1="66.548" x2="80.772" y2="69.85" width="1.27" layer="16"/>
-<via x="80.772" y="69.85" extent="1-16" drill="0.7112"/>
-<wire x1="80.772" y1="69.85" x2="80.772" y2="82.804" width="1.27" layer="1"/>
-<wire x1="80.772" y1="82.804" x2="79.756" y2="83.82" width="1.27" layer="1"/>
 <wire x1="79.756" y1="83.82" x2="79.248" y2="83.82" width="1.27" layer="1"/>
 <wire x1="46.228" y1="86.614" x2="46.482" y2="86.868" width="1.27" layer="1"/>
@@
 <contactref element="L1" pad="1"/>
 <contactref element="C29" pad="+"/>
-<contactref element="JP9" pad="8"/>
-<wire x1="76.708" y1="86.36" x2="76.708" y2="86.868" width="1.524" layer="1"/>
-<wire x1="76.708" y1="86.868" x2="76.708" y2="87.376" width="1.524" layer="1"/>
-<wire x1="76.708" y1="87.376" x2="77.978" y2="88.646" width="1.524" layer="1"/>
-<wire x1="77.978" y1="88.646" x2="102.616" y2="88.646" width="1.524" layer="1"/>
 <wire x1="102.616" y1="88.646" x2="107.188" y2="88.646" width="1.524" layer="1"/>
 <wire x1="107.188" y1="88.646" x2="108.966" y2="88.392" width="1.524" layer="1"/>
@@
 <wire x1="58.928" y1="82.296" x2="58.166" y2="81.534" width="1.27" layer="1"/>
 <wire x1="58.166" y1="81.534" x2="46.736" y2="81.534" width="1.27" layer="1"/>
-<wire x1="64.008" y1="86.36" x2="64.008" y2="87.63" width="1.27" layer="1"/>
-<wire x1="64.008" y1="87.63" x2="65.024" y2="88.646" width="1.27" layer="1"/>
-<wire x1="65.024" y1="88.646" x2="74.93" y2="88.646" width="1.27" layer="1"/>
-<wire x1="74.93" y1="88.646" x2="76.708" y2="86.868" width="1.27" layer="1"/>
-<wire x1="64.008" y1="86.36" x2="64.008" y2="87.63" width="1.27" layer="16"/>
-<wire x1="64.008" y1="87.63" x2="62.738" y2="88.9" width="1.27" layer="16"/>
-<wire x1="62.738" y1="88.9" x2="55.118" y2="88.9" width="1.27" layer="16"/>
 <wire x1="55.118" y1="88.9" x2="49.53" y2="83.312" width="1.27" layer="16"/>
 <wire x1="49.53" y1="83.312" x2="46.482" y2="83.312" width="1.27" layer="16"/>
@@
 <wire x1="45.847" y1="74.295" x2="45.604" y2="74.295" width="0.508" layer="1"/>
 <wire x1="45.604" y1="74.295" x2="45.604" y2="79.502" width="0.508" layer="1"/>
+<wire x1="55.118" y1="88.9" x2="75.946" y2="88.9" width="1.27" layer="16"/>
+<wire x1="75.946" y1="88.9" x2="76.581" y2="88.265" width="1.27" layer="16"/>
+<wire x1="76.581" y1="88.265" x2="76.708" y2="88.138" width="1.27" layer="16"/>
+<wire x1="76.708" y1="88.138" x2="76.708" y2="86.36" width="1.27" layer="16"/>
+<wire x1="76.581" y1="88.265" x2="76.962" y2="88.265" width="1.27" layer="16"/>
+<wire x1="76.962" y1="88.265" x2="77.343" y2="88.646" width="1.27" layer="16"/>
+<wire x1="77.343" y1="88.646" x2="102.362" y2="88.646" width="1.27" layer="16"/>
+<wire x1="102.362" y1="88.646" x2="102.616" y2="88.392" width="1.27" layer="16"/>
+<wire x1="102.616" y1="88.392" x2="102.616" y2="87.884" width="1.27" layer="16"/>
+<wire x1="102.616" y1="88.392" x2="102.616" y2="88.646" width="0" layer="19" extent="1-16"/>
 </signal>
 <signal name="N$24">
@@
 <wire x1="45.72" y1="54.102" x2="48.26" y2="54.102" width="0.3048" layer="16"/>
 <wire x1="48.26" y1="54.102" x2="50.8" y2="54.102" width="0.3048" layer="16"/>
-</signal>
-<signal name="N$9">
-<contactref element="JP7" pad="6"/>
-<contactref element="R3" pad="1"/>
-<contactref element="C8" pad="1"/>
-<contactref element="C9" pad="1"/>
-<contactref element="JP20" pad="2"/>
-<wire x1="78.486" y1="56.896" x2="78.486" y2="57.492" width="1.016" layer="16"/>
-<wire x1="78.486" y1="57.492" x2="76.542" y2="59.436" width="1.016" layer="16"/>
-<wire x1="81.026" y1="56.476" x2="78.906" y2="56.476" width="1.016" layer="16"/>
-<wire x1="78.906" y1="56.476" x2="78.486" y2="56.896" width="1.016" layer="16"/>
-<wire x1="86.106" y1="62.23" x2="86.106" y2="60.706" width="1.016" layer="16"/>
-<wire x1="86.106" y1="60.706" x2="84.836" y2="59.436" width="1.016" layer="16"/>
-<wire x1="84.836" y1="59.436" x2="82.042" y2="59.436" width="1.016" layer="16"/>
-<wire x1="82.042" y1="59.436" x2="79.502" y2="61.976" width="1.016" layer="16"/>
-<wire x1="79.502" y1="61.976" x2="76.796" y2="61.976" width="1.016" layer="16"/>
-<wire x1="76.796" y1="61.976" x2="76.542" y2="61.722" width="1.016" layer="16"/>
-<wire x1="76.542" y1="59.436" x2="76.542" y2="61.722" width="1.016" layer="16"/>
 </signal>
 <signal name="N$32">
@@
 <wire x1="48.387" y1="74.295" x2="50.331" y2="74.295" width="0.508" layer="16"/>
 </signal>
+<signal name="VREF">
+<contactref element="JP9" pad="8"/>
+<contactref element="JP7" pad="6"/>
+<contactref element="R3" pad="1"/>
+<contactref element="C8" pad="1"/>
+<contactref element="C9" pad="1"/>
+<contactref element="JP20" pad="2"/>
+<wire x1="78.486" y1="56.896" x2="78.486" y2="57.492" width="1.016" layer="16"/>
+<wire x1="78.486" y1="57.492" x2="76.542" y2="59.436" width="1.016" layer="16"/>
+<wire x1="81.026" y1="56.476" x2="78.906" y2="56.476" width="1.016" layer="16"/>
+<wire x1="78.906" y1="56.476" x2="78.486" y2="56.896" width="1.016" layer="16"/>
+<wire x1="86.106" y1="62.23" x2="86.106" y2="60.706" width="1.016" layer="16"/>
+<wire x1="86.106" y1="60.706" x2="84.836" y2="59.436" width="1.016" layer="16"/>
+<wire x1="84.836" y1="59.436" x2="82.042" y2="59.436" width="1.016" layer="16"/>
+<wire x1="82.042" y1="59.436" x2="79.502" y2="61.976" width="1.016" layer="16"/>
+<wire x1="79.502" y1="61.976" x2="76.796" y2="61.976" width="1.016" layer="16"/>
+<wire x1="76.796" y1="61.976" x2="76.542" y2="61.722" width="1.016" layer="16"/>
+<wire x1="76.542" y1="59.436" x2="76.542" y2="61.722" width="1.016" layer="16"/>
+<wire x1="64.008" y1="86.36" x2="64.008" y2="87.503" width="0.8128" layer="1"/>
+<wire x1="64.008" y1="87.503" x2="65.024" y2="88.519" width="0.8128" layer="1"/>
+<wire x1="65.024" y1="88.519" x2="81.026" y2="88.519" width="0.8128" layer="1"/>
+<wire x1="81.026" y1="88.519" x2="82.169" y2="87.376" width="0.8128" layer="1"/>
+<wire x1="82.169" y1="87.376" x2="82.169" y2="83.82" width="0.8128" layer="1"/>
+<wire x1="82.169" y1="83.82" x2="79.248" y2="80.899" width="0.8128" layer="1"/>
+<wire x1="79.248" y1="80.899" x2="79.248" y2="72.644" width="0.8128" layer="1"/>
+<wire x1="79.248" y1="72.644" x2="81.026" y2="70.866" width="0.8128" layer="1"/>
+<via x="81.026" y="70.866" extent="1-16" drill="0.6"/>
+<wire x1="81.026" y1="70.866" x2="81.026" y2="63.5" width="0.8128" layer="16"/>
+<wire x1="81.026" y1="63.5" x2="79.502" y2="61.976" width="0.8128" layer="16"/>
+</signal>
 </signals>

Commit message: Fix ZTEX generic victim
Parts:
- added C31: 100nF, rcl:C0805
Connections:
- net GND: now also C31.2
- net VREF: now also C31.1
Routing:
- net VREF: track 69.3 -> 71.6 mm
- net +3V3: track 322.9 -> 325.0 mm
Changed lines of the file:
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@@
 <attribute name="VALUE" x="13.081" y="55.626" size="1.27" layer="27"/>
 </element>
+<element name="C31" library="rcl" package="C0805" value="100nF" x="83.693" y="87.249" rot="R270"/>
 </elements>
 <signals>
@@
 <via x="120.396" y="60.706" extent="1-16" drill="0.4318"/>
 <via x="120.396" y="64.008" extent="1-16" drill="0.4318"/>
+<contactref element="C31" pad="2"/>
 </signal>
 <signal name="N$1">
@@
 <wire x1="102.362" y1="88.646" x2="102.616" y2="88.392" width="1.27" layer="16"/>
 <wire x1="102.616" y1="88.392" x2="102.616" y2="87.884" width="1.27" layer="16"/>
-<wire x1="102.616" y1="88.392" x2="102.616" y2="88.646" width="0" layer="19" extent="1-16"/>
+<wire x1="102.616" y1="87.884" x2="102.616" y2="85.852" width="1.27" layer="16"/>
 </signal>
 <signal name="N$24">
@@
 <wire x1="64.008" y1="87.503" x2="65.024" y2="88.519" width="0.8128" layer="1"/>
 <wire x1="65.024" y1="88.519" x2="81.026" y2="88.519" width="0.8128" layer="1"/>
-<wire x1="81.026" y1="88.519" x2="82.169" y2="87.376" width="0.8128" layer="1"/>
+<wire x1="81.026" y1="88.519" x2="81.788" y2="87.757" width="0.8128" layer="1"/>
+<wire x1="81.788" y1="87.757" x2="82.169" y2="87.376" width="0.8128" layer="1"/>
 <wire x1="82.169" y1="87.376" x2="82.169" y2="83.82" width="0.8128" layer="1"/>
 <wire x1="82.169" y1="83.82" x2="79.248" y2="80.899" width="0.8128" layer="1"/>
@@
 <wire x1="81.026" y1="70.866" x2="81.026" y2="63.5" width="0.8128" layer="16"/>
 <wire x1="81.026" y1="63.5" x2="79.502" y2="61.976" width="0.8128" layer="16"/>
+<contactref element="C31" pad="1"/>
+<wire x1="83.693" y1="88.199" x2="81.788" y2="88.199" width="0.6096" layer="1"/>
+<wire x1="81.788" y1="88.199" x2="81.788" y2="87.757" width="0.6096" layer="1"/>
 </signal>
 </signals>

Commit message: Update BOM, load updated PCB files for target
Parts:
- added R11: 10k, resistor:R0805
- added R12: 680R, resistor:R0805
- C1, C2, C5: value (none) -> 100nF
Connections:
- net FPGA3: now also R12.1
- net RESET: now also R11.1
- net VREF: now also R11.2, R12.2
Routing:
- net GND: track 267.3 -> 221.8 mm
Other:
- board text added: "ChipWhisperer.com"
- board text added: "Rev 6JUNE2013"
- board text added: "WARNING:"
- board text added: "You can severly damage this board by setting jumpers wrong. Read manual online before use."
- board text removed: "NewAE.com"

Commit message: Sync latest changes
Parts:
- R12: value 680R -> 68k
Changed lines of the file:
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@@
 <element name="C31" library="rcl" package="C0805" value="100nF" x="83.693" y="87.249" rot="R270"/>
 <element name="R11" library="resistor" package="R0805" value="10k" x="0.635" y="0.889"/>
-<element name="R12" library="resistor" package="R0805" value="680R" x="0.635" y="-4.699"/>
+<element name="R12" library="resistor" package="R0805" value="68k" x="0.635" y="-4.699"/>
 </elements>
 <signals>

Commit message: Updates to PCBs, add new PCBs
Parts:
- R12: value 68k -> 680R
- moved R12 116.5 mm to (95.6, 62.7), flipped to the bottom
- moved R11 111.1 mm to (95.0, 59.6), flipped to the bottom, turned to 180 degrees
Connections:
- net FPGA3: no longer R12.1
- net MISO: now also R12.1
Routing:
- net VREF: track 71.6 -> 86.0 mm, vias 1 -> 3
- net N$16: track 125.5 -> 127.9 mm
- net MISO: track 141.5 -> 142.9 mm
- net RESET: track 108.7 -> 109.5 mm
- net GND: vias 214 -> 213
Other:
- board text added: "Rev 1SEPT2013"
- board text removed: "Rev 6JUNE2013"
Changed lines of the file:
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@@
 <?xml version="1.0" encoding="utf-8"?>
 <!DOCTYPE eagle SYSTEM "eagle.dtd">
-<eagle version="6.4">
+<eagle version="6.5.0">
 <drawing>
 <settings>
@@
 <grid distance="5" unitdist="mil" unit="mm" style="lines" multiple="1" display="no" altdistance="100" altunitdist="mil" altunit="mil"/>
 <layers>
-<layer number="1" name="Top" color="4" fill="1" visible="no" active="yes"/>
+<layer number="1" name="Top" color="4" fill="1" visible="yes" active="yes"/>
 <layer number="2" name="Route2" color="1" fill="3" visible="no" active="no"/>
 <layer number="3" name="Route3" color="4" fill="3" visible="no" active="no"/>
@@
 <layer number="21" name="tPlace" color="7" fill="1" visible="yes" active="yes"/>
 <layer number="22" name="bPlace" color="7" fill="1" visible="yes" active="yes"/>
-<layer number="23" name="tOrigins" color="15" fill="1" visible="no" active="yes"/>
+<layer number="23" name="tOrigins" color="15" fill="1" visible="yes" active="yes"/>
 <layer number="24" name="bOrigins" color="15" fill="1" visible="yes" active="yes"/>
-<layer number="25" name="tNames" color="7" fill="1" visible="no" active="yes"/>
+<layer number="25" name="tNames" color="7" fill="1" visible="yes" active="yes"/>
 <layer number="26" name="bNames" color="7" fill="1" visible="yes" active="yes"/>
 <layer number="27" name="tValues" color="7" fill="1" visible="no" active="yes"/>
@@
 <wire x1="55.626" y1="72.517" x2="55.626" y2="49.784" width="1.016" layer="21"/>
 <text x="110.236" y="39.243" size="2.54" layer="22" font="vector" ratio="16" rot="MR0">ChipWhisperer.com</text>
-<text x="110.236" y="36.576" size="1.778" layer="22" font="vector" ratio="16" rot="MR0">Rev 6JUNE2013</text>
+<text x="110.236" y="36.576" size="1.778" layer="22" font="vector" ratio="16" rot="MR0">Rev 1SEPT2013</text>
 <text x="111.379" y="27.94" size="2.1844" layer="22" font="vector" ratio="16" rot="MR0">WARNING:</text>
 <text x="111.379" y="22.352" size="1.27" layer="22" font="vector" ratio="16" rot="MR0">You can severly damage this board
@@
 </element>
 <element name="C31" library="rcl" package="C0805" value="100nF" x="83.693" y="87.249" rot="R270"/>
-<element name="R11" library="resistor" package="R0805" value="10k" x="0.635" y="0.889"/>
-<element name="R12" library="resistor" package="R0805" value="68k" x="0.635" y="-4.699"/>
+<element name="R11" library="resistor" package="R0805" value="10k" x="94.996" y="59.563" smashed="yes" rot="MR180">
+<attribute name="NAME" x="89.916" y="60.198" size="1.27" layer="26" font="vector" rot="MR180"/>
+<attribute name="VALUE" x="94.234" y="61.849" size="1.27" layer="28" rot="MR180"/>
+</element>
+<element name="R12" library="resistor" package="R0805" value="680R" x="95.631" y="62.738" smashed="yes" rot="MR0">
+<attribute name="NAME" x="93.726" y="62.23" size="1.27" layer="26" font="vector" rot="MR0"/>
+<attribute name="VALUE" x="96.393" y="60.452" size="1.27" layer="28" rot="MR0"/>
+</element>
 </elements>
 <signals>
@@
 <via x="102.997" y="53.721" extent="1-16" drill="0.4318"/>
 <via x="99.822" y="56.007" extent="1-16" drill="0.4318"/>
-<via x="95.377" y="59.563" extent="1-16" drill="0.4318"/>
 <via x="98.298" y="59.563" extent="1-16" drill="0.4318"/>
 <via x="83.185" y="57.15" extent="1-16" drill="0.4318"/>
@@
 <wire x1="93.218" y1="64.262" x2="97.282" y2="64.262" width="0.254" layer="1"/>
 <via x="97.282" y="64.262" extent="1-16" drill="0.4318"/>
-<wire x1="97.282" y1="64.262" x2="97.282" y2="57.15" width="0.254" layer="16"/>
+<wire x1="97.282" y1="64.262" x2="97.282" y2="62.103" width="0.254" layer="16"/>
+<wire x1="97.282" y1="62.103" x2="97.282" y2="57.15" width="0.254" layer="16"/>
 <wire x1="97.282" y1="57.15" x2="97.536" y2="56.896" width="0.254" layer="16"/>
 <wire x1="49.53" y1="20.32" x2="51.054" y2="20.32" width="0.254" layer="16"/>
 <wire x1="51.054" y1="20.32" x2="54.864" y2="24.13" width="0.254" layer="16"/>
 <wire x1="54.864" y1="24.13" x2="96.52" y2="24.13" width="0.254" layer="16"/>
-<wire x1="96.52" y1="24.13" x2="97.282" y2="23.368" width="0.254" layer="16"/>
-<wire x1="97.282" y1="23.368" x2="97.79" y2="22.86" width="0.254" layer="16"/>
+<wire x1="96.52" y1="24.13" x2="97.79" y2="22.86" width="0.254" layer="16"/>
 <via x="97.79" y="22.86" extent="1-16" drill="0.4318"/>
 <wire x1="97.79" y1="22.86" x2="98.298" y2="22.86" width="0.254" layer="1"/>
@@
 <wire x1="96.266" y1="53.086" x2="96.266" y2="55.626" width="0.254" layer="1"/>
 <wire x1="96.266" y1="55.626" x2="97.536" y2="56.896" width="0.254" layer="1"/>
+<contactref element="R12" pad="1"/>
+<wire x1="97.282" y1="62.103" x2="96.481" y2="62.103" width="0.4064" layer="16"/>
+<wire x1="96.481" y1="62.103" x2="96.481" y2="62.738" width="0.4064" layer="16"/>
 </signal>
 <signal name="SCK">
@@
 <wire x1="87.63" y1="72.644" x2="93.472" y2="66.802" width="0.254" layer="1"/>
 <via x="93.472" y="66.802" extent="1-16" drill="0.4318"/>
-<wire x1="93.472" y1="66.802" x2="93.472" y2="58.42" width="0.254" layer="16"/>
+<wire x1="93.472" y1="66.802" x2="93.472" y2="59.436" width="0.254" layer="16"/>
+<wire x1="93.472" y1="59.436" x2="93.472" y2="58.42" width="0.254" layer="16"/>
 <wire x1="93.472" y1="58.42" x2="94.996" y2="56.896" width="0.254" layer="16"/>
 <wire x1="41.91" y1="45.72" x2="41.91" y2="70.104" width="0.254" layer="16"/>
@@
 <wire x1="54.864" y1="71.628" x2="56.134" y2="72.898" width="0.254" layer="16"/>
 <contactref element="R11" pad="1"/>
-<wire x1="-0.215" y1="0.889" x2="41.91" y2="45.72" width="0" layer="19" extent="1-1"/>
+<wire x1="93.472" y1="59.436" x2="94.146" y2="59.436" width="0.254" layer="16"/>
+<wire x1="94.146" y1="59.436" x2="94.146" y2="59.563" width="0.254" layer="16"/>
 </signal>
 <signal name="TRIG">
@@
 <wire x1="73.914" y1="66.548" x2="85.09" y2="66.548" width="0.254" layer="1"/>
 <wire x1="85.09" y1="66.548" x2="87.376" y2="64.262" width="0.254" layer="1"/>
-<wire x1="87.376" y1="64.262" x2="87.376" y2="59.944" width="0.254" layer="1"/>
-<wire x1="87.376" y1="59.944" x2="88.392" y2="58.928" width="0.254" layer="1"/>
-<wire x1="88.392" y1="58.928" x2="90.932" y2="58.928" width="0.254" layer="1"/>
+<wire x1="87.376" y1="64.262" x2="87.376" y2="57.912" width="0.254" layer="1"/>
 <wire x1="90.932" y1="58.928" x2="91.186" y2="58.674" width="0.254" layer="1"/>
 <wire x1="91.186" y1="58.674" x2="91.186" y2="55.626" width="0.254" layer="1"/>
 <wire x1="91.186" y1="55.626" x2="92.456" y2="54.356" width="0.254" layer="1"/>
+<wire x1="90.932" y1="58.928" x2="89.662" y2="58.928" width="0.254" layer="1"/>
+<wire x1="89.662" y1="58.928" x2="88.265" y2="57.531" width="0.254" layer="1"/>
+<wire x1="88.265" y1="57.531" x2="87.757" y2="57.531" width="0.254" layer="1"/>
+<wire x1="87.757" y1="57.531" x2="87.376" y2="57.912" width="0.254" layer="1"/>
 </signal>
 <signal name="N$13">
@@
 <wire x1="101.346" y1="58.166" x2="102.362" y2="58.166" width="0.254" layer="16"/>
 <wire x1="102.362" y1="58.166" x2="102.616" y2="58.42" width="0.254" layer="16"/>
-<contactref element="R12" pad="1"/>
-<wire x1="-0.215" y1="-4.699" x2="86.89" y2="10" width="0" layer="19" extent="1-1"/>
 </signal>
 <signal name="N$18">
@@
 <wire x1="78.906" y1="56.476" x2="78.486" y2="56.896" width="1.016" layer="16"/>
 <wire x1="86.106" y1="62.23" x2="86.106" y2="60.706" width="1.016" layer="16"/>
-<wire x1="86.106" y1="60.706" x2="84.836" y2="59.436" width="1.016" layer="16"/>
+<wire x1="86.106" y1="60.706" x2="85.979" y2="60.579" width="1.016" layer="16"/>
+<wire x1="85.979" y1="60.579" x2="84.836" y2="59.436" width="1.016" layer="16"/>
 <wire x1="84.836" y1="59.436" x2="82.042" y2="59.436" width="1.016" layer="16"/>
 <wire x1="82.042" y1="59.436" x2="79.502" y2="61.976" width="1.016" layer="16"/>
@@
 <contactref element="R11" pad="2"/>
 <contactref element="R12" pad="2"/>
-<wire x1="1.485" y1="0.889" x2="76.542" y2="59.436" width="0" layer="19" extent="1-16"/>
-<wire x1="1.485" y1="-4.699" x2="1.485" y2="0.889" width="0" layer="19" extent="1-1"/>
+<wire x1="95.846" y1="59.563" x2="95.758" y2="59.563" width="0.254" layer="16"/>
+<wire x1="95.758" y1="59.563" x2="95.758" y2="60.452" width="0.254" layer="16"/>
+<wire x1="95.758" y1="60.452" x2="94.781" y2="61.214" width="0.254" layer="16"/>
+<wire x1="94.781" y1="61.214" x2="94.781" y2="62.738" width="0.254" layer="16"/>
+<wire x1="85.979" y1="60.579" x2="86.741" y2="60.579" width="0.254" layer="16"/>
+<wire x1="86.741" y1="60.579" x2="88.392" y2="58.928" width="0.254" layer="16"/>
+<via x="88.392" y="58.928" extent="1-16" drill="0.4318"/>
+<wire x1="88.392" y1="58.928" x2="88.392" y2="59.182" width="0.254" layer="1"/>
+<wire x1="88.392" y1="59.182" x2="89.281" y2="60.071" width="0.254" layer="1"/>
+<wire x1="89.281" y1="60.071" x2="93.638" y2="60.071" width="0.254" layer="1"/>
+<wire x1="93.638" y1="60.071" x2="94.781" y2="61.214" width="0.254" layer="1"/>
+<via x="94.781" y="61.214" extent="1-16" drill="0.4318"/>
 </signal>
 </signals>

Commit message: Update designs + gerbers
Parts:
- added JP27, JP28: (no value), pinhead:1X02
- added TP1, TP2, TP3: PTR1PAD1-13, testpad:P1-13
- added U$1, U$2, U$3, U$4, U$5, U$6: FIDUCIAL, adafruit:FIDUCIAL_1MM
- moved C1 2.26 mm to (52.9, 26.9)
- moved C4 2.26 mm to (55.6, 26.9)
Connections:
- new net N$47: IC1.23, JP28.2
- new net N$9: IC1.14, JP27.1
- net FPGAIN: now also JP27.2
- net GND: now also TP1.TP, TP2.TP, TP3.TP
- net TRIG: now also JP28.1; no longer IC1.23
Routing:
- net FPGAIN: track 66.4 -> 131.8 mm
- net N$47: track 0.00 -> 6.39 mm
- net N$9: track 0.00 -> 4.41 mm
- net TRIG: track 158.9 -> 155.2 mm, vias 7 -> 5
- net GND: track 221.8 -> 218.4 mm, vias 213 -> 217
- net VCCIO: track 189.8 -> 191.6 mm
Other:
- board text added: "2"
- board text added: "3"
- board text added: "3.3V"
- board text added: "4"
- board text added: "5"
- board text added: "ATMegaXX8"
- board text added: "CLKO"
- board text added: "IO VREF"
- board text added: "PC.0"
- board text added: "PORTC"
- board text added: "Rev 10MAR2014"
- board text removed: "Colin O'Flynn"
- board text removed: "INT."
- board text removed: "Rev 1SEPT2013"
