File: hardware/victims/ztex_multivictim/generic_victim.sch (EAGLE design)
At the start: 77 parts, among them CON1 CHIPCARD-SOCKET, IC1 ATMEGA48/88/168-PU, IC3 XMEGA16A4A, Q2 OSC-OSCILLATOR, Q3 OSC-OSCILLATOR, U1 BGA2801, U2 BGA2801, X1 BU-SMA-V, X2 BU-SMA-V, X3 BU-SMA-V, X4 BU-SMA-V

Commit message: Various small other changes
Parts:
- added JP25: (no value), pinhead:PINHD-1X6
- added JP26: (no value), pinhead:PINHD-1X1
- added LED1: (no value), adafruit:LED3MM
- added R10: 220R, resistor:R-US_R0805
- C10, C13, C17, C18, C19, C20, C21, C22, C28, C3, C8: value (none) -> 100nF
- C11: value (none) -> 470nF
- C12, C15, C16: value (none) -> 10nF
- C14, C25, C26, C4, C9: value (none) -> 1uF
- C23, C24: value (none) -> 22nF
- C27: value (none) -> 10uF
- C29, C30: value (none) -> 220uF
- C6, C7: value (none) -> 22pF
- IC3: value XMEGA16A4A -> XMEGA16A4-AU
- L1: value (none) -> 1uH
- R1, R2, R3, R4, R5, R6: value (none) -> 50R
- R7, R8: value (none) -> 100R
- R9: value (none) -> 5R
Connections:
- new net N$41: IC1.PC1(ADC1/PCINT9), JP25.1
- new net N$42: IC1.PC2(ADC2/PCINT10), JP25.2
- new net N$43: IC1.PC3(ADC3/PCINT11), JP25.3
- new net N$44: IC1.PC4(ADC4/SDA/PCINT12), JP25.4
- new net N$45: IC1.PC5(ADC5/SCLPCINT13), JP25.5
- new net N$46: LED1.C, R10.1
- net +3V3: now also LED1.A
- net GND: now also JP25.6, R10.2
- net VMON: now also JP26.1

Commit message: Fixes in PCB.. still more to go
Connections:
- removed net N$9: C8.1, C9.1, JP20.2, JP7.6, R3.1
- new net VREF: C8.1, C9.1, JP20.2, JP7.6, JP9.8, R3.1
- net +3V3: no longer JP9.8
Changed lines of the file:
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@@
 <wire x1="124.46" y1="93.98" x2="129.54" y2="93.98" width="0.1524" layer="91"/>
 <wire x1="129.54" y1="93.98" x2="129.54" y2="99.06" width="0.1524" layer="91"/>
-<pinref part="JP9" gate="A" pin="8"/>
-<wire x1="114.3" y1="119.38" x2="121.92" y2="119.38" width="0.1524" layer="91"/>
-<wire x1="121.92" y1="119.38" x2="121.92" y2="106.68" width="0.1524" layer="91"/>
-<junction x="121.92" y="106.68"/>
 <pinref part="LED1" gate="G$1" pin="A"/>
 <wire x1="124.46" y1="86.36" x2="124.46" y2="93.98" width="0.1524" layer="91"/>
@@
 <wire x1="198.12" y1="137.16" x2="175.26" y2="137.16" width="0.1524" layer="91"/>
 <label x="175.26" y="137.16" size="1.778" layer="95" rot="R180" xref="yes"/>
+</segment>
+</net>
+<net name="VREF" class="0">
+<segment>
+<pinref part="JP9" gate="A" pin="8"/>
+<wire x1="114.3" y1="119.38" x2="124.46" y2="119.38" width="0.1524" layer="91"/>
+<label x="124.46" y="119.38" size="1.778" layer="95" xref="yes"/>
 </segment>
 </net>
@@
 </segment>
 </net>
-<net name="N$9" class="0">
+<net name="VREF" class="0">
 <segment>
 <pinref part="JP7" gate="A" pin="6"/>
@@
 <pinref part="JP20" gate="A" pin="2"/>
 <wire x1="43.18" y1="139.7" x2="43.18" y2="147.32" width="0.1524" layer="91"/>
-</segment>
-</net>
+<wire x1="50.8" y1="139.7" x2="63.5" y2="139.7" width="0.1524" layer="91"/>
+<junction x="50.8" y="139.7"/>
+<label x="63.5" y="139.7" size="1.778" layer="95" xref="yes"/>
+</segment>
+</net>

Commit message: Fix ZTEX generic victim
Parts:
- added C31: 100nF, rcl:C-EUC0805
Connections:
- net GND: now also C31.2
- net VREF: now also C31.1
Changed lines of the file:
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@@
 <part name="R10" library="resistor" deviceset="R-US_" device="R0805" value="220R"/>
 <part name="JP26" library="pinhead" deviceset="PINHD-1X1" device=""/>
+<part name="SUPPLY35" library="supply2" deviceset="GND" device=""/>
+<part name="C31" library="rcl" deviceset="C-EU" device="C0805" value="100nF"/>
 </parts>
 <sheets>
@@
 <instance part="R10" gate="G$1" x="129.54" y="78.74"/>
 <instance part="JP26" gate="G$1" x="200.66" y="137.16"/>
+<instance part="SUPPLY35" gate="GND" x="182.88" y="149.86"/>
+<instance part="C31" gate="G$1" x="182.88" y="157.48"/>
 </instances>
 <busses>
@@
 <pinref part="SUPPLY33" gate="GND" pin="GND"/>
 </segment>
+<segment>
+<pinref part="C31" gate="G$1" pin="2"/>
+<pinref part="SUPPLY35" gate="GND" pin="GND"/>
+</segment>
 </net>
 <net name="N$6" class="0">
@@
 <label x="124.46" y="119.38" size="1.778" layer="95" xref="yes"/>
 </segment>
-</net>
+<segment>
+<pinref part="C31" gate="G$1" pin="1"/>
+<wire x1="182.88" y1="160.02" x2="182.88" y2="165.1" width="0.1524" layer="91"/>
+<wire x1="182.88" y1="165.1" x2="172.72" y2="165.1" width="0.1524" layer="91"/>
+<label x="172.72" y="165.1" size="1.778" layer="95" rot="R180" xref="yes"/>
+</segment>
+</net>

Commit message: Update BOM, load updated PCB files for target
Parts:
- added R11: 10k, resistor:R-US_R0805
- added R12: 680R, resistor:R-US_R0805
- C1, C2, C5: value (none) -> 100nF
Connections:
- net FPGA3: now also R12.1
- net RESET: now also R11.1
- net VREF: now also R11.2, R12.2
Changed lines of the file:
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@@
 <part name="IC1" library="atmega8" deviceset="ATMEGA48/88/168-PU" device=""/>
 <part name="SUPPLY1" library="supply2" deviceset="GND" device=""/>
-<part name="C1" library="resistor" deviceset="C-EU" device="C0805"/>
-<part name="C2" library="resistor" deviceset="C-EU" device="C0805"/>
+<part name="C1" library="resistor" deviceset="C-EU" device="C0805" value="100nF"/>
+<part name="C2" library="resistor" deviceset="C-EU" device="C0805" value="100nF"/>
 <part name="R1" library="resistor" deviceset="R-US_" device="R0805" value="50R"/>
 <part name="R2" library="resistor" deviceset="R-US_" device="R0805" value="50R"/>
@@
 <part name="IC2" library="ic-package" deviceset="DIL14" device="S"/>
 <part name="SUPPLY5" library="supply2" deviceset="GND" device=""/>
-<part name="C5" library="resistor" deviceset="C-EU" device="C0805"/>
+<part name="C5" library="resistor" deviceset="C-EU" device="C0805" value="100nF"/>
 <part name="Q1" library="crystal" deviceset="CRYSTAL" device="HC49U70"/>
 <part name="C6" library="resistor" deviceset="C-EU" device="C0805" value="22pF"/>
@@
 <part name="SUPPLY35" library="supply2" deviceset="GND" device=""/>
 <part name="C31" library="rcl" deviceset="C-EU" device="C0805" value="100nF"/>
+<part name="R11" library="resistor" deviceset="R-US_" device="R0805" value="10k"/>
+<part name="R12" library="resistor" deviceset="R-US_" device="R0805" value="680R"/>
 </parts>
 <sheets>
@@
 <instance part="JP22" gate="A" x="152.4" y="71.12"/>
 <instance part="JP23" gate="A" x="182.88" y="93.98"/>
+<instance part="R11" gate="G$1" x="116.84" y="55.88"/>
+<instance part="R12" gate="G$1" x="116.84" y="48.26"/>
 </instances>
 <busses>
@@
 <segment>
 <pinref part="JP8" gate="A" pin="6"/>
-<wire x1="101.6" y1="66.04" x2="114.3" y2="66.04" width="0.1524" layer="91"/>
+<wire x1="101.6" y1="66.04" x2="109.22" y2="66.04" width="0.1524" layer="91"/>
 <label x="114.3" y="66.04" size="1.778" layer="95" xref="yes"/>
+<pinref part="R11" gate="G$1" pin="1"/>
+<wire x1="109.22" y1="66.04" x2="114.3" y2="66.04" width="0.1524" layer="91"/>
+<wire x1="111.76" y1="55.88" x2="109.22" y2="55.88" width="0.1524" layer="91"/>
+<wire x1="109.22" y1="55.88" x2="109.22" y2="66.04" width="0.1524" layer="91"/>
+<junction x="109.22" y="66.04"/>
 </segment>
 </net>
@@
 <pinref part="JP23" gate="A" pin="1"/>
 <wire x1="167.64" y1="96.52" x2="180.34" y2="96.52" width="0.1524" layer="91"/>
+<pinref part="R12" gate="G$1" pin="1"/>
+<wire x1="111.76" y1="48.26" x2="83.82" y2="48.26" width="0.1524" layer="91"/>
+<wire x1="83.82" y1="48.26" x2="83.82" y2="63.5" width="0.1524" layer="91"/>
+<junction x="83.82" y="63.5"/>
 </segment>
 </net>
@@
 <junction x="50.8" y="139.7"/>
 <label x="63.5" y="139.7" size="1.778" layer="95" xref="yes"/>
-</segment>
-</net>
+<pinref part="R11" gate="G$1" pin="2"/>
+<wire x1="121.92" y1="55.88" x2="124.46" y2="55.88" width="0.1524" layer="91"/>
+<wire x1="124.46" y1="55.88" x2="124.46" y2="50.8" width="0.1524" layer="91"/>
+<pinref part="R12" gate="G$1" pin="2"/>
+<wire x1="124.46" y1="50.8" x2="124.46" y2="48.26" width="0.1524" layer="91"/>
+<wire x1="124.46" y1="48.26" x2="121.92" y2="48.26" width="0.1524" layer="91"/>
+<wire x1="124.46" y1="50.8" x2="132.08" y2="50.8" width="0.1524" layer="91"/>
+<wire x1="132.08" y1="50.8" x2="132.08" y2="43.18" width="0.1524" layer="91"/>
+<junction x="124.46" y="50.8"/>
+<wire x1="132.08" y1="43.18" x2="12.7" y2="43.18" width="0.1524" layer="91"/>
+<wire x1="12.7" y1="43.18" x2="12.7" y2="139.7" width="0.1524" layer="91"/>
+<wire x1="12.7" y1="139.7" x2="35.56" y2="139.7" width="0.1524" layer="91"/>
+<junction x="35.56" y="139.7"/>
+</segment>
+</net>

Commit message: Sync latest changes
Parts:
- R12: value 680R -> 68k
Changed lines of the file:
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@@
 <part name="C31" library="rcl" deviceset="C-EU" device="C0805" value="100nF"/>
 <part name="R11" library="resistor" deviceset="R-US_" device="R0805" value="10k"/>
-<part name="R12" library="resistor" deviceset="R-US_" device="R0805" value="680R"/>
+<part name="R12" library="resistor" deviceset="R-US_" device="R0805" value="68k"/>
 </parts>
 <sheets>

Commit message: Updates to PCBs, add new PCBs
Parts:
- R12: value 68k -> 680R
Connections:
- net FPGA3: no longer R12.1
- net MISO: now also R12.1
Changed lines of the file:
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@@
 <?xml version="1.0" encoding="utf-8"?>
 <!DOCTYPE eagle SYSTEM "eagle.dtd">
-<eagle version="6.4">
+<eagle version="6.5.0">
 <drawing>
 <settings>
@@
 <part name="C31" library="rcl" deviceset="C-EU" device="C0805" value="100nF"/>
 <part name="R11" library="resistor" deviceset="R-US_" device="R0805" value="10k"/>
-<part name="R12" library="resistor" deviceset="R-US_" device="R0805" value="68k"/>
+<part name="R12" library="resistor" deviceset="R-US_" device="R0805" value="680R"/>
 </parts>
 <sheets>
@@
 <pinref part="JP23" gate="A" pin="1"/>
 <wire x1="167.64" y1="96.52" x2="180.34" y2="96.52" width="0.1524" layer="91"/>
+</segment>
+</net>
+<net name="MISO" class="0">
+<segment>
+<pinref part="JP8" gate="A" pin="8"/>
+<wire x1="101.6" y1="63.5" x2="106.68" y2="63.5" width="0.1524" layer="91"/>
+<label x="114.3" y="63.5" size="1.778" layer="95" xref="yes"/>
 <pinref part="R12" gate="G$1" pin="1"/>
-<wire x1="111.76" y1="48.26" x2="83.82" y2="48.26" width="0.1524" layer="91"/>
-<wire x1="83.82" y1="48.26" x2="83.82" y2="63.5" width="0.1524" layer="91"/>
-<junction x="83.82" y="63.5"/>
-</segment>
-</net>
-<net name="MISO" class="0">
-<segment>
-<pinref part="JP8" gate="A" pin="8"/>
-<wire x1="101.6" y1="63.5" x2="114.3" y2="63.5" width="0.1524" layer="91"/>
-<label x="114.3" y="63.5" size="1.778" layer="95" xref="yes"/>
-</segment>
-</net>
+<wire x1="106.68" y1="63.5" x2="114.3" y2="63.5" width="0.1524" layer="91"/>
+<wire x1="111.76" y1="48.26" x2="106.68" y2="48.26" width="0.1524" layer="91"/>
+<wire x1="106.68" y1="48.26" x2="106.68" y2="63.5" width="0.1524" layer="91"/>
+<junction x="106.68" y="63.5"/>
+</segment>
+</net>

Commit message: Update designs + gerbers
Parts:
- added JP27, JP28: (no value), pinhead:PINHD-1X2
- added TP1, TP2, TP3: PTR1PAD1-13, testpad:PTR1PAD1-13
- added U$1, U$2, U$3, U$4, U$5, U$6: FIDUCIAL, adafruit:FIDUCIAL
Connections:
- new net N$47: IC1.PC0(ADC0/PCINT8), JP28.2
- new net N$9: IC1.PB0(ICP1/CLKO/PCINT0), JP27.1
- net FPGAIN: now also JP27.2
- net GND: now also TP1.TP, TP2.TP, TP3.TP
- net TRIG: now also JP28.1; no longer IC1.PC0(ADC0/PCINT8)
Changed lines of the file:
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@@
 <part name="R11" library="resistor" deviceset="R-US_" device="R0805" value="10k"/>
 <part name="R12" library="resistor" deviceset="R-US_" device="R0805" value="680R"/>
+<part name="TP1" library="testpad" deviceset="PTR1" device="PAD1-13"/>
+<part name="TP2" library="testpad" deviceset="PTR1" device="PAD1-13"/>
+<part name="TP3" library="testpad" deviceset="PTR1" device="PAD1-13"/>
+<part name="SUPPLY36" library="supply2" deviceset="GND" device=""/>
+<part name="SUPPLY37" library="supply2" deviceset="GND" device=""/>
+<part name="SUPPLY38" library="supply2" deviceset="GND" device=""/>
+<part name="JP27" library="pinhead" deviceset="PINHD-1X2" device=""/>
+<part name="U$1" library="adafruit" deviceset="FIDUCIAL" device=""/>
+<part name="U$2" library="adafruit" deviceset="FIDUCIAL" device=""/>
+<part name="U$3" library="adafruit" deviceset="FIDUCIAL" device=""/>
+<part name="U$4" library="adafruit" deviceset="FIDUCIAL" device=""/>
+<part name="U$5" library="adafruit" deviceset="FIDUCIAL" device=""/>
+<part name="U$6" library="adafruit" deviceset="FIDUCIAL" device=""/>
+<part name="JP28" library="pinhead" deviceset="PINHD-1X2" device=""/>
 </parts>
 <sheets>
@@
 <instance part="JP25" gate="A" x="175.26" y="119.38"/>
 <instance part="SUPPLY34" gate="GND" x="167.64" y="111.76"/>
+<instance part="JP27" gate="G$1" x="190.5" y="88.9" rot="R90"/>
+<instance part="JP28" gate="G$1" x="187.96" y="127" rot="R270"/>
 </instances>
 <busses>
@@
 <net name="TRIG" class="0">
 <segment>
-<pinref part="IC1" gate="1" pin="PC0(ADC0/PCINT8)"/>
-<wire x1="167.64" y1="129.54" x2="185.42" y2="129.54" width="0.1524" layer="91"/>
-<label x="185.42" y="129.54" size="1.778" layer="95" xref="yes"/>
+<label x="200.66" y="129.54" size="1.778" layer="95" xref="yes"/>
+<pinref part="JP28" gate="G$1" pin="1"/>
+<wire x1="190.5" y1="129.54" x2="200.66" y2="129.54" width="0.1524" layer="91"/>
 </segment>
 </net>
@@
 <segment>
 <pinref part="JP4" gate="A" pin="5"/>
-<wire x1="96.52" y1="152.4" x2="106.68" y2="152.4" width="0.1524" layer="91"/>
+<wire x1="96.52" y1="152.4" x2="101.6" y2="152.4" width="0.1524" layer="91"/>
 <label x="106.68" y="152.4" size="1.778" layer="95" xref="yes"/>
+<pinref part="JP27" gate="G$1" pin="2"/>
+<wire x1="101.6" y1="152.4" x2="106.68" y2="152.4" width="0.1524" layer="91"/>
+<wire x1="190.5" y1="86.36" x2="190.5" y2="83.82" width="0.1524" layer="91"/>
+<wire x1="190.5" y1="83.82" x2="231.14" y2="83.82" width="0.1524" layer="91"/>
+<wire x1="231.14" y1="83.82" x2="231.14" y2="160.02" width="0.1524" layer="91"/>
+<wire x1="231.14" y1="160.02" x2="101.6" y2="160.02" width="0.1524" layer="91"/>
+<wire x1="101.6" y1="160.02" x2="101.6" y2="152.4" width="0.1524" layer="91"/>
+<junction x="101.6" y="152.4"/>
 </segment>
 </net>
@@
 <pinref part="JP25" gate="A" pin="5"/>
 <wire x1="172.72" y1="116.84" x2="167.64" y2="116.84" width="0.1524" layer="91"/>
+</segment>
+</net>
+<net name="N$9" class="0">
+<segment>
+<pinref part="IC1" gate="1" pin="PB0(ICP1/CLKO/PCINT0)"/>
+<pinref part="JP27" gate="G$1" pin="1"/>
+<wire x1="167.64" y1="83.82" x2="187.96" y2="83.82" width="0.1524" layer="91"/>
+<wire x1="187.96" y1="83.82" x2="187.96" y2="86.36" width="0.1524" layer="91"/>
+</segment>
+</net>
+<net name="N$47" class="0">
+<segment>
+<pinref part="JP28" gate="G$1" pin="2"/>
+<pinref part="IC1" gate="1" pin="PC0(ADC0/PCINT8)"/>
+<wire x1="187.96" y1="129.54" x2="167.64" y2="129.54" width="0.1524" layer="91"/>
 </segment>
 </net>
@@
 <instance part="SUPPLY35" gate="GND" x="182.88" y="149.86"/>
 <instance part="C31" gate="G$1" x="182.88" y="157.48"/>
+<instance part="TP1" gate="G$1" x="40.64" y="86.36" rot="R180"/>
+<instance part="TP2" gate="G$1" x="48.26" y="86.36" rot="R180"/>
+<instance part="TP3" gate="G$1" x="55.88" y="86.36" rot="R180"/>
+<instance part="SUPPLY36" gate="GND" x="40.64" y="81.28"/>
+<instance part="SUPPLY37" gate="GND" x="48.26" y="81.28"/>
+<instance part="SUPPLY38" gate="GND" x="55.88" y="81.28"/>
+<instance part="U$1" gate="G$1" x="15.24" y="45.72"/>
+<instance part="U$2" gate="G$1" x="22.86" y="45.72"/>
+<instance part="U$3" gate="G$1" x="30.48" y="45.72"/>
+<instance part="U$4" gate="G$1" x="15.24" y="38.1"/>
+<instance part="U$5" gate="G$1" x="22.86" y="38.1"/>
+<instance part="U$6" gate="G$1" x="30.48" y="38.1"/>
 </instances>
 <busses>
@@
 <pinref part="SUPPLY35" gate="GND" pin="GND"/>
 </segment>
-</net>
+<segment>
+<pinref part="TP1" gate="G$1" pin="TP"/>
+<pinref part="SUPPLY36" gate="GND" pin="GND"/>
+</segment>
+<segment>
+<pinref part="SUPPLY38" gate="GND" pin="GND"/>
+<pinref part="TP3" gate="G$1" pin="TP"/>
+</segment>
+<segment>
+<pinref part="SUPPLY37" gate="GND" pin="GND"/>
+<pinref part="TP2" gate="G$1" pin="TP"/>
+</segment>
+</net>
