File: hardware/victims/ztex_multivictim/smartcard/smartcard.brd (EAGLE design)
At the start: 85.6 x 54 mm, 11 parts

Commit message: HW: Update SASEBO-W Adapter
Parts:
- moved E$3 3.81 mm to (74.1, 35.0)
Routing:
- net S$1: track 76.0 -> 135.0 mm
- net S$2: track 60.8 -> 65.9 mm
Other:
- board size 85.6 x 54 mm -> 85.6 x 53.6 mm
- board text added: "CLK"
- board text added: "RST"
- board text added: "SASEBO-W Adapter"
Changed lines of the file:
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@@
 <?xml version="1.0" encoding="utf-8"?>
 <!DOCTYPE eagle SYSTEM "eagle.dtd">
-<eagle version="6.5.0">
+<eagle version="6.6.0">
 <drawing>
 <settings>
@@
 <grid distance="0.635" unitdist="mm" unit="mm" style="lines" multiple="1" display="no" altdistance="0.025" altunitdist="inch" altunit="inch"/>
 <layers>
-<layer number="1" name="Top" color="4" fill="1" visible="yes" active="yes"/>
+<layer number="1" name="Top" color="4" fill="1" visible="no" active="yes"/>
 <layer number="2" name="Route2" color="1" fill="3" visible="no" active="no"/>
 <layer number="3" name="Route3" color="4" fill="3" visible="no" active="no"/>
@@
 <layer number="23" name="tOrigins" color="15" fill="1" visible="yes" active="yes"/>
 <layer number="24" name="bOrigins" color="15" fill="1" visible="yes" active="yes"/>
-<layer number="25" name="tNames" color="7" fill="1" visible="yes" active="yes"/>
-<layer number="26" name="bNames" color="7" fill="1" visible="yes" active="yes"/>
+<layer number="25" name="tNames" color="7" fill="1" visible="no" active="yes"/>
+<layer number="26" name="bNames" color="7" fill="1" visible="no" active="yes"/>
 <layer number="27" name="tValues" color="7" fill="1" visible="no" active="yes"/>
 <layer number="28" name="bValues" color="7" fill="1" visible="no" active="yes"/>
@@
 <wire x1="83.82" y1="36.83" x2="78.105" y2="36.83" width="1.016" layer="22"/>
 <wire x1="78.105" y1="36.195" x2="78.105" y2="36.83" width="1.016" layer="22"/>
+<text x="69.85" y="37.465" size="1.016" layer="22" font="vector" ratio="16" rot="MR0">VCC</text>
+<text x="69.85" y="40.005" size="1.016" layer="22" font="vector" ratio="16" rot="MR0">RST</text>
+<text x="69.85" y="29.21" size="1.016" layer="22" font="vector" ratio="16" rot="MR0">I/O</text>
+<text x="69.85" y="26.67" size="1.016" layer="22" font="vector" ratio="16" rot="MR0">AUX2</text>
+<text x="69.85" y="23.495" size="1.016" layer="22" font="vector" ratio="16" rot="MR0">AUX1</text>
+<text x="69.85" y="19.685" size="1.016" layer="22" font="vector" ratio="16" rot="MR0">CLK</text>
+<text x="55.88" y="10.795" size="1.27" layer="21" font="vector" ratio="16">SASEBO-W Adapter</text>
+<text x="66.675" y="19.685" size="1.016" layer="21" font="vector" ratio="16">CLK</text>
+<text x="66.675" y="23.495" size="1.016" layer="21" font="vector" ratio="16">AUX1</text>
+<text x="66.675" y="26.67" size="1.016" layer="21" font="vector" ratio="16">AUX2</text>
+<text x="66.675" y="29.21" size="1.016" layer="21" font="vector" ratio="16">I/O</text>
+<text x="66.675" y="37.465" size="1.016" layer="21" font="vector" ratio="16">VCC</text>
+<text x="66.675" y="40.005" size="1.016" layer="21" font="vector" ratio="16">RST</text>
 </plain>
 <attributes>
@@
 <param name="mlMinCreamFrame" value="0mil"/>
 <param name="mlMaxCreamFrame" value="0mil"/>
-<param name="mlViaStopLimit" value="0mil"/>
+<param name="mlViaStopLimit" value="50mil"/>
 <param name="srRoundness" value="0"/>
 <param name="srMinRoundness" value="0mil"/>
@@
 <attribute name="VALUE" x="76.835" y="26.035" size="1.27" layer="28" rot="MR90"/>
 </element>
-<element name="E$3" library="SparkFun" package="SJ-NC" value="" x="77.935" y="35" smashed="yes" rot="MR0">
-<attribute name="NAME" x="80.475" y="36.27" size="0.4064" layer="26" ratio="10" rot="MR0"/>
-<attribute name="VALUE" x="77.935" y="36.27" size="0.4064" layer="28" rot="MR0"/>
+<element name="E$3" library="SparkFun" package="SJ-NC" value="" x="74.125" y="35" smashed="yes" rot="MR0">
+<attribute name="VALUE" x="74.125" y="36.27" size="0.4064" layer="28" rot="MR0"/>
 </element>
 <element name="E$4" library="pinhead" package="1X01" value="" x="80.01" y="48.26" smashed="yes">
@@
 <contactref element="E$8" pad="1"/>
 <wire x1="71.755" y1="38.1" x2="80.645" y2="38.1" width="1.016" layer="1"/>
+<wire x1="12.7" y1="38.1" x2="71.755" y2="38.1" width="1.016" layer="1"/>
 </signal>
 <signal name="S$2">
@@
 <wire x1="19.25" y1="34.85" x2="79.935" y2="34.85" width="1.016" layer="1"/>
 <wire x1="79.935" y1="34.85" x2="80.01" y2="34.925" width="1.016" layer="1"/>
+<wire x1="80.01" y1="34.925" x2="74.93" y2="34.925" width="1.016" layer="16"/>
 </signal>
 <signal name="S$3">
