File: hardware/tools/lna_3v/lna3v_eagleproj/lna_simple.brd (EAGLE design)
At the start: 27.9 x 16.2 mm, 11 parts, among them U1 BGA2801, X1 SMA-142-0701-801/806, X2 SMA-142-0701-801/806

Commit message: Update PCBs
Parts:
- JP1: device pinhead:1X02/90 -> pinhead:2X03
- moved JP1 6.35 mm to (29.2, 19.1), flipped to the bottom, turned to 0 degrees
- moved D1 2.84 mm to (34.3, 20.3), turned to 90 degrees
- moved C4 0.64 mm to (30.5, 22.2)
Connections:
- net AGND: now also JP1.6; no longer JP1.2
- net AVCC: now also JP1.4; no longer JP1.1
Routing:
- net AVCC: track 13.4 -> 14.0 mm
- net AGND: vias 26 -> 24
Other:
- board text removed: "3.3V Only"
Changed lines of the file:
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@@
 <?xml version="1.0" encoding="utf-8"?>
 <!DOCTYPE eagle SYSTEM "eagle.dtd">
-<eagle version="6.4">
+<eagle version="6.5.0">
 <drawing>
 <settings>
@@
 <wire x1="31.75" y1="26.67" x2="38.1" y2="26.67" width="2.032" layer="41"/>
 <rectangle x1="23.495" y1="21.2725" x2="28.2575" y2="23.1775" layer="41"/>
-<rectangle x1="27.94" y1="17.78" x2="30.7975" y2="22.5425" layer="41"/>
-<rectangle x1="25.4" y1="17.78" x2="28.8925" y2="20.0025" layer="41"/>
 <text x="16.51" y="19.3675" size="1.27" layer="21" font="vector" ratio="16">INPUT</text>
 <text x="35.2425" y="19.3675" size="1.27" layer="21" font="vector" ratio="16">OUTPUT</text>
 <text x="20.955" y="29.21" size="1.27" layer="21" font="vector" ratio="16">ChipWhisperer.com</text>
-<text x="26.9875" y="16.8275" size="1.016" layer="21" font="vector" ratio="16">3.3V Only</text>
 <rectangle x1="15.24" y1="24.765" x2="20.955" y2="28.575" layer="41"/>
 <rectangle x1="37.7825" y1="24.765" x2="43.18" y2="28.575" layer="41"/>
@@
 <element name="C2" library="rcl" package="C0603" value="100nF" x="34.925" y="26.67"/>
 <element name="C3" library="rcl" package="C0603" value="100nF" x="24.13" y="26.67"/>
-<element name="C4" library="rcl" package="C0805" value="4u7" x="30.48" y="21.59"/>
+<element name="C4" library="rcl" package="C0805" value="4u7" x="30.48" y="22.225"/>
 <element name="X1" library="con-coax" package="J502-ND-142-0701-801/806" value="SMA-142-0701-801/806" x="15.24" y="26.67">
 <attribute name="OC_NEWARK" value="90F2624" x="15.24" y="26.67" size="1.778" layer="27" display="off"/>
@@
 </element>
 <element name="R1" library="resistor" package="R0603" value="330R" x="26.67" y="22.225"/>
-<element name="D1" library="diode" package="DO214AC" value="" x="31.75" y="19.05"/>
-<element name="JP1" library="pinhead" package="1X02/90" value="" x="24.13" y="15.24" rot="R180"/>
+<element name="D1" library="diode" package="DO214AC" value="" x="34.29" y="20.32" rot="R90"/>
 <element name="LED1" library="adafruit" package="CHIP-LED0603" value="" x="24.13" y="22.86"/>
+<element name="JP1" library="pinhead" package="2X03" value="" x="29.21" y="19.05" rot="MR0"/>
 </elements>
 <signals>
@@
 <via x="21.59" y="24.765" extent="1-16" drill="0.381" shape="octagon"/>
 <contactref element="D1" pad="A"/>
-<contactref element="JP1" pad="2"/>
 <contactref element="LED1" pad="C"/>
 <via x="21.59" y="21.59" extent="1-16" drill="0.381" shape="octagon"/>
@@
 <via x="36.83" y="31.115" extent="1-16" drill="0.381" shape="octagon"/>
 <via x="36.83" y="21.59" extent="1-16" drill="0.381" shape="octagon"/>
-<via x="34.925" y="21.59" extent="1-16" drill="0.381" shape="octagon"/>
-<via x="36.83" y="19.05" extent="1-16" drill="0.381" shape="octagon"/>
 <via x="40.005" y="19.05" extent="1-16" drill="0.381" shape="octagon"/>
 <via x="19.05" y="19.05" extent="1-16" drill="0.381" shape="octagon"/>
 <via x="29.21" y="28.575" extent="1-16" drill="0.381" shape="octagon"/>
+<contactref element="JP1" pad="6"/>
 </signal>
 <signal name="N$4">
@@
 <contactref element="R1" pad="2"/>
 <contactref element="D1" pad="C"/>
-<contactref element="JP1" pad="1"/>
 <wire x1="29.63" y1="24.13" x2="29.560759375" y2="24.13" width="0.4064" layer="1"/>
 <wire x1="29.560759375" y1="24.13" x2="29.560759375" y2="25.750759375" width="0.4064" layer="1"/>
-<wire x1="29.53" y1="21.59" x2="29.63" y2="24.13" width="0.4064" layer="1"/>
-<wire x1="29.53" y1="21.59" x2="28.155" y2="21.59" width="0.6096" layer="1"/>
-<wire x1="28.155" y1="21.59" x2="27.52" y2="22.225" width="0.6096" layer="1"/>
-<wire x1="29.7" y1="19.05" x2="29.7" y2="21.42" width="0.6096" layer="1"/>
-<wire x1="29.7" y1="21.42" x2="29.53" y2="21.59" width="0.6096" layer="1"/>
-<wire x1="25.4" y1="19.05" x2="29.7" y2="19.05" width="0.6096" layer="1"/>
+<wire x1="29.53" y1="22.225" x2="29.63" y2="24.13" width="0.4064" layer="1"/>
+<wire x1="29.53" y1="22.225" x2="27.52" y2="22.225" width="0.6096" layer="1"/>
+<wire x1="29.7" y1="22.055" x2="29.53" y2="22.225" width="0.6096" layer="1"/>
+<contactref element="JP1" pad="4"/>
+<wire x1="29.53" y1="20.32" x2="29.53" y2="22.225" width="1.4224" layer="1"/>
+<wire x1="29.53" y1="20" x2="30.48" y2="19.05" width="0.6096" layer="1"/>
+<wire x1="30.48" y1="19.05" x2="33.51" y2="19.05" width="0.6096" layer="1"/>
+<wire x1="33.51" y1="19.05" x2="34.29" y2="18.27" width="0.6096" layer="1"/>
+<wire x1="29.53" y1="20.32" x2="29.53" y2="20" width="0.6096" layer="1"/>
+<wire x1="29.21" y1="20.32" x2="29.53" y2="20" width="0.6096" layer="1"/>
 </signal>
 <signal name="N$7">

Commit message: HW: Update LNA PCB to Latest beta, not tested in HW yet
Parts:
- moved C4 6.68 mm to (24.4, 19.4), turned to 90 degrees
- moved R1 6.26 mm to (21.3, 19.1), turned to 270 degrees
- moved LED1 6.10 mm to (19.4, 19.1), turned to 180 degrees
- moved D1 3.43 mm to (37.1, 18.4), turned to 0 degrees
- moved C1 0.63 mm to (31.1, 24.1)
Routing:
- net AVCC: track 14.0 -> 30.2 mm, vias 0 -> 2
- net AGND: vias 24 -> 26
Other:
- board text added: "+20dB"
- board text added: "1"
- board text added: "2"
- board text added: "3.3V"
- board text added: "4:+3.3V"
- board text added: "5"
- board text added: "6"
- board text added: "6:GND"
- board text added: "GND"
- board text added: "IN"
- board text added: "Inc."
- board text added: "NPCB-LNA-02"
- board text added: "NewAE"
- board text added: "OUT"
- board text added: "Technology"
- board text removed: "INPUT"
- board text removed: "OUTPUT"

Commit message: HW: Update LNA + Diff probe with latest version
Parts:
- added U$1, U$2: FIDUCIAL, adafruit:FIDUCIAL_1MM
Changed lines of the file:
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@@
 <layer number="3" name="Route3" color="4" fill="3" visible="no" active="no"/>
 <layer number="14" name="Route14" color="1" fill="6" visible="no" active="no"/>
-<layer number="15" name="Route15" color="4" fill="6" visible="no" active="no"/>
+<layer number="15" name="Route15" color="4" fill="6" visible="yes" active="yes"/>
 <layer number="16" name="Bottom" color="1" fill="1" visible="yes" active="yes"/>
 <layer number="17" name="Pads" color="2" fill="1" visible="yes" active="yes"/>
@@
 <layer number="23" name="tOrigins" color="15" fill="1" visible="yes" active="yes"/>
 <layer number="24" name="bOrigins" color="15" fill="1" visible="yes" active="yes"/>
-<layer number="25" name="tNames" color="7" fill="1" visible="no" active="yes"/>
+<layer number="25" name="tNames" color="7" fill="1" visible="yes" active="yes"/>
 <layer number="26" name="bNames" color="7" fill="1" visible="no" active="yes"/>
 <layer number="27" name="tValues" color="7" fill="1" visible="no" active="yes"/>
 <layer number="28" name="bValues" color="7" fill="1" visible="no" active="yes"/>
-<layer number="29" name="tStop" color="7" fill="3" visible="no" active="yes"/>
+<layer number="29" name="tStop" color="7" fill="3" visible="yes" active="yes"/>
 <layer number="30" name="bStop" color="7" fill="6" visible="no" active="yes"/>
 <layer number="31" name="tCream" color="7" fill="4" visible="no" active="yes"/>
@@
 <wire x1="31.75" y1="26.67" x2="38.1" y2="26.67" width="2.032" layer="41"/>
 <rectangle x1="20.955" y1="17.4625" x2="25.7175" y2="19.3675" layer="41"/>
-<text x="17.4625" y="18.415" size="1.27" layer="21" font="vector" ratio="16" rot="R90">IN</text>
+<text x="17.145" y="19.05" size="1.27" layer="21" font="vector" ratio="16" rot="R90">IN</text>
 <text x="42.545" y="17.4625" size="1.27" layer="21" font="vector" ratio="16" rot="R90">OUT</text>
 <rectangle x1="15.24" y1="24.765" x2="20.955" y2="28.575" layer="41"/>
@@
 </autorouter>
 <elements>
-<element name="U1" library="customs" package="SOTT323-6" value="BGA2801" x="30.48" y="26.67" rot="R45"/>
-<element name="C1" library="rcl" package="C0603" value="22nF" x="31.115" y="24.13"/>
-<element name="C2" library="rcl" package="C0603" value="100nF" x="34.925" y="26.67"/>
-<element name="C3" library="rcl" package="C0603" value="100nF" x="24.13" y="26.67"/>
-<element name="C4" library="rcl" package="C0805" value="4u7" x="24.4475" y="19.3675" rot="R90"/>
-<element name="X1" library="con-coax" package="J502-ND-142-0701-801/806" value="SMA-142-0701-801/806" x="15.24" y="26.67">
+<element name="U1" library="customs" package="SOTT323-6" value="BGA2801" x="30.48" y="26.67" smashed="yes" rot="R45">
+<attribute name="NAME" x="27.18985625" y="27.6918125" size="0.8128" layer="25" font="vector" ratio="16" rot="R45"/>
+<attribute name="VALUE" x="29.4193375" y="22.639490625" size="1.27" layer="27" rot="R45"/>
+</element>
+<element name="C1" library="rcl" package="C0603" value="22nF" x="31.115" y="24.13" smashed="yes">
+<attribute name="NAME" x="33.02" y="23.495" size="0.8128" layer="25" font="vector" ratio="16"/>
+<attribute name="VALUE" x="30.48" y="22.225" size="1.27" layer="27"/>
+</element>
+<element name="C2" library="rcl" package="C0603" value="100nF" x="34.925" y="26.67" smashed="yes">
+<attribute name="NAME" x="33.3375" y="27.94" size="0.8128" layer="25" font="vector" ratio="16"/>
+<attribute name="VALUE" x="34.29" y="24.765" size="1.27" layer="27"/>
+</element>
+<element name="C3" library="rcl" package="C0603" value="100nF" x="24.13" y="26.67" smashed="yes">
+<attribute name="NAME" x="21.9075" y="27.94" size="0.8128" layer="25" font="vector" ratio="16"/>
+<attribute name="VALUE" x="23.495" y="24.765" size="1.27" layer="27"/>
+</element>
+<element name="C4" library="rcl" package="C0805" value="4u7" x="24.4475" y="19.3675" smashed="yes" rot="R90">
+<attribute name="NAME" x="23.8125" y="16.8275" size="0.8128" layer="25" font="vector" ratio="16"/>
+<attribute name="VALUE" x="26.9875" y="18.0975" size="1.27" layer="27" rot="R90"/>
+</element>
+<element name="X1" library="con-coax" package="J502-ND-142-0701-801/806" value="SMA-142-0701-801/806" x="15.24" y="26.67" smashed="yes">
 <attribute name="OC_NEWARK" value="90F2624" x="15.24" y="26.67" size="1.778" layer="27" display="off"/>
 <attribute name="MPN" value="142-0701-801" x="15.24" y="26.67" size="1.778" layer="27" display="off"/>
 <attribute name="MF" value="JOHNSON COMPONENTS" x="15.24" y="26.67" size="1.778" layer="27" display="off"/>
 <attribute name="OC_FARNELL" value="1608592" x="15.24" y="26.67" size="1.778" layer="27" display="off"/>
-</element>
-<element name="X2" library="con-coax" package="J502-ND-142-0701-801/806" value="SMA-142-0701-801/806" x="43.18" y="26.67" rot="R180">
+<attribute name="VALUE" x="16.51" y="17.78" size="1.778" layer="27"/>
+</element>
+<element name="X2" library="con-coax" package="J502-ND-142-0701-801/806" value="SMA-142-0701-801/806" x="43.18" y="26.67" smashed="yes" rot="R180">
 <attribute name="OC_NEWARK" value="90F2624" x="43.18" y="26.67" size="1.778" layer="27" rot="R180" display="off"/>
 <attribute name="MPN" value="142-0701-801" x="43.18" y="26.67" size="1.778" layer="27" rot="R180" display="off"/>
 <attribute name="MF" value="JOHNSON COMPONENTS" x="43.18" y="26.67" size="1.778" layer="27" rot="R180" display="off"/>
 <attribute name="OC_FARNELL" value="1608592" x="43.18" y="26.67" size="1.778" layer="27" rot="R180" display="off"/>
-</element>
-<element name="R1" library="resistor" package="R0603" value="330R" x="21.2725" y="19.05" rot="R270"/>
-<element name="D1" library="diode" package="DO214AC" value="" x="37.1475" y="18.415"/>
-<element name="LED1" library="adafruit" package="CHIP-LED0603" value="" x="19.3675" y="19.05" rot="R180"/>
+<attribute name="VALUE" x="41.91" y="35.56" size="1.778" layer="27" rot="R180"/>
+</element>
+<element name="R1" library="resistor" package="R0603" value="330R" x="21.2725" y="19.05" smashed="yes" rot="R270">
+<attribute name="NAME" x="22.9235" y="19.431" size="0.8128" layer="25" font="vector" ratio="16" rot="R90"/>
+<attribute name="VALUE" x="19.2405" y="19.939" size="1.27" layer="27" rot="R270"/>
+</element>
+<element name="D1" library="diode" package="DO214AC" value="" x="37.1475" y="18.415" smashed="yes">
+<attribute name="NAME" x="34.5075" y="20.0185" size="0.8128" layer="25" font="vector" ratio="16"/>
+<attribute name="VALUE" x="34.5075" y="15.859" size="1.27" layer="27" ratio="10"/>
+</element>
+<element name="LED1" library="adafruit" package="CHIP-LED0603" value="" x="19.3675" y="19.05" smashed="yes" rot="R180">
+<attribute name="NAME" x="17.78" y="20.6375" size="0.8128" layer="25" font="vector" ratio="16" rot="R270"/>
+<attribute name="VALUE" x="17.4625" y="19.685" size="1.27" layer="27" rot="R270"/>
+</element>
 <element name="JP1" library="pinhead" package="2X03" value="" x="29.21" y="19.05" rot="MR0"/>
+<element name="U$1" library="adafruit" package="FIDUCIAL_1MM" value="FIDUCIAL" x="16.51" y="17.78"/>
+<element name="U$2" library="adafruit" package="FIDUCIAL_1MM" value="FIDUCIAL" x="35.8775" y="29.5275"/>
 </elements>
 <signals>
