File: hardware/tools/clockextractor/lnafilter-pcb/lna-plug.brd (EAGLE design)
At the start: 151.7 x 22.2 mm, 81 parts, among them U1 AD8331, U2 BGA2801, X1 SMA-142-0701-851/861, X2 SMA-142-0711-821/826, X3 SMA-142-0701-851/861

Commit message: Update CW PCB & Clock Recovery PCB
Parts:
- C1, C11, C12, C2, C3, C33, C36, C4, C5, C7, C8: value (none) -> 100n
- C32: value (none) -> 22nF
- C34: value (none) -> 1u
- C42, C43: value (none) -> 330pF
Changed lines of the file:
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@@
 <attribute name="VALUE" x="121.539" y="41.402" size="1.016" layer="27" font="vector" rot="R180"/>
 </element>
-<element name="C1" library="resistor" package="C0603" value="" x="137.16" y="41.275" smashed="yes" rot="R270">
+<element name="C1" library="resistor" package="C0603" value="100n" x="137.16" y="41.275" smashed="yes" rot="R270">
 <attribute name="NAME" x="137.922" y="42.164" size="1.016" layer="25" font="vector" ratio="16" rot="R270"/>
 <attribute name="VALUE" x="135.128" y="42.164" size="1.27" layer="27" rot="R270"/>
 </element>
-<element name="C2" library="resistor" package="C0603" value="" x="126.365" y="43.815" smashed="yes" rot="R180">
+<element name="C2" library="resistor" package="C0603" value="100n" x="126.365" y="43.815" smashed="yes" rot="R180">
 <attribute name="NAME" x="127.254" y="45.9105" size="1.27" layer="25" rot="R180"/>
 <attribute name="VALUE" x="127.254" y="45.847" size="1.27" layer="27" rot="R180"/>
 </element>
-<element name="C3" library="resistor" package="C0603" value="" x="133.35" y="41.91" smashed="yes" rot="R270">
+<element name="C3" library="resistor" package="C0603" value="100n" x="133.35" y="41.91" smashed="yes" rot="R270">
 <attribute name="NAME" x="134.112" y="42.799" size="1.016" layer="25" font="vector" ratio="16" rot="R270"/>
 <attribute name="VALUE" x="131.318" y="42.799" size="1.27" layer="27" rot="R270"/>
 </element>
-<element name="C4" library="resistor" package="C0603" value="" x="137.16" y="45.72" smashed="yes" rot="R270">
+<element name="C4" library="resistor" package="C0603" value="100n" x="137.16" y="45.72" smashed="yes" rot="R270">
 <attribute name="NAME" x="136.652" y="49.149" size="1.016" layer="25" font="vector" ratio="16" rot="R270"/>
 <attribute name="VALUE" x="135.128" y="46.609" size="1.27" layer="27" rot="R270"/>
 </element>
-<element name="C5" library="resistor" package="C0603" value="" x="128.27" y="53.34" smashed="yes" rot="R90">
+<element name="C5" library="resistor" package="C0603" value="100n" x="128.27" y="53.34" smashed="yes" rot="R90">
 <attribute name="NAME" x="128.778" y="54.991" size="1.016" layer="25" font="vector" ratio="16" rot="R90"/>
 <attribute name="VALUE" x="130.302" y="52.451" size="1.27" layer="27" rot="R90"/>
@@
 <attribute name="VALUE" x="132.842" y="53.4035" size="1.27" layer="27" rot="R90"/>
 </element>
-<element name="C7" library="resistor" package="C0603" value="" x="127" y="47.625" smashed="yes" rot="R90">
+<element name="C7" library="resistor" package="C0603" value="100n" x="127" y="47.625" smashed="yes" rot="R90">
 <attribute name="NAME" x="126.238" y="46.736" size="1.016" layer="25" font="vector" ratio="16" rot="R90"/>
 <attribute name="VALUE" x="129.032" y="46.736" size="1.27" layer="27" rot="R90"/>
 </element>
-<element name="C8" library="resistor" package="C0603" value="" x="124.46" y="47.625" smashed="yes" rot="R270">
+<element name="C8" library="resistor" package="C0603" value="100n" x="124.46" y="47.625" smashed="yes" rot="R270">
 <attribute name="NAME" x="122.682" y="48.514" size="1.016" layer="25" font="vector" ratio="16" rot="R270"/>
 <attribute name="VALUE" x="122.428" y="48.514" size="1.27" layer="27" rot="R270"/>
@@
 <attribute name="VALUE" x="113.157" y="49.276" size="1.27" layer="27" rot="R90"/>
 </element>
-<element name="C11" library="resistor" package="C0603" value="" x="144.145" y="46.99" smashed="yes">
+<element name="C11" library="resistor" package="C0603" value="100n" x="144.145" y="46.99" smashed="yes">
 <attribute name="NAME" x="142.9385" y="45.212" size="1.016" layer="25" font="vector" ratio="16"/>
 <attribute name="VALUE" x="143.256" y="44.958" size="1.27" layer="27"/>
 </element>
-<element name="C12" library="resistor" package="C0603" value="" x="144.145" y="49.53" smashed="yes">
+<element name="C12" library="resistor" package="C0603" value="100n" x="144.145" y="49.53" smashed="yes">
 <attribute name="NAME" x="142.9385" y="50.292" size="1.016" layer="25" font="vector" ratio="16"/>
 <attribute name="VALUE" x="143.256" y="47.498" size="1.27" layer="27"/>
@@
 <attribute name="VALUE" x="21.971" y="48.768" size="1.27" layer="27"/>
 </element>
-<element name="C32" library="resistor" package="C0603" value="" x="26.035" y="48.26" smashed="yes">
+<element name="C32" library="resistor" package="C0603" value="22nF" x="26.035" y="48.26" smashed="yes">
 <attribute name="NAME" x="24.1935" y="45.847" size="1.27" layer="25" font="vector" ratio="16"/>
 <attribute name="VALUE" x="25.146" y="46.228" size="1.27" layer="27"/>
 </element>
-<element name="C33" library="resistor" package="C0603" value="" x="29.21" y="48.26" smashed="yes" rot="R180">
+<element name="C33" library="resistor" package="C0603" value="100n" x="29.21" y="48.26" smashed="yes" rot="R180">
 <attribute name="NAME" x="31.369" y="47.1805" size="1.27" layer="25" font="vector" ratio="16" rot="R180"/>
 <attribute name="VALUE" x="30.099" y="50.292" size="1.27" layer="27" rot="R180"/>
 </element>
-<element name="C34" library="resistor" package="C0603" value="" x="29.21" y="48.26" smashed="yes" rot="MR0">
+<element name="C34" library="resistor" package="C0603" value="1u" x="29.21" y="48.26" smashed="yes" rot="MR0">
 <attribute name="NAME" x="30.099" y="49.022" size="1.27" layer="26" font="vector" ratio="16" rot="MR0"/>
 <attribute name="VALUE" x="30.099" y="46.228" size="1.27" layer="28" rot="MR0"/>
@@
 <attribute name="VALUE" x="32.131" y="43.688" size="1.27" layer="27"/>
 </element>
-<element name="C36" library="resistor" package="C0603" value="" x="132.715" y="54.2925" smashed="yes" rot="R90">
+<element name="C36" library="resistor" package="C0603" value="100n" x="132.715" y="54.2925" smashed="yes" rot="R90">
 <attribute name="NAME" x="133.223" y="55.9435" size="1.016" layer="25" font="vector" ratio="16" rot="R90"/>
 <attribute name="VALUE" x="134.747" y="53.4035" size="1.27" layer="27" rot="R90"/>
@@
 <attribute name="VALUE" x="120.015" y="40.64" size="1.27" layer="27"/>
 </element>
-<element name="C42" library="resistor" package="C0603" value="" x="149.86" y="50.165" smashed="yes" rot="R90">
+<element name="C42" library="resistor" package="C0603" value="330pF" x="149.86" y="50.165" smashed="yes" rot="R90">
 <attribute name="NAME" x="148.7805" y="48.9585" size="1.016" layer="25" font="vector" ratio="16" rot="R90"/>
 <attribute name="VALUE" x="151.892" y="49.276" size="1.27" layer="27" rot="R90"/>
 </element>
-<element name="C43" library="resistor" package="C0603" value="" x="149.86" y="46.0375" smashed="yes" rot="R90">
+<element name="C43" library="resistor" package="C0603" value="330pF" x="149.86" y="46.0375" smashed="yes" rot="R90">
 <attribute name="NAME" x="148.7805" y="44.831" size="1.016" layer="25" font="vector" ratio="16" rot="R90"/>
 <attribute name="VALUE" x="151.892" y="45.1485" size="1.27" layer="27" rot="R90"/>

Commit message: HW: Update clock recovery board
Parts:
- C10, C28, C29, C30, C31, C35, C38: value (none) -> 100nF
Changed lines of the file:
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@@
 <?xml version="1.0" encoding="utf-8"?>
 <!DOCTYPE eagle SYSTEM "eagle.dtd">
-<eagle version="6.5.0">
+<eagle version="7.1.0">
 <drawing>
 <settings>
@@
 <pass name="Default">
 <param name="RoutingGrid" value="50mil"/>
+<param name="AutoGrid" value="1"/>
+<param name="Efforts" value="0"/>
+<param name="TopRouterVariant" value="1"/>
 <param name="tpViaShape" value="round"/>
 <param name="PrefDir.1" value="|"/>
@@
 <attribute name="VALUE" x="124.841" y="48.133" size="1.016" layer="27" font="vector"/>
 </element>
-<element name="C10" library="resistor" package="C0603" value="" x="111.125" y="50.165" smashed="yes" rot="R90">
+<element name="C10" library="resistor" package="C0603" value="100nF" x="111.125" y="50.165" smashed="yes" rot="R90">
 <attribute name="NAME" x="113.2205" y="48.641" size="1.27" layer="25" font="vector" ratio="16" rot="R90"/>
 <attribute name="VALUE" x="113.157" y="49.276" size="1.27" layer="27" rot="R90"/>
@@
 <attribute name="VALUE" x="53.975" y="52.07" size="1.27" layer="27" rot="R270"/>
 </element>
-<element name="C28" library="resistor" package="C0603" value="" x="108.585" y="48.26" smashed="yes">
+<element name="C28" library="resistor" package="C0603" value="100nF" x="108.585" y="48.26" smashed="yes">
 <attribute name="NAME" x="107.3785" y="46.1645" size="1.27" layer="25" font="vector" ratio="16"/>
 <attribute name="VALUE" x="107.696" y="46.228" size="1.27" layer="27"/>
@@
 <attribute name="VALUE" x="28.1493375" y="46.769490625" size="1.27" layer="27" rot="R45"/>
 </element>
-<element name="C30" library="resistor" package="C0603" value="" x="33.02" y="50.8" smashed="yes">
+<element name="C30" library="resistor" package="C0603" value="100nF" x="33.02" y="50.8" smashed="yes">
 <attribute name="NAME" x="31.496" y="51.562" size="1.27" layer="25" font="vector" ratio="16"/>
 <attribute name="VALUE" x="32.131" y="48.768" size="1.27" layer="27"/>
 </element>
-<element name="C31" library="resistor" package="C0603" value="" x="22.86" y="50.8" smashed="yes">
+<element name="C31" library="resistor" package="C0603" value="100nF" x="22.86" y="50.8" smashed="yes">
 <attribute name="NAME" x="21.336" y="51.562" size="1.27" layer="25" font="vector" ratio="16"/>
 <attribute name="VALUE" x="21.971" y="48.768" size="1.27" layer="27"/>
@@
 <attribute name="VALUE" x="33.655" y="50.8" size="1.27" layer="27" rot="R270"/>
 </element>
-<element name="C35" library="resistor" package="C0603" value="" x="33.02" y="45.72" smashed="yes">
+<element name="C35" library="resistor" package="C0603" value="100nF" x="33.02" y="45.72" smashed="yes">
 <attribute name="NAME" x="31.1785" y="43.6245" size="1.27" layer="25" font="vector" ratio="16"/>
 <attribute name="VALUE" x="32.131" y="43.688" size="1.27" layer="27"/>
@@
 <attribute name="VALUE" x="38.735" y="57.785" size="1.778" layer="27" rot="R270"/>
 </element>
-<element name="C29" library="resistor" package="C0603" value="" x="47.625" y="50.165" smashed="yes" rot="R90">
+<element name="C29" library="resistor" package="C0603" value="100nF" x="47.625" y="50.165" smashed="yes" rot="R90">
 <attribute name="NAME" x="46.863" y="49.276" size="1.27" layer="25" font="vector" ratio="16" rot="R90"/>
 <attribute name="VALUE" x="49.657" y="49.276" size="1.27" layer="27" rot="R90"/>
 </element>
-<element name="C38" library="resistor" package="C0603" value="" x="45.085" y="48.26" smashed="yes" rot="R180">
+<element name="C38" library="resistor" package="C0603" value="100nF" x="45.085" y="48.26" smashed="yes" rot="R180">
 <attribute name="NAME" x="46.9265" y="47.498" size="1.27" layer="25" font="vector" ratio="16" rot="R180"/>
 <attribute name="VALUE" x="45.974" y="50.292" size="1.27" layer="27" rot="R180"/>

Commit message: PCBs: Add LNA/Diff-Probe updates, + firmware temp fixes
Parts:
- C37, C6: value (none) -> 22nF
Changed lines of the file:
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@@
 <attribute name="VALUE" x="130.302" y="52.451" size="1.27" layer="27" rot="R90"/>
 </element>
-<element name="C6" library="resistor" package="C0603" value="" x="130.81" y="54.2925" smashed="yes" rot="R90">
+<element name="C6" library="resistor" package="C0603" value="22nF" x="130.81" y="54.2925" smashed="yes" rot="R90">
 <attribute name="NAME" x="131.318" y="55.9435" size="1.016" layer="25" font="vector" ratio="16" rot="R90"/>
 <attribute name="VALUE" x="132.842" y="53.4035" size="1.27" layer="27" rot="R90"/>
@@
 <attribute name="VALUE" x="134.747" y="53.4035" size="1.27" layer="27" rot="R90"/>
 </element>
-<element name="C37" library="resistor" package="C0603" value="" x="139.065" y="45.72" smashed="yes" rot="R270">
+<element name="C37" library="resistor" package="C0603" value="22nF" x="139.065" y="45.72" smashed="yes" rot="R270">
 <attribute name="NAME" x="139.827" y="46.609" size="1.016" layer="25" font="vector" ratio="16" rot="R270"/>
 <attribute name="VALUE" x="137.033" y="46.609" size="1.27" layer="27" rot="R270"/>
