File: hardware/tools/clockextractor/lnafilter-pcb/lna-plug.sch (EAGLE design)
At the start: 81 parts, among them U1 AD8331, U2 BGA2801, X1 SMA-142-0701-851/861, X2 SMA-142-0711-821/826, X3 SMA-142-0701-851/861

Commit message: Update CW PCB & Clock Recovery PCB
Parts:
- C1, C11, C12, C2, C3, C33, C36, C4, C5, C7, C8: value (none) -> 100n
- C32: value (none) -> 22nF
- C34: value (none) -> 1u
- C42, C43: value (none) -> 330pF
Changed lines of the file:
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@@
 <grid distance="0.1" unitdist="inch" unit="inch" style="lines" multiple="1" display="no" altdistance="0.01" altunitdist="inch" altunit="inch"/>
 <layers>
-<layer number="1" name="Top" color="4" fill="1" visible="yes" active="no"/>
-<layer number="2" name="Route2" color="1" fill="3" visible="yes" active="no"/>
-<layer number="3" name="Route3" color="4" fill="3" visible="yes" active="no"/>
-<layer number="14" name="Route14" color="1" fill="6" visible="yes" active="no"/>
-<layer number="15" name="Route15" color="4" fill="6" visible="yes" active="no"/>
-<layer number="16" name="Bottom" color="1" fill="1" visible="yes" active="no"/>
-<layer number="17" name="Pads" color="2" fill="1" visible="yes" active="no"/>
-<layer number="18" name="Vias" color="2" fill="1" visible="yes" active="no"/>
-<layer number="19" name="Unrouted" color="6" fill="1" visible="yes" active="no"/>
-<layer number="20" name="Dimension" color="15" fill="1" visible="yes" active="no"/>
-<layer number="21" name="tPlace" color="7" fill="1" visible="yes" active="no"/>
-<layer number="22" name="bPlace" color="7" fill="1" visible="yes" active="no"/>
-<layer number="23" name="tOrigins" color="15" fill="1" visible="yes" active="no"/>
-<layer number="24" name="bOrigins" color="15" fill="1" visible="yes" active="no"/>
-<layer number="25" name="tNames" color="7" fill="1" visible="yes" active="no"/>
-<layer number="26" name="bNames" color="7" fill="1" visible="yes" active="no"/>
-<layer number="27" name="tValues" color="7" fill="1" visible="yes" active="no"/>
-<layer number="28" name="bValues" color="7" fill="1" visible="yes" active="no"/>
+<layer number="1" name="Top" color="4" fill="1" visible="no" active="no"/>
+<layer number="2" name="Route2" color="1" fill="3" visible="no" active="no"/>
+<layer number="3" name="Route3" color="4" fill="3" visible="no" active="no"/>
+<layer number="14" name="Route14" color="1" fill="6" visible="no" active="no"/>
+<layer number="15" name="Route15" color="4" fill="6" visible="no" active="no"/>
+<layer number="16" name="Bottom" color="1" fill="1" visible="no" active="no"/>
+<layer number="17" name="Pads" color="2" fill="1" visible="no" active="no"/>
+<layer number="18" name="Vias" color="2" fill="1" visible="no" active="no"/>
+<layer number="19" name="Unrouted" color="6" fill="1" visible="no" active="no"/>
+<layer number="20" name="Dimension" color="15" fill="1" visible="no" active="no"/>
+<layer number="21" name="tPlace" color="7" fill="1" visible="no" active="no"/>
+<layer number="22" name="bPlace" color="7" fill="1" visible="no" active="no"/>
+<layer number="23" name="tOrigins" color="15" fill="1" visible="no" active="no"/>
+<layer number="24" name="bOrigins" color="15" fill="1" visible="no" active="no"/>
+<layer number="25" name="tNames" color="7" fill="1" visible="no" active="no"/>
+<layer number="26" name="bNames" color="7" fill="1" visible="no" active="no"/>
+<layer number="27" name="tValues" color="7" fill="1" visible="no" active="no"/>
+<layer number="28" name="bValues" color="7" fill="1" visible="no" active="no"/>
 <layer number="29" name="tStop" color="7" fill="3" visible="no" active="no"/>
 <layer number="30" name="bStop" color="7" fill="6" visible="no" active="no"/>
@@
 <layer number="35" name="tGlue" color="7" fill="4" visible="no" active="no"/>
 <layer number="36" name="bGlue" color="7" fill="5" visible="no" active="no"/>
-<layer number="37" name="tTest" color="7" fill="1" visible="yes" active="no"/>
-<layer number="38" name="bTest" color="7" fill="1" visible="yes" active="no"/>
+<layer number="37" name="tTest" color="7" fill="1" visible="no" active="no"/>
+<layer number="38" name="bTest" color="7" fill="1" visible="no" active="no"/>
 <layer number="39" name="tKeepout" color="4" fill="11" visible="no" active="no"/>
 <layer number="40" name="bKeepout" color="1" fill="11" visible="no" active="no"/>
@@
 <layer number="44" name="Drills" color="7" fill="1" visible="no" active="no"/>
 <layer number="45" name="Holes" color="7" fill="1" visible="no" active="no"/>
-<layer number="46" name="Milling" color="3" fill="1" visible="yes" active="no"/>
-<layer number="47" name="Measures" color="7" fill="1" visible="yes" active="no"/>
-<layer number="48" name="Document" color="7" fill="1" visible="yes" active="no"/>
-<layer number="49" name="Reference" color="7" fill="1" visible="yes" active="no"/>
-<layer number="50" name="dxf" color="7" fill="1" visible="yes" active="no"/>
-<layer number="51" name="tDocu" color="7" fill="1" visible="yes" active="no"/>
-<layer number="52" name="bDocu" color="7" fill="1" visible="yes" active="no"/>
-<layer number="53" name="tGND_GNDA" color="7" fill="1" visible="yes" active="no"/>
-<layer number="54" name="bGND_GNDA" color="7" fill="1" visible="yes" active="no"/>
-<layer number="56" name="wert" color="7" fill="1" visible="yes" active="no"/>
+<layer number="46" name="Milling" color="3" fill="1" visible="no" active="no"/>
+<layer number="47" name="Measures" color="7" fill="1" visible="no" active="no"/>
+<layer number="48" name="Document" color="7" fill="1" visible="no" active="no"/>
+<layer number="49" name="Reference" color="7" fill="1" visible="no" active="no"/>
+<layer number="50" name="dxf" color="7" fill="1" visible="no" active="no"/>
+<layer number="51" name="tDocu" color="7" fill="1" visible="no" active="no"/>
+<layer number="52" name="bDocu" color="7" fill="1" visible="no" active="no"/>
+<layer number="53" name="tGND_GNDA" color="7" fill="1" visible="no" active="no"/>
+<layer number="54" name="bGND_GNDA" color="7" fill="1" visible="no" active="no"/>
+<layer number="56" name="wert" color="7" fill="1" visible="no" active="no"/>
 <layer number="91" name="Nets" color="2" fill="1" visible="yes" active="yes"/>
 <layer number="92" name="Busses" color="1" fill="1" visible="yes" active="yes"/>
@@
 <part name="R1" library="resistor" deviceset="R-US_" device="R0603" value="10k"/>
 <part name="R2" library="resistor" deviceset="R-US_" device="R0603" value="2k2"/>
-<part name="C1" library="resistor" deviceset="C-EU" device="C0603"/>
-<part name="C2" library="resistor" deviceset="C-EU" device="C0603"/>
-<part name="C3" library="resistor" deviceset="C-EU" device="C0603"/>
-<part name="C4" library="resistor" deviceset="C-EU" device="C0603"/>
-<part name="C5" library="resistor" deviceset="C-EU" device="C0603"/>
+<part name="C1" library="resistor" deviceset="C-EU" device="C0603" value="100n"/>
+<part name="C2" library="resistor" deviceset="C-EU" device="C0603" value="100n"/>
+<part name="C3" library="resistor" deviceset="C-EU" device="C0603" value="100n"/>
+<part name="C4" library="resistor" deviceset="C-EU" device="C0603" value="100n"/>
+<part name="C5" library="resistor" deviceset="C-EU" device="C0603" value="100n"/>
 <part name="C6" library="resistor" deviceset="C-EU" device="C0603"/>
-<part name="C7" library="resistor" deviceset="C-EU" device="C0603"/>
-<part name="C8" library="resistor" deviceset="C-EU" device="C0603"/>
+<part name="C7" library="resistor" deviceset="C-EU" device="C0603" value="100n"/>
+<part name="C8" library="resistor" deviceset="C-EU" device="C0603" value="100n"/>
 <part name="C9" library="resistor" deviceset="C-EU" device="C0603" value="18nF"/>
 <part name="C10" library="resistor" deviceset="C-EU" device="C0603"/>
-<part name="C11" library="resistor" deviceset="C-EU" device="C0603"/>
-<part name="C12" library="resistor" deviceset="C-EU" device="C0603"/>
+<part name="C11" library="resistor" deviceset="C-EU" device="C0603" value="100n"/>
+<part name="C12" library="resistor" deviceset="C-EU" device="C0603" value="100n"/>
 <part name="SUPPLY1" library="supply2" deviceset="GND" device=""/>
 <part name="SUPPLY2" library="supply2" deviceset="GND" device=""/>
@@
 <part name="C30" library="resistor" deviceset="C-EU" device="C0603"/>
 <part name="C31" library="resistor" deviceset="C-EU" device="C0603"/>
-<part name="C32" library="resistor" deviceset="C-EU" device="C0603"/>
-<part name="C33" library="resistor" deviceset="C-EU" device="C0603"/>
-<part name="C34" library="resistor" deviceset="C-EU" device="C0603"/>
+<part name="C32" library="resistor" deviceset="C-EU" device="C0603" value="22nF"/>
+<part name="C33" library="resistor" deviceset="C-EU" device="C0603" value="100n"/>
+<part name="C34" library="resistor" deviceset="C-EU" device="C0603" value="1u"/>
 <part name="X2" library="con-coax" deviceset="SMA-" device="142-0711-821/826"/>
 <part name="JP4" library="pinhead" deviceset="PINHD-2X2" device=""/>
@@
 <part name="C35" library="resistor" deviceset="C-EU" device="C0603"/>
 <part name="SUPPLY18" library="supply2" deviceset="GND" device=""/>
-<part name="C36" library="resistor" deviceset="C-EU" device="C0603"/>
+<part name="C36" library="resistor" deviceset="C-EU" device="C0603" value="100n"/>
 <part name="C37" library="resistor" deviceset="C-EU" device="C0603"/>
 <part name="SUPPLY19" library="supply2" deviceset="GND" device=""/>
@@
 <part name="SUPPLY26" library="supply2" deviceset="GND" device=""/>
 <part name="JP11" library="pinhead" deviceset="PINHD-1X1" device=""/>
-<part name="C42" library="resistor" deviceset="C-EU" device="C0603"/>
-<part name="C43" library="resistor" deviceset="C-EU" device="C0603"/>
+<part name="C42" library="resistor" deviceset="C-EU" device="C0603" value="330pF"/>
+<part name="C43" library="resistor" deviceset="C-EU" device="C0603" value="330pF"/>
 <part name="SUPPLY27" library="supply2" deviceset="GND" device=""/>
 <part name="SUPPLY28" library="supply2" deviceset="GND" device=""/>

Commit message: HW: Update clock recovery board
Parts:
- C10, C28, C29, C30, C31, C35, C38: value (none) -> 100nF
Changed lines of the file:
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@@
 <?xml version="1.0" encoding="utf-8"?>
 <!DOCTYPE eagle SYSTEM "eagle.dtd">
-<eagle version="6.5.0">
+<eagle version="7.1.0">
 <drawing>
 <settings>
@@
 <part name="C8" library="resistor" deviceset="C-EU" device="C0603" value="100n"/>
 <part name="C9" library="resistor" deviceset="C-EU" device="C0603" value="18nF"/>
-<part name="C10" library="resistor" deviceset="C-EU" device="C0603"/>
+<part name="C10" library="resistor" deviceset="C-EU" device="C0603" value="100nF"/>
 <part name="C11" library="resistor" deviceset="C-EU" device="C0603" value="100n"/>
 <part name="C12" library="resistor" deviceset="C-EU" device="C0603" value="100n"/>
@@
 <part name="+3V1" library="supply1" deviceset="+3V3" device=""/>
 <part name="FRAME3" library="frames" deviceset="LETTER_L" device=""/>
-<part name="C28" library="resistor" deviceset="C-EU" device="C0603"/>
+<part name="C28" library="resistor" deviceset="C-EU" device="C0603" value="100nF"/>
 <part name="U2" library="customs" deviceset="BGA2801" device=""/>
 <part name="SUPPLY17" library="supply2" deviceset="GND" device=""/>
-<part name="C30" library="resistor" deviceset="C-EU" device="C0603"/>
-<part name="C31" library="resistor" deviceset="C-EU" device="C0603"/>
+<part name="C30" library="resistor" deviceset="C-EU" device="C0603" value="100nF"/>
+<part name="C31" library="resistor" deviceset="C-EU" device="C0603" value="100nF"/>
 <part name="C32" library="resistor" deviceset="C-EU" device="C0603" value="22nF"/>
 <part name="C33" library="resistor" deviceset="C-EU" device="C0603" value="100n"/>
@@
 <part name="JP4" library="pinhead" deviceset="PINHD-2X2" device=""/>
 <part name="JP5" library="pinhead" deviceset="PINHD-2X2" device=""/>
-<part name="C35" library="resistor" deviceset="C-EU" device="C0603"/>
+<part name="C35" library="resistor" deviceset="C-EU" device="C0603" value="100nF"/>
 <part name="SUPPLY18" library="supply2" deviceset="GND" device=""/>
 <part name="C36" library="resistor" deviceset="C-EU" device="C0603" value="100n"/>
@@
 <part name="X1" library="con-coax" deviceset="SMA-" device="142-0701-851/861"/>
 <part name="X3" library="con-coax" deviceset="SMA-" device="142-0701-851/861"/>
-<part name="C29" library="resistor" deviceset="C-EU" device="C0603"/>
-<part name="C38" library="resistor" deviceset="C-EU" device="C0603"/>
+<part name="C29" library="resistor" deviceset="C-EU" device="C0603" value="100nF"/>
+<part name="C38" library="resistor" deviceset="C-EU" device="C0603" value="100nF"/>
 <part name="SUPPLY21" library="supply2" deviceset="GND" device=""/>
 <part name="SUPPLY22" library="supply2" deviceset="GND" device=""/>

Commit message: PCBs: Add LNA/Diff-Probe updates, + firmware temp fixes
Parts:
- C37, C6: value (none) -> 22nF
Changed lines of the file:
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@@
 <part name="C4" library="resistor" deviceset="C-EU" device="C0603" value="100n"/>
 <part name="C5" library="resistor" deviceset="C-EU" device="C0603" value="100n"/>
-<part name="C6" library="resistor" deviceset="C-EU" device="C0603"/>
+<part name="C6" library="resistor" deviceset="C-EU" device="C0603" value="22nF"/>
 <part name="C7" library="resistor" deviceset="C-EU" device="C0603" value="100n"/>
 <part name="C8" library="resistor" deviceset="C-EU" device="C0603" value="100n"/>
@@
 <part name="SUPPLY18" library="supply2" deviceset="GND" device=""/>
 <part name="C36" library="resistor" deviceset="C-EU" device="C0603" value="100n"/>
-<part name="C37" library="resistor" deviceset="C-EU" device="C0603"/>
+<part name="C37" library="resistor" deviceset="C-EU" device="C0603" value="22nF"/>
 <part name="SUPPLY19" library="supply2" deviceset="GND" device=""/>
 <part name="SUPPLY20" library="supply2" deviceset="GND" device=""/>
