File: hardware/tools/diffprobe/diffprobe_eagle/diff_probe.sch (EAGLE design)
At the start: 24 parts, among them U1 AD8129, X1 SMA-142-0701-801/806

Commit message: Fix issues with differential probe
Parts:
- added C10, C9: 0R, rcl:C-EUC0603
- added R10: 1K, 1%, resistor:R-US_R0603
- added R5: 49.9R, resistor:R-US_R0603
- added R6: DNM, resistor:R-US_M0805
- added R7, R8, R9: DNM, resistor:R-US_R0603
- R1: value 10k -> 2k, 1%
- R2: value 2K -> 221R
Connections:
- new net N$12: JP2.1, R5.2, X1G1.1
- new net N$13: C10.1, R6.2, R7.1, U1.VIN-
- new net N$14: C10.2, JP1.2
- new net N$15: R10.1, R7.2, R8.2, R9.2
- net AGND: now also R10.2
- net N$2: now also R9.1
- net N$5: now also R5.1; no longer JP2.1, X1G1.1
- net N$6: now also C9.2; no longer U1.VIN+
- net N$7: now also C9.1, R6.1, R8.1, U1.VIN+; no longer JP1.2, U1.VIN-
Other:
- moved on the sheet: JP1, X1, X1G

Commit message: HW: Update differential probe with latest design
Parts:
- removed SJ2: SOLDERJUMPERNC, SparkFun:SOLDERJUMPERNC
- added C11, C12, C13: (no value), resistor:C-EUC0402
- added LED1, LED3: RIGHT, led:LEDCHIPLED_0603
- added LED2: LEFT, led:LEDCHIPLED_0603
- added R11, R14: 10k, 1%, rcl:R-US_R0402
- added R12: 4k7, resistor:R-US_R0603
- added R13: 510R, 1%, rcl:R-US_R0402
- added R15: 25k, rcl:R-US_R0402
- added R16, R17: (no value), rcl:R-US_R0402
- added U$1, U$2, U$3, U$4, U$5, U$6: FIDUCIAL, adafruit:FIDUCIAL
- added U2: LM2903PWR, Texas Instruments_By_element14_Batch_1:LM2903PWR
- SJ1: value SOLDERJUMPERNC -> (none); device SparkFun:SOLDERJUMPERNC -> SparkFun:SOLDERJUMPER_2WAYPASTE1&2
Connections:
- new net N$16: R11.1, R13.1, U2.1IN+
- new net N$17: R13.2, R14.1, U2.2IN-
- new net N$18: R16.1, U2.1OUT
- new net N$19: C11.2, R15.2, U2.1IN-, U2.2IN+
- new net N$20: LED1.C, R16.2
- new net N$21: R17.1, U2.2OUT
- new net N$22: LED2.C, R17.2
- new net N$9: LED3.C, R12.1
- net AGND: now also C11.1, C12.2, C13.1, R12.2
- net N$1: now also LED3.A
- net N$10: now also SJ1.3; no longer SJ2.1
- net N$12: now also R15.1
- net N$2: now also C12.1, LED1.A, LED2.A, R11.2, U2.VCC
- net N$3: no longer SJ2.2
- net N$8: now also C13.2, R14.2, U2.GND

Commit message: Update differential probe stuff
Parts:
- removed C10, C9: 0R, rcl:C-EUC0603
- added R18, R19: 10R, resistor:R-US_R0603
- C11: value (none) -> 680pF
- C12, C13: value (none) -> 100nF
Connections:
- net N$13: now also R19.2; no longer C10.1
- net N$14: now also R19.1; no longer C10.2
- net N$6: now also R18.1; no longer C9.2
- net N$7: now also R18.2; no longer C9.1
Changed lines of the file:
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@@
 <part name="JP6" library="pinhead" deviceset="PINHD-1X1" device=""/>
 <part name="R5" library="resistor" deviceset="R-US_" device="R0603" value="49.9R"/>
-<part name="C9" library="rcl" deviceset="C-EU" device="C0603" value="0R"/>
-<part name="C10" library="rcl" deviceset="C-EU" device="C0603" value="0R"/>
 <part name="R6" library="resistor" deviceset="R-US_" device="M0805" value="DNM"/>
 <part name="R7" library="resistor" deviceset="R-US_" device="R0603" value="DNM"/>
@@
 <part name="R14" library="rcl" deviceset="R-US_" device="R0402" value="10k, 1%"/>
 <part name="R15" library="rcl" deviceset="R-US_" device="R0402" value="25k"/>
-<part name="C11" library="resistor" deviceset="C-EU" device="C0402"/>
+<part name="C11" library="resistor" deviceset="C-EU" device="C0402" value="680pF"/>
 <part name="SUPPLY13" library="adc_microboard" deviceset="AGND" device=""/>
 <part name="R16" library="rcl" deviceset="R-US_" device="R0402"/>
@@
 <part name="LED1" library="led" deviceset="LED" device="CHIPLED_0603" value="RIGHT"/>
 <part name="LED2" library="led" deviceset="LED" device="CHIPLED_0603" value="LEFT"/>
-<part name="C12" library="resistor" deviceset="C-EU" device="C0402"/>
-<part name="C13" library="resistor" deviceset="C-EU" device="C0402"/>
+<part name="C12" library="resistor" deviceset="C-EU" device="C0402" value="100nF"/>
+<part name="C13" library="resistor" deviceset="C-EU" device="C0402" value="100nF"/>
 <part name="SUPPLY14" library="adc_microboard" deviceset="AGND" device=""/>
 <part name="SUPPLY15" library="adc_microboard" deviceset="AGND" device=""/>
@@
 <part name="U$5" library="adafruit" deviceset="FIDUCIAL" device=""/>
 <part name="U$6" library="adafruit" deviceset="FIDUCIAL" device=""/>
+<part name="R18" library="resistor" deviceset="R-US_" device="R0603" value="10R"/>
+<part name="R19" library="resistor" deviceset="R-US_" device="R0603" value="10R"/>
 </parts>
 <sheets>
@@
 <instance part="JP6" gate="G$1" x="175.26" y="48.26"/>
 <instance part="R5" gate="G$1" x="132.08" y="119.38"/>
-<instance part="C9" gate="G$1" x="40.64" y="154.94" rot="R270"/>
-<instance part="C10" gate="G$1" x="40.64" y="144.78" rot="R270"/>
 <instance part="R6" gate="G$1" x="58.42" y="149.86" rot="R270"/>
 <instance part="R7" gate="G$1" x="63.5" y="144.78"/>
@@
 <instance part="U$5" gate="G$1" x="226.06" y="139.7"/>
 <instance part="U$6" gate="G$1" x="226.06" y="132.08"/>
+<instance part="R18" gate="G$1" x="40.64" y="154.94"/>
+<instance part="R19" gate="G$1" x="40.64" y="144.78"/>
 </instances>
 <busses>
@@
 <wire x1="17.78" y1="152.4" x2="33.02" y2="152.4" width="0.1524" layer="91"/>
 <wire x1="33.02" y1="152.4" x2="33.02" y2="154.94" width="0.1524" layer="91"/>
-<pinref part="C9" gate="G$1" pin="2"/>
 <wire x1="33.02" y1="154.94" x2="35.56" y2="154.94" width="0.1524" layer="91"/>
+<pinref part="R18" gate="G$1" pin="1"/>
 </segment>
 </net>
 <net name="N$7" class="0">
 <segment>
-<pinref part="C9" gate="G$1" pin="1"/>
 <pinref part="R6" gate="G$1" pin="1"/>
-<wire x1="43.18" y1="154.94" x2="50.8" y2="154.94" width="0.1524" layer="91"/>
+<wire x1="43.18" y1="154.94" x2="45.72" y2="154.94" width="0.1524" layer="91"/>
 <pinref part="R8" gate="G$1" pin="1"/>
 <junction x="58.42" y="154.94"/>
 <pinref part="U1" gate="G$1" pin="VIN+"/>
+<wire x1="45.72" y1="154.94" x2="50.8" y2="154.94" width="0.1524" layer="91"/>
 <wire x1="50.8" y1="154.94" x2="58.42" y2="154.94" width="0.1524" layer="91"/>
 <wire x1="96.52" y1="124.46" x2="50.8" y2="124.46" width="0.1524" layer="91"/>
 <wire x1="50.8" y1="124.46" x2="50.8" y2="154.94" width="0.1524" layer="91"/>
 <junction x="50.8" y="154.94"/>
+<pinref part="R18" gate="G$1" pin="2"/>
+<junction x="45.72" y="154.94"/>
 </segment>
 </net>
@@
 <segment>
 <pinref part="R6" gate="G$1" pin="2"/>
-<pinref part="C10" gate="G$1" pin="1"/>
 <wire x1="58.42" y1="144.78" x2="48.26" y2="144.78" width="0.1524" layer="91"/>
 <pinref part="R7" gate="G$1" pin="1"/>
 <junction x="58.42" y="144.78"/>
 <pinref part="U1" gate="G$1" pin="VIN-"/>
-<wire x1="48.26" y1="144.78" x2="43.18" y2="144.78" width="0.1524" layer="91"/>
+<wire x1="48.26" y1="144.78" x2="45.72" y2="144.78" width="0.1524" layer="91"/>
+<wire x1="45.72" y1="144.78" x2="43.18" y2="144.78" width="0.1524" layer="91"/>
 <wire x1="96.52" y1="121.92" x2="48.26" y2="121.92" width="0.1524" layer="91"/>
 <wire x1="48.26" y1="121.92" x2="48.26" y2="144.78" width="0.1524" layer="91"/>
 <junction x="48.26" y="144.78"/>
+<pinref part="R19" gate="G$1" pin="2"/>
+<junction x="45.72" y="144.78"/>
 </segment>
 </net>
 <net name="N$14" class="0">
 <segment>
-<pinref part="C10" gate="G$1" pin="2"/>
 <wire x1="35.56" y1="144.78" x2="33.02" y2="144.78" width="0.1524" layer="91"/>
 <wire x1="33.02" y1="144.78" x2="33.02" y2="149.86" width="0.1524" layer="91"/>
 <pinref part="JP1" gate="G$1" pin="2"/>
 <wire x1="33.02" y1="149.86" x2="17.78" y2="149.86" width="0.1524" layer="91"/>
-</segment>
-</net>
+<pinref part="R19" gate="G$1" pin="1"/>
+</segment>
+</net>

Commit message: HW: Update LNA + Diff probe with latest version
Parts:
- removed U$5: FIDUCIAL, adafruit:FIDUCIAL
Changed lines of the file:
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@@
 <grid distance="0.1" unitdist="inch" unit="inch" style="lines" multiple="1" display="no" altdistance="0.01" altunitdist="inch" altunit="inch"/>
 <layers>
-<layer number="1" name="Top" color="4" fill="1" visible="yes" active="no"/>
-<layer number="2" name="Route2" color="1" fill="3" visible="yes" active="no"/>
-<layer number="3" name="Route3" color="4" fill="3" visible="yes" active="no"/>
-<layer number="14" name="Route14" color="1" fill="6" visible="yes" active="no"/>
-<layer number="15" name="Route15" color="4" fill="6" visible="yes" active="no"/>
-<layer number="16" name="Bottom" color="1" fill="1" visible="yes" active="no"/>
-<layer number="17" name="Pads" color="2" fill="1" visible="yes" active="no"/>
-<layer number="18" name="Vias" color="2" fill="1" visible="yes" active="no"/>
-<layer number="19" name="Unrouted" color="6" fill="1" visible="yes" active="no"/>
-<layer number="20" name="Dimension" color="15" fill="1" visible="yes" active="no"/>
-<layer number="21" name="tPlace" color="7" fill="1" visible="yes" active="no"/>
-<layer number="22" name="bPlace" color="7" fill="1" visible="yes" active="no"/>
-<layer number="23" name="tOrigins" color="15" fill="1" visible="yes" active="no"/>
-<layer number="24" name="bOrigins" color="15" fill="1" visible="yes" active="no"/>
-<layer number="25" name="tNames" color="7" fill="1" visible="yes" active="no"/>
-<layer number="26" name="bNames" color="7" fill="1" visible="yes" active="no"/>
-<layer number="27" name="tValues" color="7" fill="1" visible="yes" active="no"/>
-<layer number="28" name="bValues" color="7" fill="1" visible="yes" active="no"/>
+<layer number="1" name="Top" color="4" fill="1" visible="no" active="no"/>
+<layer number="2" name="Route2" color="1" fill="3" visible="no" active="no"/>
+<layer number="3" name="Route3" color="4" fill="3" visible="no" active="no"/>
+<layer number="14" name="Route14" color="1" fill="6" visible="no" active="no"/>
+<layer number="15" name="Route15" color="4" fill="6" visible="no" active="no"/>
+<layer number="16" name="Bottom" color="1" fill="1" visible="no" active="no"/>
+<layer number="17" name="Pads" color="2" fill="1" visible="no" active="no"/>
+<layer number="18" name="Vias" color="2" fill="1" visible="no" active="no"/>
+<layer number="19" name="Unrouted" color="6" fill="1" visible="no" active="no"/>
+<layer number="20" name="Dimension" color="15" fill="1" visible="no" active="no"/>
+<layer number="21" name="tPlace" color="7" fill="1" visible="no" active="no"/>
+<layer number="22" name="bPlace" color="7" fill="1" visible="no" active="no"/>
+<layer number="23" name="tOrigins" color="15" fill="1" visible="no" active="no"/>
+<layer number="24" name="bOrigins" color="15" fill="1" visible="no" active="no"/>
+<layer number="25" name="tNames" color="7" fill="1" visible="no" active="no"/>
+<layer number="26" name="bNames" color="7" fill="1" visible="no" active="no"/>
+<layer number="27" name="tValues" color="7" fill="1" visible="no" active="no"/>
+<layer number="28" name="bValues" color="7" fill="1" visible="no" active="no"/>
 <layer number="29" name="tStop" color="7" fill="3" visible="no" active="no"/>
 <layer number="30" name="bStop" color="7" fill="6" visible="no" active="no"/>
@@
 <layer number="35" name="tGlue" color="7" fill="4" visible="no" active="no"/>
 <layer number="36" name="bGlue" color="7" fill="5" visible="no" active="no"/>
-<layer number="37" name="tTest" color="7" fill="1" visible="yes" active="no"/>
-<layer number="38" name="bTest" color="7" fill="1" visible="yes" active="no"/>
+<layer number="37" name="tTest" color="7" fill="1" visible="no" active="no"/>
+<layer number="38" name="bTest" color="7" fill="1" visible="no" active="no"/>
 <layer number="39" name="tKeepout" color="4" fill="11" visible="no" active="no"/>
 <layer number="40" name="bKeepout" color="1" fill="11" visible="no" active="no"/>
@@
 <layer number="44" name="Drills" color="7" fill="1" visible="no" active="no"/>
 <layer number="45" name="Holes" color="7" fill="1" visible="no" active="no"/>
-<layer number="46" name="Milling" color="3" fill="1" visible="yes" active="no"/>
-<layer number="47" name="Measures" color="7" fill="1" visible="yes" active="no"/>
-<layer number="48" name="Document" color="7" fill="1" visible="yes" active="no"/>
-<layer number="49" name="Reference" color="7" fill="1" visible="yes" active="no"/>
-<layer number="50" name="dxf" color="7" fill="1" visible="yes" active="no"/>
-<layer number="51" name="tDocu" color="7" fill="1" visible="yes" active="no"/>
-<layer number="52" name="bDocu" color="7" fill="1" visible="yes" active="no"/>
-<layer number="53" name="tGND_GNDA" color="7" fill="9" visible="yes" active="no"/>
-<layer number="54" name="bGND_GNDA" color="1" fill="9" visible="yes" active="no"/>
-<layer number="56" name="wert" color="7" fill="1" visible="yes" active="no"/>
+<layer number="46" name="Milling" color="3" fill="1" visible="no" active="no"/>
+<layer number="47" name="Measures" color="7" fill="1" visible="no" active="no"/>
+<layer number="48" name="Document" color="7" fill="1" visible="no" active="no"/>
+<layer number="49" name="Reference" color="7" fill="1" visible="no" active="no"/>
+<layer number="50" name="dxf" color="7" fill="1" visible="no" active="no"/>
+<layer number="51" name="tDocu" color="7" fill="1" visible="no" active="no"/>
+<layer number="52" name="bDocu" color="7" fill="1" visible="no" active="no"/>
+<layer number="53" name="tGND_GNDA" color="7" fill="9" visible="no" active="no"/>
+<layer number="54" name="bGND_GNDA" color="1" fill="9" visible="no" active="no"/>
+<layer number="56" name="wert" color="7" fill="1" visible="no" active="no"/>
 <layer number="91" name="Nets" color="2" fill="1" visible="yes" active="yes"/>
 <layer number="92" name="Busses" color="1" fill="1" visible="yes" active="yes"/>
@@
 <part name="U$3" library="adafruit" deviceset="FIDUCIAL" device=""/>
 <part name="U$4" library="adafruit" deviceset="FIDUCIAL" device=""/>
-<part name="U$5" library="adafruit" deviceset="FIDUCIAL" device=""/>
 <part name="U$6" library="adafruit" deviceset="FIDUCIAL" device=""/>
 <part name="R18" library="resistor" deviceset="R-US_" device="R0603" value="10R"/>
@@
 <instance part="U$3" gate="G$1" x="226.06" y="154.94"/>
 <instance part="U$4" gate="G$1" x="226.06" y="147.32"/>
-<instance part="U$5" gate="G$1" x="226.06" y="139.7"/>
 <instance part="U$6" gate="G$1" x="226.06" y="132.08"/>
 <instance part="R18" gate="G$1" x="40.64" y="154.94"/>

Commit message: PCBs: Add LNA/Diff-Probe updates, + firmware temp fixes
Parts:
- R13: value 510R, 1% -> 1k, 1%
- renumbered U$1 to FID5, U$2 to FID4, U$3 to FID2, U$4 to FID1, U$6 to FID6
Changed lines of the file:
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@@
 <?xml version="1.0" encoding="utf-8"?>
 <!DOCTYPE eagle SYSTEM "eagle.dtd">
-<eagle version="7.1.0">
+<eagle version="7.2.0">
 <drawing>
 <settings>
@@
 <part name="U2" library="Texas Instruments_By_element14_Batch_1" deviceset="LM2903PWR" device=""/>
 <part name="R11" library="rcl" deviceset="R-US_" device="R0402" value="10k, 1%"/>
-<part name="R13" library="rcl" deviceset="R-US_" device="R0402" value="510R, 1%"/>
+<part name="R13" library="rcl" deviceset="R-US_" device="R0402" value="1k, 1%"/>
 <part name="R14" library="rcl" deviceset="R-US_" device="R0402" value="10k, 1%"/>
 <part name="R15" library="rcl" deviceset="R-US_" device="R0402" value="25k"/>
@@
 <part name="R12" library="resistor" deviceset="R-US_" device="R0603" value="4k7"/>
 <part name="SUPPLY16" library="adc_microboard" deviceset="AGND" device=""/>
-<part name="U$1" library="adafruit" deviceset="FIDUCIAL" device=""/>
-<part name="U$2" library="adafruit" deviceset="FIDUCIAL" device=""/>
-<part name="U$3" library="adafruit" deviceset="FIDUCIAL" device=""/>
-<part name="U$4" library="adafruit" deviceset="FIDUCIAL" device=""/>
-<part name="U$6" library="adafruit" deviceset="FIDUCIAL" device=""/>
+<part name="FID5" library="adafruit" deviceset="FIDUCIAL" device=""/>
+<part name="FID4" library="adafruit" deviceset="FIDUCIAL" device=""/>
+<part name="FID2" library="adafruit" deviceset="FIDUCIAL" device=""/>
+<part name="FID1" library="adafruit" deviceset="FIDUCIAL" device=""/>
+<part name="FID6" library="adafruit" deviceset="FIDUCIAL" device=""/>
 <part name="R18" library="resistor" deviceset="R-US_" device="R0603" value="10R"/>
 <part name="R19" library="resistor" deviceset="R-US_" device="R0603" value="10R"/>
@@
 <instance part="R12" gate="G$1" x="167.64" y="129.54" rot="R270"/>
 <instance part="SUPPLY16" gate="G$1" x="167.64" y="121.92"/>
-<instance part="U$1" gate="G$1" x="226.06" y="170.18"/>
-<instance part="U$2" gate="G$1" x="226.06" y="162.56"/>
-<instance part="U$3" gate="G$1" x="226.06" y="154.94"/>
-<instance part="U$4" gate="G$1" x="226.06" y="147.32"/>
-<instance part="U$6" gate="G$1" x="226.06" y="132.08"/>
+<instance part="FID5" gate="G$1" x="226.06" y="170.18"/>
+<instance part="FID4" gate="G$1" x="226.06" y="162.56"/>
+<instance part="FID2" gate="G$1" x="226.06" y="154.94"/>
+<instance part="FID1" gate="G$1" x="226.06" y="147.32"/>
+<instance part="FID6" gate="G$1" x="226.06" y="132.08"/>
 <instance part="R18" gate="G$1" x="40.64" y="154.94"/>
 <instance part="R19" gate="G$1" x="40.64" y="144.78"/>
